File: eagle/tracker/tracker-balloon-full.brd (EAGLE design)
At the start: 100 x 75.5 mm, 90 parts, among them M1 UBLOX-NEO-6, M2 HOPE-RFM98W, M3 TFT-2.0-OPENSMART-THT, Q3 NTR5103N, U1 SI446X, U2 MCP73831, U3 A25L010A, U6 SI5351A, U8 STM32L052C8, X1 32.768kHz

Commit message: Added balloon/ground boards
Parts:
- removed C16, C27: 10p, kg-generic:C603
- removed C17, C18, C19, C20, C28: (no value), kg-generic:C603
- removed C21: 2u2, microbuilder_v3:_0603MP
- removed C22: NF/8p2/NF, microbuilder_v3:_0603MP
- removed C23: (no value), microbuilder_v3:_0603MP
- removed C24: 100n, kg-generic:C603
- removed C25, C26: 180p, kg-generic:C603
- removed CM: 10p/27p/68p, microbuilder_v3:_0603MP
- removed CM2: 15p/47p/150p, microbuilder_v3:_0603MP
- removed CM3: 8p2/27p/NF, microbuilder_v3:_0603MP
- removed ESD1: NF, microbuilder_v3:_0603MP
- removed ESD2, ESD3: 0.25p, microbuilder_v3:_0603MP
- removed FB2, FB4, FB5, FB6: (no value), microbuilder_v3:_0805
- removed JP6: PROG, pinhead:1X04
- removed L0: 56n/100n/3.9u, microbuilder_v3:_0805MP
- removed L1, L2: (no value), microbuilder_v3:_0805MP
- removed LED1, LED4: (no value), led:CHIPLED_0805
- removed LM: 18n/68n/1.5u, microbuilder_v3:_0805MP
- removed LM1: 4.7u, microbuilder_v3:_0805MP
- removed LM2: 18n/68n/330n, microbuilder_v3:_0805MP
- removed LM3: 0.47u, microbuilder_v3:_0805MP
- removed LR1, LR3: 220n/470n, microbuilder_v3:_0805MP
- removed M3: TFT-2.0-OPENSMART-THT, kg-modules:TFT-2.0-OPENSMART
- removed S1, S2, S3: MOMENTARY-SWITCH-SPST-SMD-6.2MM-TALL, SparkFun-Switches:TACTILE_SWITCH_SMD_6.2MM_TALL
- removed TP3: TPSB1,27, testpad:B1,27
- removed U$42: MINI-USB-B, kg-sdrlib:MINI-B-USB
- removed U8: STM32L052C8, kg-mcu:LQFP48
- removed X2, X3: (no value), kg-conn-rf:SMA_EDGELAUNCH
- removed XO1: 26.000MHz TCXO, kg-crystal:CRYSTAL-SMD-2.5X2
- added D1: (no value), kg-generic:R0805
- added J1: BATT, kg-amp-ct:JST-2-PTH-VERT
- added J2: USB_MINI-B_SMT, SparkFun-Connectors:USB-MINIB
- added J3: BATT_PYRO, kg-amp-ct:JST-2-PTH-VERT
- added J4: (no value), kg-amp-ct:JST-4-PTH-VERT
- added J6: (no value), kg-amp-ct:JST-3-PTH-VERT
- added JP5: LDO_BYPASS, SparkFun-Passives:PAD-JUMPER-2-NO_YES_SILK
- added L1A, L1B: (no value), kg-generic:R0603
- added M4: UBLOX-MAX-M8, kg-modules:UBLOX-MAX
- added PAD2: (no value), wirepad:SMD2,54-5,08
- added Q2, Q4: (no value), kg-generic:SOT23-3
- added R16, R17, R18, R21, R22, R23, R24, R25: 100k, kg-generic:R0603
- added R19, R26: 1k, kg-generic:R0603
- added R20: 10k, kg-generic:R0603
- added SG1: F/TMB, buzzer:F/TMB
- added U$29: STM32L063C, kg-mcu:LQFP48
- added U5: LSM6DS33, kg-ic:TFLGA16L
- added X2A, X2B, X6: COAX, kg-conn-rf:MMCX-J-P-X-ST-EM1-MKT
- C1: value 10n -> 100n
- C10, C3, C6, C7, C9: value (none) -> 100n
- C11: value 100n -> 1u; device microbuilder_v3:_0603MP -> kg-generic:C603
- C12: device kg-generic:C603 -> rcl:E3,5-8
- C13: value 10n -> 100n; device microbuilder_v3:_0603MP -> kg-generic:C603
- C14, C15: device microbuilder_v3:_0603MP -> kg-generic:C603
- C2: value (none) -> 10u; device kg-generic:C603 -> kg-generic:EIA3216
- C4: value NF/8p2/NF -> 1u; device microbuilder_v3:_0603MP -> kg-generic:C603
- C5: value NF* -> 1u
- C8: value 2n2 -> 1u; device microbuilder_v3:_0603MP -> kg-generic:C603
- JP1: value BATT -> BYPASS2; device pinhead:1X02 -> SparkFun-Passives:PAD-JUMPER-2-NO_YES_SILK
- M1: value UBLOX-NEO-6 -> UBLOX-NEO-M8
- PAD1: device wirepad:1,6/0,8 -> wirepad:SMD2,54-5,08
- Q3: value NTR5103N -> (none)
- R1: value 10k -> 1k; device rcl:R0603 -> kg-generic:R0603
- R10, R11, R13: value (none) -> 100k
- R12: value 470 -> 100; device rcl:R0603 -> kg-generic:R0603
- R14: value 5.1k -> 10k
- R15: value 10 -> 3.3k; device kg-generic:R0603 -> rcl:R0603
- R5: value (none) -> 10k
- R6, R7: value (none) -> 1k
- R8: value (none) -> 3.3k; device kg-generic:R0603 -> rcl:R0603
- R9: value 10k -> (none); device rcl:R0603 -> kg-generic:R0603
- U1: value SI446X -> MS5637-02; device kg-sdrlib:QFN20 -> kg-ic:MS5637
- U2: value MCP73831 -> (none); device kg-supply:SOT23-5 -> kg-generic:SOT23-5
- U4: value (none) -> MAG3110FCR1; device kg-generic:SOT23-3 -> kg-ic:DFN200X200X90-10N
- U6: value SI5351A -> (none); device kg-sdrlib:MSOP10 -> kg-generic:SOT23-5
- X1: value 32.768kHz -> 87758-0416; device IQD-Frequency-Products:3.2X1.5-2-PAD -> con-molex:87758-0416
- X4: value (none) -> MICROMATCH-8; device kg-conn-rf:SMA_EDGELAUNCH -> con-amp-micromatch:MICROMATCH-8
- moved R5 76.9 mm to (12.5, 18.5), flipped to the bottom, turned to 0 degrees
- moved JP1 50.3 mm to (32.5, 30.5)
- moved U4 46.5 mm to (41.0, 13.5), turned to 90 degrees
- moved C2 45.5 mm to (52.0, 32.0), flipped to the bottom, turned to 270 degrees
- moved R6 45.2 mm to (43.0, 45.0), turned to 270 degrees
- moved R8 44.5 mm to (60.0, 10.0), flipped to the bottom, turned to 90 degrees
- moved C5 43.9 mm to (49.5, 32.5), turned to 270 degrees
- moved R13 43.9 mm to (53.0, 31.5)
- moved C3 43.7 mm to (44.0, 23.5)
- moved X4 41.4 mm to (3.50, 28.0)
- moved U2 38.8 mm to (46.0, 32.5), flipped to the bottom, turned to 90 degrees
- moved R15 37.8 mm to (65.0, 16.5), turned to 180 degrees
- moved C14 37.7 mm to (38.5, 13.5), flipped to the bottom
- moved R12 37.5 mm to (23.5, 31.0), flipped to the bottom, turned to 90 degrees
- moved R2 36.2 mm to (67.5, 29.0), turned to 0 degrees
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Connections:
- removed net !LORA_CS: M2.5, U8.21
- removed net !LORA_IRQ: M2.14
- removed net !LORA_RST: M2.6, U8.22
- removed net !RADIO_ON: Q1.1, R1.1
- removed net !TFT_CS: M3.P$6, U8.26
- removed net !TFT_LED: M3.P$8, U8.28
- removed net !TFT_RST: M3.P$7, U8.25
- removed net !TRX_CS: U1.15, U8.14
- removed net !TRX_EN: U1.1, U8.11
- removed net !TRX_IRQ: U1.11, U8.18
- removed net +3V3: C2.2, C3.2, FB2.1, LED1.A, M3.P$2, Q1.2, R1.2, R3.2, R4.2, R9.2, U3.8, U4.2, U8.1, U8.24, U8.36, U8.48, U8.9
- removed net 3V3_RADIO: C12.2, FB1.2, FB3.1, FB4.2, FB6.1, XO1.4
- removed net 3V3_TRX: C11.1, C21.1, C7.2, C8.1, FB1.1, LR3.2, R11.1, U1.6
- removed net BAT_CHG: R8.1, U2.1
- removed net N$18: C18.2, JP1.2, R13.2, U2.3, U4.3
- removed net N$26: FB5.2, U$42.1
- removed net N$27: U8.4, X1.1
- removed net N$28: C10.2, FB4.1, M2.13
- removed net N$30: C24.2, R15.1
- removed net N$32: CM2.1, LM.1, LM2.2
- removed net N$33: R6.1, U$42.3
- removed net N$34: C9.2, FB2.2, M1.23
- removed net N$35: LED4.C, R12.2
- removed net N$36: C16.2, C27.2, LR1.1, Q3.3
- removed net N$37: C6.2, M2.9
- removed net N$38: C22.1, L1.1, L2.2, U1.2
- removed net N$39: C23.2, L1.2, U1.3
- removed net N$40: FB6.2, Q1.3
- removed net N$8: M1.8, M1.9
- removed net RADIO_XIN: C13.2, U1.17
- removed net RF_TANK: C23.1, CM.1, L0.1, L2.1, LM.2
- removed net RF_TANK1: C16.1, LM1.2
- removed net SHLD$1: U$42.SHLD$1
- removed net SHLD$2: U$42.SHLD$2
- removed net SHLD$3: U$42.SHLD$3
- removed net SHLD$4: U$42.SHLD$4
- removed net TCXO_OUT: C1.2, C13.1, XO1.3
- removed net TFT_RS: M3.P$5, U8.27
- removed net TRX_GPIO0: U1.9, U8.20
- removed net TRX_GPIO1: U1.10, U8.19
- removed net TRX_GPIO2: U1.19
- removed net TRX_GPIO3: U1.20
- removed net USB_DM: R5.2, U8.32
- removed net USB_DP: R6.2, U8.33
- removed net USB_VBUS: C19.2, FB5.1, U2.4
- removed net VBAT_ADC: C17.2, R10.2, R13.1, U8.10
- new net !RFM_RST: M2.6
- new net !RFM_SS: M2.5
- new net 3.3V: C15.2, C2.A, C3.2, C5.2, C7.2, FB1.2, FB3.1, JP5.2, R14.2, R3.2, R4.2, R5.1, R9.2, U$29.1, U$29.24, U$29.36, U$29.48, U$29.9, U1.1, U2.5, U3.3, U3.7, U3.8, U4.2, U4.8, U5.1, U5.16, U5.4, U5.5, U6.1, U6.3
- new net BUZZER: R7.1
- new net CMD1: R17.1, R19.1, U$29.19
- new net CMD2: R1.1, R18.1, U$29.18
- new net DBG_RX: J6.2, U$29.13
- new net DBG_TX: J6.3, U$29.12
- new net GPS_VCC: C9.2, FB3.2, M1.2, M1.23, M4.7, M4.8, R15.2
- new net PYRO1_OUT: Q2.3, R21.1, X4.4
- new net PYRO2_OUT: Q3.3, R22.1, X4.2
- new net PYRO_SENSE: R16.2, R23.2, U$29.11
- new net RFM_DIO0: M2.14, U$29.20
- new net SAFE: R20.2, X4.6
- new net SENSE1: R21.2, R24.2, U$29.15
- new net SENSE2: R22.2, R25.2, U$29.14
- new net SENSE_ARM: R26.2, U$29.17
- new net SHDN: R10.1, U2.3, X4.8
- new net VBUS: J2.VBUS
- new net VCC_PYRO: C12.+, J3.2, JP1.2, R12.2, R16.1, X4.1, X4.3
- new net V_BATT: C4.2, J1.2, JP1.1, JP5.1, PAD1.1, R10.2, R11.2, SG1.+, U2.1
- new net V_BATT_SENSE: C10.2, R11.1, R13.2, U$29.10
- net !FLASH_CS: now also R14.1
- net !RST: now also C1.2, J4.2, U$29.7; no longer C14.1, JP6.4, U8.7
- net GND: now also C1.1, C11.1, C12.-, C13.1, C14.1, C15.1, C2.C, C4.1, C5.1, C6.1, C8.1, D1.2, J1.1, J2.GND, J3.1, J4.1, J6.1, L1A.1, L1B.1, M4.1, M4.10, M4.12, M4.6, Q1.2, Q4.2, R13.1, R17.2, R18.2, R2.1, R23.1, R24.1, R25.1, U$29.23, U$29.35, U$29.44, U$29.47, U$29.8, U1.4, U4.10, U4.5, U5.10, U5.11, U5.12, U5.13, U5.15, U5.8, U5.9, U6.2, X2A.2@1, X2A.2@2, X2A.2@3, X2A.2@4, X2B.2@1, X2B.2@2, X2B.2@3, X2B.2@4, X4.5, X4.7, X6.2@1, X6.2@2, X6.2@3, X6.2@4; no longer C11.2, C12.1, C14.2, C15.2, C17.1, C18.1, C19.1, C2.1, C20.1, C21.2, C22.2, C25.1, C26.1, C27.1, C4.2, C8.2, CM.2, CM2.2, CM3.2, ESD1.1, ESD2.1, ESD3.1, JP1.1, JP6.1, M3.P$1, Q3.2, R10.1, R12.1, R14.1, R7.1, U$42.5, U1.18, U1.5, U1.PAD, U4.1, U6.8, U8.23, U8.35, U8.44, U8.47, U8.8, X2.GND@1, X2.GND@2, X2.GND@3, X2.GND@4, X3.GND@1, X3.GND@2, X3.GND@3, X3.GND@4, X4.GND@1, X4.GND@2, X4.GND@3, X4.GND@4, XO1.2
- net GPS_PPS: now also M4.4; no longer TP3.TP, U8.2
- net GPS_RXD: now also M4.2, U$29.43; no longer U8.31
- net GPS_TXD: now also M4.3, U$29.42; no longer U8.30
- net LED: now also R6.2; no longer LED4.A
- net MISO: now also U$29.40; no longer U1.13, U8.16
- net MOSI: now also U$29.41; no longer M3.P$3, U1.14, U8.17
- net N$12: now also PAD2.1, Q1.3, SG1.-; no longer C28.2, LR3.1, U1.4
- net N$13: now also C6.2, FB1.1, M2.13; no longer R15.2, U6.10
- net N$14: now also M1.8, R8.1; no longer R7.2, U2.5
- net N$15: now also M1.9, R8.2; no longer C28.1, C4.1, L0.2
- net N$16: now also C8.2, U2.4; no longer LED1.C, R8.2
- net N$17: now also Q2.2, Q3.2, Q4.3; no longer M1.14
- net N$19: now also D1.1, R6.1; no longer C5.2, M1.11, PAD1.1
- net N$20: now also Q2.1, R19.2; no longer C20.2, FB3.2, LR1.2, R2.2, U6.1, U6.7
- net N$21: now also C11.2, R12.1, U6.5; no longer U8.3, X1.2
- net N$22: now also C13.2, U4.1; no longer C15.1, R11.2, U1.8
- net N$23: now also C14.2, U4.4; no longer C1.1, U6.2
- net N$24: now also M4.9, R15.1; no longer C25.2, ESD3.2, LM3.1, X4.P
- net N$25: now also Q3.1, R1.2; no longer C26.2, LM1.1, LM3.2
- net N$29: now also Q4.1, R20.1, R26.1, R5.2; no longer R5.1, U$42.2
- net N$31: now also M2.9, X6.1; no longer C6.1, CM3.1, ESD2.2, LM2.1, X2.P
- net N$5: now also L1A.2, L1B.2, M1.11, M4.11, X2A.1, X2B.1; no longer C24.1, Q3.1, R14.2, R2.1
- net N$9: now also Q1.1, R2.2, R7.2; no longer C5.1, ESD1.2, X3.P
- net SCK: now also U$29.39; no longer M3.P$4, U1.12, U8.15
- net SCL: now also U$29.45, U1.3, U4.7, U5.2; no longer U6.4, U8.42
- net SDA: now also U$29.46, U1.2, U4.6, U5.3; no longer U6.5, U8.43
- net SWCLK: now also J4.3, U$29.37; no longer JP6.3, U8.37
- net SWDIO: now also J4.4, U$29.34; no longer JP6.2, U8.34
Routing:
- net 3.3V: track 0.00 -> 68.3 mm, vias 0 -> 8
- net SCK: track 50.8 -> 0.00 mm, vias 4 -> 0
- net MOSI: track 50.1 -> 0.00 mm, vias 3 -> 0
- net !TFT_LED: track 34.6 -> 0.00 mm, vias 1 -> 0
- net !TFT_RST: track 32.9 -> 0.00 mm, vias 1 -> 0
- net !TFT_CS: track 32.4 -> 0.00 mm, vias 1 -> 0
- net MISO: track 31.9 -> 0.00 mm, vias 5 -> 0
- net TFT_RS: track 31.6 -> 0.00 mm, vias 1 -> 0
- net GPS_VCC: track 0.00 -> 28.1 mm, vias 0 -> 3
- net !LORA_RST: track 26.5 -> 0.00 mm, vias 1 -> 0
- net V_BATT: track 0.00 -> 25.5 mm, vias 0 -> 1
- net !LORA_CS: track 24.2 -> 0.00 mm, vias 1 -> 0
- net !TRX_EN: track 16.1 -> 0.00 mm, vias 2 -> 0
- net SDA: track 0.00 -> 16.1 mm, vias 0 -> 3
- net SCL: track 0.00 -> 12.2 mm, vias 0 -> 2
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Other:
- board size 100 x 75.5 mm -> 74 x 36 mm
- board text added: "BAT"
- board text added: "EXT"
- board text added: "GNSS"
- board text added: "LoRa"
- board text added: "PROG"
- board text added: "SDN"
- board text added: "TODO: - TABS for battery straps"
- board text added: "Tracker"
- board text added: "v1.0"
- board text removed: "Ant"
- board text removed: "BKP"
- board text removed: "Bat"
- board text removed: "CFG0"
- board text removed: "Chg"
- board text removed: "Dbg"
- board text removed: "Ext"
- board text removed: "TReX"
- board text removed: "v1.1"
