File: eagle/tracker/tracker-balloon-full.brd (EAGLE design)
At the start: 74 x 74 mm, 80 parts, among them J1 BATT, J2 USB_MINI-B_SMT, J3 BATT_PYRO, J5 MICRO-SD_CARD_SOCKET, M1 UBLOX-NEO-M8, M2 HOPE-RFM98W, M3 SIM800L-MODULE, M4 UBLOX-MAX-M8, U1 MS5637-02, U3 A25L010A, U4 MAG3110FCR1, U5 LSM6DS33, U7 MCP73831, X1 87758-0416, X2A COAX, X2B COAX, X4 MICROMATCH-8, X6 COAX

Commit message: Updates to balloon flight board
Parts:
- removed L1B: (no value), kg-generic:R0603
- removed X2A, X2B: COAX, kg-conn-rf:MMCX-J-P-X-ST-EM1-MKT
- added D10, D11, D6, D7, D8, D9: (no value), kg-generic:R0805
- added D3, D4, D5: (no value), kg-generic:SOD-323
- added J7: BATT_PYRO, kg-amp-ct:JST-2-PTH-VERT
- added JP2, JP3, JP4, JP6: (no value), pinhead:1X03
- added JP7: (no value), pinhead:2X03
- added Q10, Q11, Q12, Q5, Q6, Q7, Q8, Q9: (no value), kg-generic:SOT23-3
- added R28, R29, R30, R31, R32, R33, R35, R36, R38, R39, R40, R41, R42, R43, R44, R45: 1k, kg-generic:R0603
- added R34, R37, R46: 100k, kg-generic:R0603
- added R47: (no value), kg-generic:R0603
- added X10, X7, X8, X9: (no value), con-wago-500:W237-102
- added X2, X3, X5: (no value), kg-conn-rf:SMA_EDGELAUNCH
- R17, R18: value 100k -> 1k
- X1: value 87758-0416 -> (none); device con-molex:87758-0416 -> con-wago-500:W237-102
- X4: value MICROMATCH-8 -> ANTENNA-PATCH-12X12; device con-amp-micromatch:MICROMATCH-8 -> kg-modules:ANT-PATCH-12X12
- X6: value COAX -> (none); device kg-conn-rf:MMCX-J-P-X-ST-EM1-MKT -> con-wago-500:W237-102
- moved X4 84.5 mm to (93.0, 61.0), turned to 0 degrees
- moved SG1 71.5 mm to (2.00, 45.5), turned to 270 degrees
- moved R27 71.4 mm to (2.50, 47.0), turned to 180 degrees
- moved PAD2 71.3 mm to (3.25, 49.2), turned to 270 degrees
- moved J1 70.5 mm to (9.50, 3.50), turned to 0 degrees
- moved D2 70.3 mm to (2.50, 45.0), turned to 180 degrees
- moved PAD1 68.2 mm to (3.25, 41.8), turned to 270 degrees
- moved M3 66.9 mm to (19.5, 56.0), turned to 0 degrees
- moved C4 66.2 mm to (7.00, 12.5), turned to 180 degrees
- moved M2 66.2 mm to (63.5, 57.5)
- moved R10 66.1 mm to (7.00, 13.5), turned to 0 degrees
- moved R6 66.0 mm to (5.00, 37.5), turned to 90 degrees
- moved U2 65.8 mm to (7.00, 16.0), turned to 0 degrees
- moved C5 65.8 mm to (7.00, 19.5), turned to 180 degrees
- moved C8 65.8 mm to (7.00, 18.0), turned to 180 degrees
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Connections:
- new net DO_LOAD1: R32.1, R43.1
- new net DO_LOAD2: R35.1, R44.1
- new net DO_LOAD3: R38.1, R45.1
- new net DO_SRV1: R39.1
- new net DO_SRV2: R40.1
- new net DO_SRV3: R41.1
- new net DO_SRV4: R42.1
- new net N$26: M3.1, X5.P
- new net N$28: J2.D-, R28.2
- new net N$30: J2.D+, R29.2
- new net N$32: JP6.1, R42.2
- new net N$33: D3.A, Q5.1, R30.1, R34.1
- new net N$34: Q8.3, R30.2
- new net N$35: Q8.1, R32.2
- new net N$36: Q5.3, X8.1
- new net N$37: D6.1, R43.2
- new net N$38: JP4.1, R41.2
- new net N$39: D4.A, Q6.1, R33.1, R37.1
- new net N$40: Q7.3, R33.2
- new net N$41: Q7.1, R35.2
- new net N$42: Q6.3, X9.1
- new net N$43: JP3.1, R40.2
- new net N$44: JP2.1, R39.2
- new net N$45: D5.A, Q9.1, R36.1, R46.1
- new net N$46: Q10.3, R36.2
- new net N$47: Q10.1, R38.2
- new net N$48: Q9.3, X10.1
- new net N$49: D9.1, R17.2
- new net N$50: D8.1, R45.2
- new net N$51: D7.1, R44.2
- new net N$52: D10.1, R18.2
- new net N$53: D11.1, R31.2
- new net N$54: M3.2, Q11.3
- new net N$55: Q11.1, Q12.3, R47.1
- new net USB_DM: R28.1, U$29.32
- new net USB_DP: R29.1, U$29.33
- new net V_GSM: J7.2, Q11.2, R47.2
- new net V_LOAD: D3.C, D4.C, D5.C, Q5.2, Q6.2, Q9.2, R34.2, R37.2, R46.2, X1.1
- new net V_SERVO: JP2.2, JP3.2, JP4.2, JP6.2
- net !FLASH_CS: now also J5.CS
- net 3.3V: now also J5.VCC, R31.1
- net GND: now also D10.2, D6.2, D7.2, D8.2, D9.2, J5.GND, J5.GND1, J5.GND3, J7.1, JP2.3, JP3.3, JP4.3, JP6.3, M3.6, Q10.2, Q12.2, Q7.2, Q8.2, X1.2, X10.2, X2.GND@1, X2.GND@2, X2.GND@3, X2.GND@4, X3.GND@1, X3.GND@2, X3.GND@3, X3.GND@4, X5.GND@1, X5.GND@2, X5.GND@3, X5.GND@4, X8.2, X9.2; no longer L1B.1, R17.2, R18.2, X2A.2@1, X2A.2@2, X2A.2@3, X2A.2@4, X2B.2@1, X2B.2@2, X2B.2@3, X2B.2@4, X4.5, X4.7, X6.2@1, X6.2@2, X6.2@3, X6.2@4
- net N$17: now also D11.2
- net N$31: now also X2.P; no longer X6.1
- net N$5: now also X3.P, X4.FEED; no longer L1B.2, X2A.1, X2B.1
- net PYRO1_OUT: now also X6.2; no longer X4.4
- net PYRO2_OUT: now also X7.2; no longer X4.2
- net SAFE: no longer X4.6
- net SHDN: no longer X4.8
- net VCC_PYRO: now also X6.1, X7.1; no longer X4.1, X4.3
Routing:
- net V_BATT: track 25.5 -> 14.2 mm
- net N$5: track 8.76 -> 0.00 mm, vias 3 -> 0
Other:
- board size 74 x 74 mm -> 100 x 80 mm

Commit message: Tracker ready for order
Parts:
- removed D2: (no value), kg-generic:R0805
- removed JP1: BYPASS2, SparkFun-Passives:PAD-JUMPER-2-NO_YES_SILK
- removed JP5: LDO_BYPASS, SparkFun-Passives:PAD-JUMPER-2-NO_YES_SILK
- removed JP7: (no value), pinhead:2X03
- removed PAD1, PAD2: (no value), wirepad:SMD2,54-5,08
- removed SG1: F/TMB, buzzer:F/TMB
- removed X1, X10, X6, X7, X8, X9: (no value), con-wago-500:W237-102
- added C16, C17, C18: 1u, kg-generic:C603
- added C19: 100n, kg-generic:C603
- added D12, D13, D14: (no value), kg-generic:R0805
- added J10, J11, J12, J8, J9: (no value), kg-amp-ct:SCREWTERMINAL-3.81MM-2
- added J14: 1WIRE, kg-amp-ct:JST-3-PTH-VERT
- added R48, R50, R52, R53, R54, R55, R56: 1k, kg-generic:R0603
- added R49: 100k, kg-generic:R0603
- added R51: 10k, kg-generic:R0603
- added R57: 100, kg-generic:R0603
- added SV1: PANEL, con-ml:ML6
- added SV2: I2C/GPS, con-ml:ML6
- added U8: MCP73831, kg-supply:SOT23-5
- C1: value 100n -> 10n
- J3: value BATT_PYRO -> (none); device kg-amp-ct:JST-2-PTH-VERT -> kg-amp-ct:SCREWTERMINAL-3.81MM-2
- J7: value BATT_PYRO -> BATT_GSM
- R27: value 1k -> 100k
- R47: value (none) -> 100k
- R9: value (none) -> 10k
- moved J2 91.1 mm to (5.50, 45.5), turned to 0 degrees
- moved U7 85.9 mm to (10.5, 61.0), turned to 180 degrees
- moved Q1 83.4 mm to (87.5, 30.5)
- moved R2 83.4 mm to (87.5, 27.5)
- moved R7 83.4 mm to (87.5, 25.5)
- moved R27 65.0 mm to (-9.00, -17.0), turned to 0 degrees
- moved J6 55.1 mm to (57.5, 33.0), turned to 270 degrees
- moved R6 46.6 mm to (51.5, 41.0)
- moved D1 43.2 mm to (49.5, 41.0), flipped to the top
- moved J4 39.1 mm to (51.0, 33.0), turned to 270 degrees
- moved R29 37.5 mm to (13.0, 45.0), turned to 180 degrees
- moved R28 36.7 mm to (13.0, 46.5), turned to 180 degrees
- moved C10 24.8 mm to (30.5, 34.0), turned to 0 degrees
- moved R13 22.7 mm to (30.5, 32.5), turned to 0 degrees
- moved J3 21.1 mm to (39.5, 6.00)
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Connections:
- net CMD1 renamed D_PYRO1
- net CMD2 renamed D_PYRO2
- net DO_LOAD1 renamed D_LOAD1
- net DO_LOAD2 renamed D_LOAD2
- net DO_LOAD3 renamed D_LOAD3
- net PYRO_SENSE renamed V_PYRO_SENSE
- net SENSE1 renamed PYRO1_SENSE
- net SENSE2 renamed PYRO2_SENSE
- net SENSE_ARM renamed ARM_SENSE
- removed net BUZZER: R7.1
- removed net N$8: D2.2, R27.2
- new net !GSM_RST: M3.3
- new net D_BUZZER: R2.2, R7.1
- new net GSM_ON: R48.1, R49.2
- new net GSM_RXD: M3.5
- new net GSM_TXD: M3.4
- new net N$57: M3.11, R51.2
- new net N$58: D13.1, R52.2
- new net N$59: D14.1, R53.2
- new net N$60: D14.2, U7.1
- new net N$61: D13.2, U8.1
- new net N$63: R54.2, U8.5
- new net N$64: R55.2, U7.5
- new net NTC_EXT: C19.2, R27.1, R56.2
- new net NTC_SENSE: R56.1
- new net V_BUZZER+: R57.1
- new net V_BUZZER-: Q1.3
- net 3.3V: now also R27.2; no longer JP5.2
- net GND: now also C16.1, C17.1, C18.1, C19.1, J10.1, J8.1, J9.1, R49.1, R50.1, R51.1, R54.1, R55.1, U7.2, U8.2; no longer X1.2, X10.2, X8.2, X9.2
- net N$12: now also Q12.1, R48.2; no longer PAD2.1, Q1.3, R27.1, SG1.-
- net N$27: now also D12.2, R50.2; no longer U7.3
- net N$36: now also J8.2; no longer X8.1
- net N$42: now also J9.2; no longer X9.1
- net N$48: now also J10.2; no longer X10.1
- net N$54: now also D12.1
- net N$9: no longer R2.2
- net PYRO1_OUT: now also J11.1; no longer X6.2
- net PYRO2_OUT: now also J12.1; no longer X7.2
- net VCC_PYRO: now also J11.2, J12.2; no longer J3.2, JP1.2, X6.1, X7.1
- net V_BATT: now also C17.2, R57.2, U8.3; no longer D2.1, JP1.1, JP5.1, PAD1.1, SG1.+
- net V_GSM: now also C18.2, U7.3
- net V_LOAD: now also J3.2; no longer X1.1
- net V_USB: now also C16.2, R52.1, R53.1, U8.4
Routing:
- net V_BATT: track 14.2 -> 0.00 mm, vias 1 -> 0
- net N$12: track 6.03 -> 0.00 mm
- net 3.3V: track 62.5 -> 56.5 mm, vias 6 -> 5
- net N$9: track 4.04 -> 0.00 mm
- net SHDN: track 1.23 -> 0.00 mm, vias 1 -> 0
- net N$16: track 0.72 -> 0.00 mm, vias 1 -> 0
- net GND: vias 11 -> 10

Commit message: Updates
Parts:
- moved J14 111.4 mm to (68.5, 37.5)
- moved SV2 109.4 mm to (80.0, 6.50)
Changed lines of the file:
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@@
 <element name="R56" library="kg-generic" package="R0603" value="1k" x="-8" y="-20.5"/>
 <element name="R57" library="kg-generic" package="R0603" value="100" x="87.5" y="33.5" rot="R180"/>
-<element name="J14" library="kg-amp-ct" package="JST-3-PTH-VERT" value="1WIRE" x="-1" y="-49.5"/>
-<element name="SV2" library="con-ml" package="ML6" value="I2C/GPS" x="-1.5" y="-66.5">
-<attribute name="OC_FARNELL" value="unknown" x="-1.5" y="-66.5" size="1.778" layer="27" display="off"/>
-<attribute name="MPN" value="" x="-1.5" y="-66.5" size="1.778" layer="27" display="off"/>
-<attribute name="OC_NEWARK" value="unknown" x="-1.5" y="-66.5" size="1.778" layer="27" display="off"/>
-<attribute name="MF" value="" x="-1.5" y="-66.5" size="1.778" layer="27" display="off"/>
+<element name="J14" library="kg-amp-ct" package="JST-3-PTH-VERT" value="1WIRE" x="68.5" y="37.5"/>
+<element name="SV2" library="con-ml" package="ML6" value="I2C/GPS" x="80" y="6.5">
+<attribute name="OC_FARNELL" value="unknown" x="80" y="6.5" size="1.778" layer="27" display="off"/>
+<attribute name="MPN" value="" x="80" y="6.5" size="1.778" layer="27" display="off"/>
+<attribute name="OC_NEWARK" value="unknown" x="80" y="6.5" size="1.778" layer="27" display="off"/>
+<attribute name="MF" value="" x="80" y="6.5" size="1.778" layer="27" display="off"/>
 </element>
 </elements>

Commit message: Updated balloon board
Parts:
- removed SV1: PANEL, con-ml:ML6
- removed SV2: I2C/GPS, con-ml:ML6
- removed U$29: STM32L063C, kg-mcu:LQFP48
- added J13: INTERN, kg-amp-ct:MICROMATCH-4
- added J15: EXTERN, kg-amp-ct:MICROMATCH-6
- added U9: STM32L072R, kg-mcu:LQFP64
- J10: value (none) -> AUX3
- J14: value 1WIRE -> THERMO
- J3: value (none) -> BATT AUX
- J4: value (none) -> SWD
- J6: value (none) -> UART
- J7: value BATT_GSM -> BATT GSM
- J8: value (none) -> AUX1
- J9: value (none) -> AUX2
- R12: value 100 -> 22
- moved R56 96.6 mm to (63.5, 44.5)
- moved R27 93.2 mm to (63.5, 41.5), turned to 180 degrees
- moved C19 91.9 mm to (63.5, 43.0)
- moved C6 63.0 mm to (54.0, 59.0), turned to 90 degrees
- moved FB1 59.8 mm to (51.5, 59.0), turned to 270 degrees
- moved D1 49.7 mm to (91.5, 67.5)
- moved R6 49.7 mm to (93.5, 67.5)
- moved J6 48.1 mm to (37.0, 76.5), turned to 0 degrees
- moved J4 45.0 mm to (62.5, 76.5), turned to 0 degrees
- moved J14 35.1 mm to (89.0, 9.00), turned to 90 degrees
- moved U6 34.0 mm to (44.0, 14.0), turned to 90 degrees
- moved J7 32.1 mm to (11.1, 33.6), turned to 300 degrees
- moved R12 31.8 mm to (44.0, 18.0), turned to 180 degrees
- moved C12 31.6 mm to (44.0, 10.5)
- moved L1A 31.0 mm to (86.2, 45.5)
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Connections:
- net D_BUZZER renamed BUZZER_ON
- net LED renamed LED_STATUS
- removed net D_PYRO1: R17.1, R19.1, U$29.19
- removed net D_PYRO2: R1.1, R18.1, U$29.18
- removed net N$21: C11.2, R12.1, U6.5
- new net N$8: C11.2, R12.1, U6.1, U6.3
- new net PYRO1_ON: R17.1, R19.1
- new net PYRO2_ON: R1.1, R18.1
- net !RST: no longer U$29.7
- net 3.3V: now also R12.2; no longer U$29.1, U$29.24, U$29.36, U$29.48, U$29.9, U6.1, U6.3
- net ARM_SENSE: no longer U$29.17
- net DBG_RX: no longer U$29.13
- net DBG_TX: no longer U$29.12
- net GND: no longer U$29.23, U$29.35, U$29.44, U$29.47, U$29.8
- net GPS_RXD: no longer U$29.43
- net GPS_TXD: no longer U$29.42
- net MISO: no longer U$29.40
- net MOSI: no longer U$29.41
- net PYRO1_SENSE: no longer U$29.15
- net PYRO2_SENSE: no longer U$29.14
- net RFM_DIO0: no longer U$29.20
- net SCK: no longer U$29.39
- net SCL: no longer U$29.45
- net SDA: no longer U$29.46
- net SWCLK: no longer U$29.37
- net SWDIO: no longer U$29.34
- net USB_DM: now also U9.44; no longer U$29.32
- net USB_DP: now also U9.45; no longer U$29.33
- net VCC_PYRO: now also U6.5; no longer R12.2
- net V_BATT_SENSE: no longer U$29.10
- net V_PYRO_SENSE: no longer U$29.11
Routing:
- net 3.3V: track 56.5 -> 24.4 mm
- net GND: track 18.5 -> 2.19 mm, vias 10 -> 5
- net SDA: track 16.1 -> 3.25 mm, vias 3 -> 2
- net SCL: track 12.2 -> 3.53 mm, vias 2 -> 1
- net PYRO2_SENSE: track 7.66 -> 0.00 mm, vias 1 -> 0
- net D_PYRO1: track 6.24 -> 0.00 mm, vias 1 -> 0
- net N$29: track 3.82 -> 0.00 mm, vias 1 -> 0
- net PYRO1_SENSE: track 3.40 -> 0.00 mm
- net SAFE: track 3.36 -> 0.00 mm, vias 2 -> 0
- net N$17: track 3.36 -> 0.00 mm, vias 1 -> 0
- net PYRO1_OUT: track 2.60 -> 0.00 mm
- net PYRO2_OUT: track 2.57 -> 0.00 mm
- net N$25: track 2.17 -> 0.00 mm
- net N$20: track 2.17 -> 0.00 mm
- net ARM_SENSE: track 1.36 -> 0.00 mm
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Other:
- board size 100 x 80 mm -> 92 x 80 mm

Commit message: Updates
Parts:
- added SV1: (no value), con-ml:ML6
- X2, X3, X5: device kg-conn-rf:SMA_EDGELAUNCH -> kg-conn-rf:SMA90_DIP
- moved C19 38.8 mm to (85.5, 75.0)
- moved R27 38.8 mm to (85.5, 73.5)
- moved R56 38.8 mm to (85.5, 76.5)
- moved C6 9.92 mm to (46.5, 52.5)
- moved FB1 9.92 mm to (44.0, 52.5)
- moved C18 7.76 mm to (13.0, 35.0), flipped to the top
- moved X5 6.16 mm to (13.0, 45.6), turned to 60 degrees
- moved X3 5.22 mm to (87.2, 45.6), turned to 300 degrees
- moved X2 5.00 mm to (50.0, 75.0), turned to 0 degrees
- moved X4 4.30 mm to (75.0, 42.5)
- moved C7 3.35 mm to (26.7, 55.9)
- moved J5 3.35 mm to (34.6, 60.9)
- moved R14 3.35 mm to (28.0, 55.1)
- moved U3 3.35 mm to (26.3, 56.1)
- moved R51 3.35 mm to (32.0, 63.6)
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Connections:
- net GND: now also X2.GND1, X2.GND2, X2.GND3, X2.GND4, X3.GND1, X3.GND2, X3.GND3, X3.GND4, X5.GND1, X5.GND2, X5.GND3, X5.GND4; no longer X2.GND@1, X2.GND@2, X2.GND@3, X2.GND@4, X3.GND@1, X3.GND@2, X3.GND@3, X3.GND@4, X5.GND@1, X5.GND@2, X5.GND@3, X5.GND@4
- net N$26: now also X5.ANTENNA; no longer X5.P
- net N$31: now also X2.ANTENNA; no longer X2.P
- net N$5: now also X3.ANTENNA; no longer X3.P
