File: eagle/tracker/tracker-balloon-full.brd (EAGLE design)
At the start: 104 x 90 mm, 141 parts, among them J1 BATT, J10 AUX3, J13 INTERN, J14 THERMO, J15 EXTERN, J2 USB_MINI-B_SMT, J3 BATT AUX, J4 SWD, J5 MICRO-SD_CARD_SOCKET, J6 UART, J7 BATT GSM, J8 AUX1, J9 AUX2, M1 UBLOX-NEO-M8, M2 HOPE-RFM98W, M3 SIM800L-MODULE, M4 UBLOX-MAX-M8, U1 MS5637-02, U3 A25L010A, U4 MAG3110FCR1, U5 LSM6DS33, U7 MCP73831, U8 MCP73831, U9 STM32L072R, X4 ANTENNA-PATCH-12X12

Commit message: Added standalone GSM tracker
Parts:
- moved JP3 11.5 mm to (70.1, 39.1)
- moved JP4 11.5 mm to (68.1, 35.6)
- moved JP6 11.5 mm to (66.1, 32.1)
- moved R39 11.5 mm to (66.4, 44.7)
- moved R40 11.5 mm to (64.7, 41.6)
- moved R41 11.5 mm to (62.9, 38.6)
- moved SV1 11.5 mm to (79.5, 31.5)
- moved JP2 11.5 mm to (72.1, 42.5)
- moved R42 11.5 mm to (61.2, 35.1)
- moved R15 8.78 mm to (70.9, 76.3), turned to 210 degrees
- moved FB3 7.47 mm to (57.6, 74.4), turned to 150 degrees
- moved X4 6.90 mm to (80.4, 56.8), turned to 30 degrees
- moved M4 6.12 mm to (70.5, 70.6), turned to 60 degrees
- moved X2 6.00 mm to (42.0, 85.0)
- moved M1 5.19 mm to (67.5, 70.3), turned to 300 degrees
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