File: eagle/tracker/tracker-uno-v1.brd (EAGLE design)
At the start: 74 x 74 mm, 80 parts, among them J1 BATT, J2 USB_MINI-B_SMT, J3 BATT_PYRO, J5 MICRO-SD_CARD_SOCKET, M1 UBLOX-NEO-M8, M2 HOPE-RFM98W, M3 SIM800L-MODULE, M4 UBLOX-MAX-M8, U1 MS5637-02, U3 A25L010A, U4 MAG3110FCR1, U5 LSM6DS33, U7 MCP73831, X1 87758-0416, X2A COAX, X2B COAX, X4 MICROMATCH-8, X6 COAX

Commit message: Updates to tracker
Parts:
- removed D1, D2: (no value), kg-generic:R0805
- removed J1: BATT, kg-amp-ct:JST-2-PTH-VERT
- removed J2: USB_MINI-B_SMT, SparkFun-Connectors:USB-MINIB
- removed J3: BATT_PYRO, kg-amp-ct:JST-2-PTH-VERT
- removed J4: (no value), kg-amp-ct:JST-4-PTH-VERT
- removed J5: MICRO-SD_CARD_SOCKET, SparkFun-Connectors:MICRO-SD-SOCKET
- removed J6: (no value), kg-amp-ct:JST-3-PTH-VERT
- removed JP5: LDO_BYPASS, SparkFun-Passives:PAD-JUMPER-2-NO_YES_SILK
- removed L1A, L1B: (no value), kg-generic:R0603
- removed M3: SIM800L-MODULE, kg-modules:SIM800L
- removed M4: UBLOX-MAX-M8, kg-modules:UBLOX-MAX
- removed PAD1, PAD2: (no value), wirepad:SMD2,54-5,08
- removed R15: 3.3k, rcl:R0603
- removed R16, R17, R18, R21, R22, R23, R24, R25: 100k, kg-generic:R0603
- removed R19, R26, R27: 1k, kg-generic:R0603
- removed R20: 10k, kg-generic:R0603
- removed SG1: F/TMB, buzzer:F/TMB
- removed U$29: STM32L063C, kg-mcu:LQFP48
- removed U5: LSM6DS33, kg-ic:TFLGA16L
- removed U7: MCP73831, kg-supply:SOT23-5
- removed X2A, X2B, X6: COAX, kg-conn-rf:MMCX-J-P-X-ST-EM1-MKT
- added B1: ARDUINO_UNO_R3, SparkFun-Boards:ARDUINO_R3
- added C0: 10p/330p/68p, microbuilder_v3:_0603MP
- added C16, C17, C18, C19, C20: (no value), kg-generic:C603
- added C21: 2u2, microbuilder_v3:_0603MP
- added CM: 10p/27p/68p, microbuilder_v3:_0603MP
- added CM1, CM2: 15p/47p/150p, microbuilder_v3:_0603MP
- added CM3, CM4: 8p2/27p/NF, microbuilder_v3:_0603MP
- added ESD1: NF, microbuilder_v3:_0603MP
- added ESD2, ESD3: 0.25p, microbuilder_v3:_0603MP
- added FB2, FB4, FB5: (no value), microbuilder_v3:_0805
- added JP4: JUMPER-PAD-2-NOYES_SILK, SparkFun-Passives:PAD-JUMPER-2-NO_YES_SILK
- added JP6: PROG, pinhead:1X04
- added JP9: (no value), pinhead:1X08
- added L0: 56n/100n/3.9u, microbuilder_v3:_0805MP
- added LED1, LED4: (no value), led:CHIPLED_0805
- added LM, LM1: 18n/68n/1.5u, microbuilder_v3:_0805MP
- added LM2, LM3: 18n/68n/330n, microbuilder_v3:_0805MP
- added LR1, LR3: 220n/470n, microbuilder_v3:_0805MP
- added S1: MOMENTARY-SWITCH-SPST-SMD-6.2MM-TALL, SparkFun-Switches:TACTILE_SWITCH_SMD_6.2MM_TALL
- added TP10, TP11, TP3: TPSB1,27, testpad:B1,27
- added U$42: MINI-USB-B, kg-sdrlib:MINI-B-USB
- added U8: STM32L052C8, kg-mcu:LQFP48
- added X2, X3: (no value), kg-conn-rf:SMA_EDGELAUNCH
- added XO1: 26.000MHz TCXO, kg-crystal:CRYSTAL-SMD-2.5X2
- C1, C13: value 100n -> 10n; device kg-generic:C603 -> microbuilder_v3:_0603MP
- C10, C6, C7, C9: value 100n -> (none)
- C11, C5: value 1u -> 100n; device kg-generic:C603 -> microbuilder_v3:_0603MP
- C12: device rcl:E3,5-8 -> kg-generic:C603
- C14, C15: device kg-generic:C603 -> microbuilder_v3:_0603MP
- C2: value 10u -> (none); device kg-generic:EIA3216 -> kg-generic:C603
- C3: value 100n -> 0R; device kg-generic:C603 -> microbuilder_v3:_0603MP
- C4: value 1u -> NF/8p2/NF; device kg-generic:C603 -> microbuilder_v3:_0603MP
- C8: value 1u -> 2n2; device kg-generic:C603 -> microbuilder_v3:_0603MP
- JP1: value BYPASS2 -> BATT; device SparkFun-Passives:PAD-JUMPER-2-NO_YES_SILK -> pinhead:1X02
- M1: value UBLOX-NEO-M8 -> UBLOX-NEO-6; device kg-modules:UBLOX-NEO -> kg-modules:UBLOX-NEO-6
- Q3, Q4: value (none) -> NTR5103N
- R1: value 1k -> 10k; device kg-generic:R0603 -> rcl:R0603
- R10, R11, R13, R5: value 100k -> (none)
- R12: value 100 -> 470; device kg-generic:R0603 -> rcl:R0603
- R14: value 10k -> (none)
- R2: value 10k -> 100k; device kg-generic:R0603 -> rcl:R0603
- R6, R7: value 1k -> (none)
- R8: value 3.3k -> (none); device rcl:R0603 -> kg-generic:R0603
- R9: value (none) -> 10k; device kg-generic:R0603 -> rcl:R0603
- U1: value MS5637-02 -> SI446X; device kg-ic:MS5637 -> kg-sdrlib:QFN20
- U2: value (none) -> MCP73831; device kg-generic:SOT23-5 -> kg-supply:SOT23-5
- U4: value MAG3110FCR1 -> (none); device kg-ic:DFN200X200X90-10N -> kg-generic:SOT23-3
- U6: value (none) -> SI5351A; device kg-generic:SOT23-5 -> kg-sdrlib:MSOP10
- X1: value 87758-0416 -> 32.768kHz; device con-molex:87758-0416 -> IQD-Frequency-Products:3.2X1.5-2-PAD
- X4: value MICROMATCH-8 -> (none); device con-amp-micromatch:MICROMATCH-8 -> kg-conn-rf:SMA_EDGELAUNCH
- moved X4 82.3 mm to (90.5, 56.5), turned to 0 degrees
- moved C7 69.1 mm to (17.5, 26.5), flipped to the top
- moved R6 65.8 mm to (13.5, 6.00)
- moved M1 65.6 mm to (19.0, 65.0), turned to 90 degrees
- moved C3 60.6 mm to (6.50, 64.5), turned to 270 degrees
- moved U2 59.6 mm to (32.5, 8.00), flipped to the top
- moved JP1 59.0 mm to (36.5, 3.50), turned to 180 degrees
- moved R10 57.4 mm to (42.0, 7.50), turned to 0 degrees
- moved C9 56.9 mm to (74.5, 69.5), flipped to the top, turned to 90 degrees
- moved R13 55.1 mm to (42.0, 3.50), turned to 180 degrees
- moved Q2 52.1 mm to (66.5, 68.0), turned to 90 degrees
- moved C8 51.3 mm to (19.0, 26.5), turned to 270 degrees
- moved R5 50.7 mm to (13.5, 8.00), flipped to the top
- moved C6 48.0 mm to (9.50, 30.5), turned to 90 degrees
- moved R12 46.2 mm to (42.2, 18.8), flipped to the top, turned to 180 degrees
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Connections:
- net !RFM_RST renamed !LORA_RST
- net !RFM_SS renamed !LORA_CS
- removed net 3.3V: C15.2, C2.A, C3.2, C5.2, C7.2, FB1.2, FB3.1, JP5.2, R14.2, R3.2, R4.2, R5.1, R9.2, U$29.1, U$29.24, U$29.36, U$29.48, U$29.9, U1.1, U2.5, U3.3, U3.7, U3.8, U4.2, U4.8, U5.1, U5.16, U5.4, U5.5, U6.1, U6.3
- removed net BUZZER: R7.1
- removed net CMD1: R17.1, R19.1, U$29.19
- removed net CMD2: R1.1, R18.1, U$29.18
- removed net GPS_VCC: C9.2, FB3.2, M1.2, M1.23, M4.7, M4.8, R15.2
- removed net PYRO1_OUT: Q2.3, R21.1, X4.4
- removed net PYRO2_OUT: Q3.3, R22.1, X4.2
- removed net PYRO_SENSE: R16.2, R23.2, U$29.11
- removed net RFM_DIO0: M2.14, U$29.20
- removed net SAFE: R20.2, X4.6
- removed net SENSE1: R21.2, R24.2, U$29.15
- removed net SENSE2: R22.2, R25.2, U$29.14
- removed net SENSE_ARM: R26.2, U$29.17
- removed net SHDN: R10.1, U2.3, X4.8
- removed net VCC_PYRO: C12.+, J3.2, JP1.2, R12.2, R16.1, X4.1, X4.3
- removed net V_BATT: C4.2, D2.1, J1.2, JP1.1, JP5.1, PAD1.1, R10.2, R11.2, SG1.+, U2.1
- removed net V_BATT_SENSE: C10.2, R11.1, R13.2, U$29.10
- removed net V_USB: J2.VBUS, U7.4
- new net !GPS_ON: Q2.1, R14.1
- new net !LORA_IRQ: M2.14
- new net !RADIO_ON: Q1.1, R1.1
- new net !TFT_CS: JP9.6
- new net !TFT_LED: JP9.8
- new net !TFT_RST: JP9.7
- new net !TRX_CS: U1.15
- new net !TRX_EN: U1.1
- new net !TRX_IRQ: U1.11
- new net +3V3: C2.2, C5.1, M1.22, Q1.2, Q2.2, R1.2, R14.2, R3.2, R4.2, R9.2, U3.8, U4.2, U8.1, U8.24, U8.36, U8.48, U8.9
- new net 3V3_RADIO: C11.1, C12.2, C21.1, C7.2, C8.1, FB1.1, FB1.2, FB3.1, FB4.2, LR3.2, Q1.3, R11.1, U1.6, XO1.4
- new net CHG_STATUS: LED1.C, U2.1
- new net N$18: C18.2, JP1.2, R13.2, U2.3, U4.3
- new net N$26: FB5.2, U$42.1
- new net N$28: C10.2, FB4.1, M2.13
- new net N$30: JP9.2
- new net N$32: CM2.1, LM.1, LM2.2
- new net N$33: R6.1, U$42.3
- new net N$34: C9.2, FB2.2, M1.23
- new net N$35: LED4.C, R12.2
- new net N$36: C16.2, LR1.1, Q3.3, Q4.3
- new net N$37: C6.2, M2.9
- new net RADIO_XIN: C13.2, U1.17
- new net RF_TANK: CM.1, L0.1, LM.2
- new net RF_TANK1: C16.1, LM1.2
- new net SHLD$1: U$42.SHLD$1
- new net SHLD$2: U$42.SHLD$2
- new net SHLD$3: U$42.SHLD$3
- new net SHLD$4: U$42.SHLD$4
- new net TCXO_OUT: C1.1, C13.1, XO1.3
- new net TFT_RS: JP9.5
- new net TRX_GPIO0: U1.9
- new net TRX_GPIO1: U1.10
- new net TRX_GPIO2: TP11.TP, U1.19
- new net TRX_GPIO3: TP10.TP, U1.20
- new net USB_DM: R5.2, U8.32
- new net USB_DP: R6.2, U8.33
- new net USB_VBUS: C19.2, FB5.1, R8.2, U2.4
- new net VBAT_ADC: C17.2, R10.2, R13.1
- net !FLASH_CS: no longer R14.1
- net !RST: now also C14.1, JP6.4, U8.7; no longer C1.2, J4.2, U$29.7
- net DBG_RX: now also U8.31; no longer J6.2, U$29.13
- net DBG_TX: now also U8.30; no longer J6.3, U$29.12
- net GND: now also C11.2, C12.1, C14.2, C15.2, C17.1, C18.1, C19.1, C2.1, C20.1, C21.2, C4.2, C5.2, C8.2, CM.2, CM1.2, CM2.2, CM3.2, CM4.2, ESD1.1, ESD2.1, ESD3.1, JP1.1, JP4.2, JP6.1, JP9.1, Q3.2, R10.1, R12.1, R7.1, U$42.5, U1.18, U1.5, U1.PAD, U4.1, U6.8, U8.23, U8.35, U8.44, U8.47, U8.8, X2.GND@1, X2.GND@2, X2.GND@3, X2.GND@4, X3.GND@1, X3.GND@2, X3.GND@3, X3.GND@4, X4.GND@1, X4.GND@2, X4.GND@3, X4.GND@4, XO1.2; no longer C1.1, C11.1, C12.-, C13.1, C14.1, C15.1, C2.C, C3.1, C4.1, C5.1, C6.1, C8.1, D1.2, J1.1, J2.GND, J3.1, J4.1, J6.1, L1A.1, L1B.1, M1.22, M4.1, M4.10, M4.12, M4.6, Q1.2, R13.1, R17.2, R18.2, R23.1, R24.1, R25.1, U$29.23, U$29.35, U$29.44, U$29.47, U$29.8, U1.4, U4.10, U4.5, U5.10, U5.11, U5.12, U5.13, U5.15, U5.8, U5.9, U6.2, X2A.2@1, X2A.2@2, X2A.2@3, X2A.2@4, X2B.2@1, X2B.2@2, X2B.2@3, X2B.2@4, X4.5, X4.7, X6.2@1, X6.2@2, X6.2@3, X6.2@4
- net GPS_PPS: now also TP3.TP, U8.2; no longer M4.4
- net GPS_RXD: now also U8.22; no longer M4.2, U$29.43
- net GPS_TXD: now also U8.21; no longer M4.3, U$29.42
- net LED: now also LED4.A; no longer R6.2
- net MISO: now also U1.13, U8.16; no longer J5.DO, U$29.40
- net MOSI: now also JP9.3, U1.14, U8.17; no longer J5.DI, U$29.41
- net N$12: now also C0.2, LR3.1, U1.4; no longer PAD2.1, Q1.3, R27.1, SG1.-
- net N$13: now also FB2.1, Q2.3; no longer C6.2, FB1.1, M2.13
- net N$14: now also R7.2, U2.5; no longer M1.8, R8.1
- net N$15: now also C0.1, C4.1, L0.2; no longer M1.9, R8.2
- net N$16: now also C3.2, M1.11; no longer C8.2, U2.4
- net N$17: now also JP4.1, M1.14; no longer Q2.2, Q3.2, Q4.3
- net N$19: now also C3.1, ESD1.2, X3.P; no longer D1.1, R6.1
- net N$20: now also C20.2, FB3.2, LR1.2, U6.1, U6.7; no longer Q2.1, R19.2
- net N$21: now also U8.3, X1.2; no longer C11.2, R12.1, U6.5
- net N$22: now also C15.1, R11.2, U1.8; no longer C13.2, U4.1
- net N$23: now also C1.2, U6.2; no longer C14.2, U4.4
- net N$24: now also CM4.1, ESD3.2, LM3.1, X4.P; no longer M4.9, R15.1
- net N$25: now also CM1.1, LM1.1, LM3.2; no longer Q3.1, R1.2
- net N$27: now also U8.4, X1.1; no longer U7.3
- net N$29: now also R5.1, U$42.2; no longer Q4.1, R20.1, R26.1, R5.2
- net N$31: now also C6.1, CM3.1, ESD2.2, LM2.1, X2.P; no longer M2.9, X6.1
- net N$5: now also Q3.1, Q4.1, R2.2, U6.10; no longer L1A.2, L1B.2, M1.11, M4.11, X2A.1, X2B.1
- net N$8: now also M1.8, M1.9; no longer D2.2, R27.2
- net N$9: now also LED1.A, R8.1; no longer Q1.1, R2.2, R7.2
- net SCK: now also JP9.4, U1.12, U8.15; no longer J5.SCLK, U$29.39
- net SCL: now also U6.4, U8.42; no longer U$29.45, U1.3, U4.7, U5.2
- net SDA: now also U6.5, U8.43; no longer U$29.46, U1.2, U4.6, U5.3
- net SWCLK: now also JP6.3, U8.37; no longer J4.3, U$29.37
- net SWDIO: now also JP6.2, U8.34; no longer J4.4, U$29.34
Routing:
- net 3.3V: track 62.5 -> 0.00 mm, vias 6 -> 0
- net +3V3: track 0.00 -> 43.0 mm, vias 0 -> 3
- net MISO: track 0.00 -> 37.9 mm, vias 0 -> 3
- net MOSI: track 0.00 -> 31.5 mm, vias 0 -> 2
- net SCK: track 0.00 -> 29.5 mm, vias 0 -> 3
- net GPS_VCC: track 27.6 -> 0.00 mm, vias 3 -> 0
- net V_BATT: track 25.5 -> 0.00 mm, vias 1 -> 0
- net SDA: track 16.1 -> 2.46 mm, vias 3 -> 0
- net !RST: track 0.00 -> 12.5 mm, vias 0 -> 2
- net 3V3_RADIO: track 0.00 -> 9.87 mm
- net GND: track 18.5 -> 8.91 mm, vias 11 -> 30
- net SCL: track 12.2 -> 4.27 mm, vias 2 -> 0
- net SENSE2: track 7.66 -> 0.00 mm, vias 1 -> 0
- net N$31: track 0.00 -> 7.43 mm
- net !FLASH_CS: track 1.98 -> 9.03 mm, vias 1 -> 2
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Other:
- board size 74 x 74 mm -> 99.5 x 75.5 mm
- board text added: "Ant"
- board text added: "BKP"
- board text added: "Bat"
- board text added: "CFG0"
- board text added: "Chg"
- board text added: "Dbg"
- board text added: "Ext"
- board text added: "TReX"
- board text added: "v1.1"
- board text removed: "LoRa"
- board text removed: "TODO: - TABS for battery straps"
