File: eagle/tracker/tracker-25mm.sch (EAGLE design)
At the start: 45 parts, among them J1 BATT, J2 SHDN, M1 UBLOX-NEO-M8, M2 HOPE-RFM98W, U1 MS5637-02, U3 A25L010A, X1 MICROMATCH-4, X5 B3710U410

Commit message: Tracker ready for order
Parts:
- removed X5: B3710U410, kg-radio:B3710U410
- added L1: (no value), kg-generic:L-0805
- added M3: UBLOX-MAX-M8, kg-modules:UBLOX-MAX-M8
- added R12, R15, R16, R17, R18, R19, R20: (no value), kg-generic:RESISTOR-0603
- D2: device kg-generic:DIODE-SCHOTTKY-SOD323 -> kg-generic:LED0805
- J1, J2: device kg-amp-ct:M2-CT-V -> kg-amp-ct:M2-2MM-JST
- R1: value (none) -> 3.3k; device kg-generic:RESISTOR-0603 -> rcl:R-EU_R0603
Connections:
- removed net BUS: R5.2, X1-2.S
- removed net CMD1: U$29.PA11, X1-3.S
- removed net CMD2: U$29.PA12, X1-4.S
- removed net LED: R6.2, U$29.PA15
- new net LED1: R6.2, U$29.PA12
- new net LED2: R15.2, U$29.PA11
- new net N$20: R12.2, X1-3.S
- new net N$21: R5.2, X1-4.S
- new net N$22: D2.A, R15.1
- new net N$23: R18.2, U$29.PA2
- new net N$24: R16.2, X1-2.S
- new net N$25: R19.2, U$29.PA3
- net !FLASH_CS: now also U$29.PB12; no longer U$29.PA8
- net 3.3V: now also R17.2, R20.2; no longer R1.2
- net DBG_RX: now also R12.1, R20.1, U$29.PB7; no longer D2.A, R1.1, R5.1, U$29.PA10
- net DBG_TX: now also R17.1, R5.1, U$29.PB6; no longer D2.C, U$29.PA9
- net GND: now also D2.C, L1.1, M3.GND, M3.V_BCKP; no longer X5.1, X5.3, X5.4, X5.6
- net GPS_PPS: now also M3.TIMEPULSE, R16.1
- net GPS_RXD: now also M3.TXD, R19.1; no longer U$29.PA3
- net GPS_TXD: now also M3.RXD, R18.1; no longer U$29.PA2
- net GPS_VCC: now also M3.VCC, M3.VCC_IO, R1.2
- net N$5: now also L1.2, M1.RF_IN, M3.RF_IN; no longer X5.2
- net N$8: now also M3.!RESET, R1.1; no longer M1.RF_IN, X5.5
- net SCL: now also U$29.PB13; no longer U$29.PB6
- net SDA: now also U$29.PB14; no longer U$29.PB7
Other:
- note added: "TODO:"
- note removed: "TODO: - SAW filter for GPS - NEO 6/7/8 compatibility - Buzzer package - VBat sensing"
- moved on the sheet: C5, C8, D1, R10, R5, R6
