File: eagle/tracker/tracker-balloon-full.sch (EAGLE design)
At the start: 75 parts, among them J1 BATT, J2 USB_MINI-B_SMT, J3 BATT_PYRO, M1 UBLOX-NEO-M8, M2 HOPE-RFM98W, M4 UBLOX-MAX-M8, U1 MS5637-02, U3 A25L010A, U4 MAG3110FCR1, U5 LSM6DS33, X1 87758-0416, X2A COAX, X2B COAX, X4 MICROMATCH-8, X6 COAX

Commit message: Updates to tracker
Parts:
- added D2: (no value), kg-generic:LED0805
- added J5: MICRO-SD_CARD_SOCKET, SparkFun-Connectors:MICRO-SD_CARD_SOCKET
- added M3: SIM800L-MODULE, kg-modules:SIM800L-MODULE
- added R27: 1k, kg-generic:RESISTOR-0603
- added U7: MCP73831, kg-supply:MCP73831
- R5: value 10k -> 100k
Connections:
- new net N$27: U7.BAT
- new net N$8: D2.C, R27.2
- new net V_USB: J2.VBUS, U7.VDD
- net MISO: now also J5.DO
- net MOSI: now also J5.DI
- net N$12: now also R27.1
- net SCK: now also J5.SCK
- net V_BATT: now also D2.A
Other:
- note added: "TODO: - External buzzer/LED/NTC connector - GPIO header w/ rich periph (AN/UART/I2C/SPI) - Separate I2C connector - Dallas 3pin connector - Servo 3pin connectors - Dev area? - 2-3 extra mosfet switches - Single batt. option with cutoff/fuse - SD card w/ separate SPI bus?"
- note removed: "TODO: - SAW filter for GPS - NEO 6/7/8 compatibility - Buzzer package - VBat sensing"
Changed lines of the file:
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@@
 <part name="Q3" library="kg-generic" deviceset="MOSFET-N" device="-SOT23-3"/>
 <part name="R1" library="kg-generic" deviceset="RESISTOR" device="-0603" value="1k"/>
-<part name="R5" library="kg-generic" deviceset="RESISTOR" device="-0603" value="10k"/>
+<part name="R5" library="kg-generic" deviceset="RESISTOR" device="-0603" value="100k"/>
 <part name="M4" library="kg-modules" deviceset="UBLOX-MAX-M8" device=""/>
 <part name="U$26" library="kg-generic" deviceset="GND" device=""/>
@@
 <part name="L1B" library="kg-generic" deviceset="L" device="-0603"/>
 <part name="U$24" library="kg-generic" deviceset="GND" device=""/>
+<part name="U7" library="kg-supply" deviceset="MCP73831" device=""/>
+<part name="D2" library="kg-generic" deviceset="LED" device="0805"/>
+<part name="R27" library="kg-generic" deviceset="RESISTOR" device="-0603" value="1k"/>
+<part name="FRAME5" library="SparkFun-Aesthetics" deviceset="FRAME-A4L" device=""/>
+<part name="J5" library="SparkFun-Connectors" deviceset="MICRO-SD_CARD_SOCKET" device=""/>
+<part name="M3" library="kg-modules" deviceset="SIM800L-MODULE" device=""/>
 </parts>
 <sheets>
@@
 <plain>
 <text x="558.8" y="-106.68" size="3.81" layer="90" font="vector" ratio="12" align="top-left">TODO:
-- SAW filter for GPS
-- NEO 6/7/8 compatibility
-- Buzzer package
-- VBat sensing</text>
+- External buzzer/LED/NTC connector
+- GPIO header w/ rich periph (AN/UART/I2C/SPI)
+- Separate I2C connector
+- Dallas 3pin connector
+- Servo 3pin connectors
+- Dev area?
+- 2-3 extra mosfet switches
+- Single batt. option with cutoff/fuse
+- SD card w/ separate SPI bus?</text>
 <text x="335.28" y="58.42" size="1.27" layer="97">75uA in Inactive State
 15uA Backup battery current</text>
@@
 <instance part="L1B" gate="G$1" x="269.24" y="35.56" rot="R90"/>
 <instance part="U$24" gate="G$1" x="271.78" y="25.4"/>
+<instance part="U7" gate="G$1" x="353.06" y="-162.56"/>
+<instance part="D2" gate="G$1" x="728.98" y="73.66"/>
+<instance part="R27" gate="G$1" x="723.9" y="60.96"/>
+<instance part="FRAME5" gate="G$1" x="236.22" y="-373.38"/>
+<instance part="J5" gate="1" x="558.8" y="48.26"/>
+<instance part="M3" gate="G$1" x="454.66" y="132.08"/>
 </instances>
 <busses>
@@
 <wire x1="561.34" y1="132.08" x2="568.96" y2="132.08" width="0.1524" layer="91"/>
 </segment>
+<segment>
+<pinref part="J5" gate="1" pin="SCK"/>
+<wire x1="543.56" y1="45.72" x2="538.48" y2="45.72" width="0.1524" layer="91"/>
+<label x="538.48" y="45.72" size="1.27" layer="95" rot="R180" xref="yes"/>
+</segment>
 </net>
 <net name="MISO" class="0">
@@
 <wire x1="561.34" y1="129.54" x2="568.96" y2="129.54" width="0.1524" layer="91"/>
 </segment>
+<segment>
+<pinref part="J5" gate="1" pin="DO"/>
+<wire x1="543.56" y1="43.18" x2="538.48" y2="43.18" width="0.1524" layer="91"/>
+<label x="538.48" y="43.18" size="1.27" layer="95" rot="R180" xref="yes"/>
+</segment>
 </net>
 <net name="MOSI" class="0">
@@
 <pinref part="U$29" gate="G$1" pin="PB5"/>
 <wire x1="561.34" y1="127" x2="568.96" y2="127" width="0.1524" layer="91"/>
+</segment>
+<segment>
+<pinref part="J5" gate="1" pin="DI"/>
+<wire x1="543.56" y1="48.26" x2="538.48" y2="48.26" width="0.1524" layer="91"/>
+<label x="538.48" y="48.26" size="1.27" layer="95" rot="R180" xref="yes"/>
 </segment>
 </net>
@@
 <wire x1="706.12" y1="73.66" x2="711.2" y2="73.66" width="0.1524" layer="91"/>
 <junction x="711.2" y="73.66"/>
+<pinref part="D2" gate="G$1" pin="A"/>
+<wire x1="711.2" y1="73.66" x2="726.44" y2="73.66" width="0.1524" layer="91"/>
 </segment>
 <segment>
@@
 <wire x1="706.12" y1="60.96" x2="711.2" y2="60.96" width="0.1524" layer="91"/>
 <junction x="711.2" y="60.96"/>
+<pinref part="R27" gate="G$1" pin="1"/>
+<wire x1="723.9" y1="60.96" x2="711.2" y2="60.96" width="0.1524" layer="91"/>
 </segment>
 </net>
@@
 </segment>
 </net>
+<net name="V_USB" class="0">
+<segment>
+<label x="736.6" y="48.26" size="1.27" layer="95" rot="R180" xref="yes"/>
+<pinref part="J2" gate="G$1" pin="VBUS"/>
+<wire x1="762" y1="48.26" x2="736.6" y2="48.26" width="0.1524" layer="91"/>
+</segment>
+<segment>
+<pinref part="U7" gate="G$1" pin="VDD"/>
+<wire x1="342.9" y1="-160.02" x2="332.74" y2="-160.02" width="0.1524" layer="91"/>
+<label x="332.74" y="-160.02" size="1.27" layer="95" rot="R180" xref="yes"/>
+</segment>
+</net>
+<net name="N$27" class="0">
+<segment>
+<pinref part="U7" gate="G$1" pin="BAT"/>
+<wire x1="363.22" y1="-160.02" x2="368.3" y2="-160.02" width="0.1524" layer="91"/>
+</segment>
+</net>
+<net name="N$8" class="0">
+<segment>
+<pinref part="D2" gate="G$1" pin="C"/>
+<wire x1="731.52" y1="73.66" x2="734.06" y2="73.66" width="0.1524" layer="91"/>
+<wire x1="734.06" y1="73.66" x2="734.06" y2="60.96" width="0.1524" layer="91"/>
+<pinref part="R27" gate="G$1" pin="2"/>
+<wire x1="734.06" y1="60.96" x2="731.52" y2="60.96" width="0.1524" layer="91"/>
+</segment>
+</net>

Commit message: Updates to balloon flight board
Parts:
- removed L1B: (no value), kg-generic:L-0603
- removed X2A, X2B: COAX, kg-conn-rf:COAX
- added D10, D11, D6, D7, D8, D9: (no value), kg-generic:LED0805
- added D3, D4, D5: (no value), kg-generic:DIODE-ZENER-SOD323
- added J7: BATT_PYRO, kg-amp-ct:M2-CT-V
- added JP2, JP3, JP4, JP6: (no value), pinhead:PINHD-1X3
- added JP7: (no value), pinhead:PINHD-2X3
- added Q10, Q12, Q7, Q8: (no value), kg-generic:MOSFET-N-SOT23-3
- added Q11, Q5, Q6, Q9: (no value), kg-generic:MOSFET-P-SOT23-3
- added R28, R29, R30, R31, R32, R33, R35, R36, R38, R39, R40, R41, R42, R43, R44, R45: 1k, kg-generic:RESISTOR-0603
- added R34, R37, R46: 100k, kg-generic:RESISTOR-0603
- added R47: (no value), kg-generic:RESISTOR-0603
- added X10, X7, X8, X9: (no value), con-wago-500:W237-102
- added X2, X3, X5: (no value), kg-conn-rf:SMACONNECTOR_EDGE
- R17, R18: value 100k -> 1k
- X1: value 87758-0416 -> (none); device con-molex:87758-0416 -> con-wago-500:W237-102
- X4: value MICROMATCH-8 -> ANTENNA-PATCH-12X12; device con-amp-micromatch:MICROMATCH-8 -> kg-modules:ANTENNA-PATCH-12X12
- X6: value COAX -> (none); device kg-conn-rf:COAX -> con-wago-500:W237-102
Connections:
- new net DO_LOAD1: R32.1, R43.1
- new net DO_LOAD2: R35.1, R44.1
- new net DO_LOAD3: R38.1, R45.1
- new net DO_SRV1: R39.1
- new net DO_SRV2: R40.1
- new net DO_SRV3: R41.1
- new net DO_SRV4: R42.1
- new net N$26: M3.ANT, X5.ANT
- new net N$28: J2.D-, R28.2
- new net N$30: J2.D+, R29.2
- new net N$32: JP6.1, R42.2
- new net N$33: D3.A, Q5.G, R30.1, R34.1
- new net N$34: Q8.D, R30.2
- new net N$35: Q8.G, R32.2
- new net N$36: Q5.D, X8-1.KL
- new net N$37: D6.A, R43.2
- new net N$38: JP4.1, R41.2
- new net N$39: D4.A, Q6.G, R33.1, R37.1
- new net N$40: Q7.D, R33.2
- new net N$41: Q7.G, R35.2
- new net N$42: Q6.D, X9-1.KL
- new net N$43: JP3.1, R40.2
- new net N$44: JP2.1, R39.2
- new net N$45: D5.A, Q9.G, R36.1, R46.1
- new net N$46: Q10.D, R36.2
- new net N$47: Q10.G, R38.2
- new net N$48: Q9.D, X10-1.KL
- new net N$49: D9.A, R17.2
- new net N$50: D8.A, R45.2
- new net N$51: D7.A, R44.2
- new net N$52: D10.A, R18.2
- new net N$53: D11.A, R31.2
- new net N$54: M3.VCC, Q11.D
- new net N$55: Q11.G, Q12.D, R47.1
- new net USB_DM: R28.1, U$29.PA11
- new net USB_DP: R29.1, U$29.PA12
- new net V_GSM: J7.2, Q11.S, R47.2
- new net V_LOAD: D3.C, D4.C, D5.C, Q5.S, Q6.S, Q9.S, R34.2, R37.2, R46.2, X1-1.KL
- new net V_SERVO: JP2.2, JP3.2, JP4.2, JP6.2
- net !FLASH_CS: now also J5.!CS
- net 3.3V: now also J5.VCC, R31.1
- net GND: now also D10.C, D6.C, D7.C, D8.C, D9.C, J5.GND, J5.SHIELD@1, J5.SHIELD@3, J7.1, JP2.3, JP3.3, JP4.3, JP6.3, M3.GND, Q10.S, Q12.S, Q7.S, Q8.S, X1-2.KL, X10-2.KL, X2.GND1, X2.GND2, X2.GND3, X2.GND4, X3.GND1, X3.GND2, X3.GND3, X3.GND4, X5.GND1, X5.GND2, X5.GND3, X5.GND4, X8-2.KL, X9-2.KL; no longer L1B.1, R17.2, R18.2, X2ACOAX.GND, X2BCOAX.GND, X4-5.S, X4-7.S, X6COAX.GND
- net N$17: now also D11.C
- net N$31: now also X2.ANT; no longer X6COAX.1
- net N$5: now also X3.ANT, X4.FEED; no longer L1B.2, X2ACOAX.1, X2BCOAX.1
- net PYRO1_OUT: now also X6-2.KL; no longer X4-4.S
- net PYRO2_OUT: now also X7-2.KL; no longer X4-2.S
- net SAFE: no longer X4-6.S
- net SHDN: no longer X4-8.S
- net VCC_PYRO: now also X6-1.KL, X7-1.KL; no longer X4-1.S, X4-3.S
Other:
- note added: "ARMED"
- note added: "Load switches"
- note added: "P1 ACT"
- note added: "P2 ACT"
- note added: "Servo PWM outputs"
- note added: "TODO: - External buzzer/LED/NTC connector - GPIO header w/ rich periph (AN/UART/I2C/SPI) - Separate I2C connector - Dallas / Servo 3pin connectors - Dev area? - 2-3 mosfet load switches - Single batt. option with cutoff/fuse? - SD card w/ separate SPI bus? - Rich LED indication - GPS backup supercap"
- note removed: "TODO: - External buzzer/LED/NTC connector - GPIO header w/ rich periph (AN/UART/I2C/SPI) - Separate I2C connector - Dallas 3pin connector - Servo 3pin connectors - Dev area? - 2-3 extra mosfet switches - Single batt. option with cutoff/fuse - SD card w/ separate SPI bus?"
- moved on the sheet: C13, C14, C15, C8, C9, D1, D2, FB3, J2, L1A, PAD1, PAD2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

Commit message: Tracker ready for order
Parts:
- removed D2: (no value), kg-generic:LED0805
- removed JP1: BYPASS2, SparkFun-Passives:JUMPER-PAD-2-NOYES_SILK
- removed JP5: LDO_BYPASS, SparkFun-Passives:JUMPER-PAD-2-NOYES_SILK
- removed JP7: (no value), pinhead:PINHD-2X3
- removed PAD1, PAD2: (no value), wirepad:SMD5
- removed SG1: F/TMB, buzzer:F/TMB
- removed X1, X10, X6, X7, X8, X9: (no value), con-wago-500:W237-102
- added C16, C17, C18: 1u, kg-generic:CAPACITOR_NPOL-0603
- added C19: 100n, kg-generic:CAPACITOR_NPOL-0603
- added D12, D13, D14: (no value), kg-generic:LED0805
- added J10, J11, J12, J8, J9: (no value), kg-amp-ct:M2-3.81MM
- added J14: 1WIRE, kg-amp-ct:M3-CT-V
- added R48, R50, R52, R53, R54, R55, R56: 1k, kg-generic:RESISTOR-0603
- added R49: 100k, kg-generic:RESISTOR-0603
- added R51: 10k, kg-generic:RESISTOR-0603
- added R57: 100, kg-generic:RESISTOR-0603
- added SV1: PANEL, con-ml:ML6
- added SV2: I2C/GPS, con-ml:ML6
- added U8: MCP73831, kg-supply:MCP73831
- C1: value 100n -> 10n
- J1: device kg-amp-ct:M2-CT-V -> kg-amp-ct:M2-2MM-JST
- J3: value BATT_PYRO -> (none); device kg-amp-ct:M2-CT-V -> kg-amp-ct:M2-3.81MM
- J7: value BATT_PYRO -> BATT_GSM; device kg-amp-ct:M2-CT-V -> kg-amp-ct:M2-2MM-JST
- R27: value 1k -> 100k
- R47: value (none) -> 100k
- R9: value (none) -> 10k
Connections:
- net CMD1 renamed D_PYRO1
- net CMD2 renamed D_PYRO2
- net DO_LOAD1 renamed D_LOAD1
- net DO_LOAD2 renamed D_LOAD2
- net DO_LOAD3 renamed D_LOAD3
- net PYRO_SENSE renamed V_PYRO_SENSE
- net SENSE1 renamed PYRO1_SENSE
- net SENSE2 renamed PYRO2_SENSE
- net SENSE_ARM renamed ARM_SENSE
- removed net BUZZER: R7.1
- removed net N$8: D2.C, R27.2
- new net !GSM_RST: M3.!RST
- new net D_BUZZER: R2.2, R7.1
- new net GSM_ON: R48.1, R49.2
- new net GSM_RXD: M3.TXD
- new net GSM_TXD: M3.RXD
- new net N$57: M3.DTR, R51.2
- new net N$58: D13.A, R52.2
- new net N$59: D14.A, R53.2
- new net N$60: D14.C, U7.STAT
- new net N$61: D13.C, U8.STAT
- new net N$63: R54.2, U8.PRG
- new net N$64: R55.2, U7.PRG
- new net NTC_EXT: C19.2, R27.1, R56.2
- new net NTC_SENSE: R56.1
- new net V_BUZZER+: R57.1
- new net V_BUZZER-: Q1.D
- net 3.3V: now also R27.2; no longer JP5.2
- net GND: now also C16.1, C17.1, C18.1, C19.1, J10.1, J8.1, J9.1, R49.1, R50.1, R51.1, R54.1, R55.1, U7.VSS, U8.VSS; no longer X1-2.KL, X10-2.KL, X8-2.KL, X9-2.KL
- net N$12: now also Q12.G, R48.2; no longer PAD2.P, Q1.D, R27.1, SG1.-
- net N$27: now also D12.C, R50.2; no longer U7.BAT
- net N$36: now also J8.2; no longer X8-1.KL
- net N$42: now also J9.2; no longer X9-1.KL
- net N$48: now also J10.2; no longer X10-1.KL
- net N$54: now also D12.A
- net N$9: no longer R2.2
- net PYRO1_OUT: now also J11.1; no longer X6-2.KL
- net PYRO2_OUT: now also J12.1; no longer X7-2.KL
- net VCC_PYRO: now also J11.2, J12.2; no longer J3.2, JP1.2, X6-1.KL, X7-1.KL
- net V_BATT: now also C17.2, R57.2, U8.BAT; no longer D2.A, JP1.1, JP5.1, PAD1.P, SG1.+
- net V_GSM: now also C18.2, U7.BAT
- net V_LOAD: now also J3.2; no longer X1-1.KL
- net V_USB: now also C16.2, R52.1, R53.1, U8.VDD
Other:
- moved on the sheet: C10, C11, C12, C2, C4, C5, C6, C8, D10, D11, D3, D4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

Commit message: Updated balloon board
Parts:
- removed SV1: PANEL, con-ml:ML6
- removed SV2: I2C/GPS, con-ml:ML6
- removed U$29: STM32L063C, kg-mcu:STM32L063C
- added J13: INTERN, kg-amp-ct:M4-MM-4
- added J15: EXTERN, kg-amp-ct:M6-MM-6
- added U9: STM32L072R, kg-mcu:STM32L072R
- J10: value (none) -> AUX3
- J14: value 1WIRE -> THERMO
- J3: value (none) -> BATT AUX
- J4: value (none) -> SWD
- J6: value (none) -> UART
- J7: value BATT_GSM -> BATT GSM
- J8: value (none) -> AUX1
- J9: value (none) -> AUX2
- R12: value 100 -> 22
Connections:
- net D_BUZZER renamed BUZZER_ON
- net LED renamed LED_STATUS
- removed net D_PYRO1: R17.1, R19.1, U$29.PB1
- removed net D_PYRO2: R1.1, R18.1, U$29.PB0
- removed net N$21: C11.2, R12.1, U6.OUT
- new net N$8: C11.2, R12.1, U6.EN, U6.IN
- new net PYRO1_ON: R17.1, R19.1
- new net PYRO2_ON: R1.1, R18.1
- net !RST: no longer U$29.NRST
- net 3.3V: now also R12.2; no longer U$29.VBAT, U$29.VDD1, U$29.VDD2, U$29.VDDA, U$29.VDDIO2/PF7, U6.EN, U6.IN
- net ARM_SENSE: no longer U$29.PA7
- net DBG_RX: no longer U$29.PA3
- net DBG_TX: no longer U$29.PA2
- net GND: no longer U$29.BOOT0, U$29.VSS/PF6, U$29.VSS1, U$29.VSS2, U$29.VSSA
- net GPS_RXD: no longer U$29.PB7
- net GPS_TXD: no longer U$29.PB6
- net MISO: no longer U$29.PB4
- net MOSI: no longer U$29.PB5
- net PYRO1_SENSE: no longer U$29.PA5
- net PYRO2_SENSE: no longer U$29.PA4
- net RFM_DIO0: no longer U$29.PB2
- net SCK: no longer U$29.PB3
- net SCL: no longer U$29.PB8
- net SDA: no longer U$29.PB9
- net SWCLK: no longer U$29.SWCLK/PA14
- net SWDIO: no longer U$29.SWDIO/PA13
- net USB_DM: now also U9.PA11; no longer U$29.PA11
- net USB_DP: now also U9.PA12; no longer U$29.PA12
- net VCC_PYRO: now also U6.OUT; no longer R12.2
- net V_BATT_SENSE: no longer U$29.PA0
- net V_PYRO_SENSE: no longer U$29.PA1
Other:
- note added: "GSM ON"
- moved on the sheet: C11, R12
