File: eagle/tracker/tracker-balloon-full-sq.brd (EAGLE design)
At the start: 104 x 90 mm, 141 parts, among them J1 BATT, J10 AUX3, J13 INTERN, J14 THERMO, J15 EXTERN, J2 USB_MINI-B_SMT, J3 BATT AUX, J4 SWD, J5 MICRO-SD_CARD_SOCKET, J6 UART, J7 BATT GSM, J8 AUX1, J9 AUX2, M1 UBLOX-NEO-M8, M2 HOPE-RFM98W, M3 SIM800L-MODULE, M4 UBLOX-MAX-M8, U1 MS5637-02, U3 A25L010A, U4 MAG3110FCR1, U5 LSM6DS33, U7 MCP73831, U8 MCP73831, U9 STM32L072R, X4 ANTENNA-PATCH-12X12

Commit message: Updated ground board
Parts:
- added JP1: (no value), pinhead:1X10
- moved C13 110.5 mm to (140.0, 34.0), turned to 90 degrees
- moved R4 109.1 mm to (141.5, 29.5), turned to 270 degrees
- moved U1 107.8 mm to (140.5, 29.5), turned to 180 degrees
- moved U4 107.6 mm to (137.5, 34.0), turned to 270 degrees
- moved R3 106.6 mm to (139.5, 29.5), turned to 270 degrees
- moved C3 105.8 mm to (140.5, 26.5), turned to 0 degrees
- moved C14 104.6 mm to (135.0, 34.0), turned to 270 degrees
- moved U5 100.5 mm to (134.5, 29.5), turned to 180 degrees
- moved C15 100.2 mm to (136.0, 26.5), turned to 180 degrees
- moved J14 59.3 mm to (148.0, 14.5)
- moved FB3 29.7 mm to (68.5, 46.0), flipped to the top, turned to 270 degrees
- moved C9 25.8 mm to (71.5, 46.0), flipped to the top, turned to 0 degrees
- moved R15 24.9 mm to (84.0, 46.5), flipped to the bottom, turned to 0 degrees
- moved J15 23.3 mm to (136.5, 8.00)
- moved SV1 22.6 mm to (61.0, 31.5), turned to 90 degrees
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Other:
- board size 104 x 90 mm -> 80 x 80 mm
