File: eagle/tracker/tracker-balloon-full-sq.sch (EAGLE design)
At the start: 141 parts, among them J1 BATT, J10 AUX3, J13 INTERN, J14 THERMO, J15 EXTERN, J2 USB_MINI-B_SMT, J3 BATT AUX, J4 SWD, J5 MICRO-SD_CARD_SOCKET, J6 UART, J7 BATT GSM, J8 AUX1, J9 AUX2, M1 UBLOX-NEO-M8, M2 HOPE-RFM98W, M3 SIM800L-MODULE, M4 UBLOX-MAX-M8, U1 MS5637-02, U3 A25L010A, U4 MAG3110FCR1, U5 LSM6DS33, U7 MCP73831, U8 MCP73831, U9 STM32L072R, X4 ANTENNA-PATCH-12X12

Commit message: Updated ground board
Parts:
- added JP1: (no value), pinhead:PINHD-1X10
Changed lines of the file:
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@@
 <part name="J15" library="kg-amp-ct" deviceset="M6" device="-MM-6" value="EXTERN"/>
 <part name="SV1" library="con-ml" deviceset="ML6" device=""/>
+<part name="JP1" library="pinhead" deviceset="PINHD-1X10" device=""/>
 </parts>
 <sheets>
@@
 <instance part="J15" gate="G$1" x="779.78" y="91.44" rot="MR0"/>
 <instance part="SV1" gate="1" x="741.68" y="111.76"/>
+<instance part="JP1" gate="A" x="1049.02" y="71.12"/>
 </instances>
 <busses>
