File: eagle/tracker/tracker-ground-v1.brd (EAGLE design)
At the start: 100 x 75.5 mm, 90 parts, among them M1 UBLOX-NEO-6, M2 HOPE-RFM98W, M3 TFT-2.0-OPENSMART-THT, Q3 NTR5103N, U1 SI446X, U2 MCP73831, U3 A25L010A, U6 SI5351A, U8 STM32L052C8, X1 32.768kHz

Commit message: Updated ground board
Parts:
- removed C11, C14, C15: 100n, microbuilder_v3:_0603MP
- removed C12, C20, C28, C6, C7: (no value), kg-generic:C603
- removed C13: 10n, microbuilder_v3:_0603MP
- removed C16, C27: 10p, kg-generic:C603
- removed C21: 2u2, microbuilder_v3:_0603MP
- removed C22: NF/8p2/NF, microbuilder_v3:_0603MP
- removed C23: (no value), microbuilder_v3:_0603MP
- removed C24: 100n, kg-generic:C603
- removed C25, C26: 180p, kg-generic:C603
- removed C8: 2n2, microbuilder_v3:_0603MP
- removed CM: 10p/27p/68p, microbuilder_v3:_0603MP
- removed CM2: 15p/47p/150p, microbuilder_v3:_0603MP
- removed CM3: 8p2/27p/NF, microbuilder_v3:_0603MP
- removed ESD3: 0.25p, microbuilder_v3:_0603MP
- removed FB1, FB3, FB6: (no value), microbuilder_v3:_0805
- removed L0: 56n/100n/3.9u, microbuilder_v3:_0805MP
- removed L2: (no value), microbuilder_v3:_0805MP
- removed LM: 18n/68n/1.5u, microbuilder_v3:_0805MP
- removed LM1: 4.7u, microbuilder_v3:_0805MP
- removed LM2: 18n/68n/330n, microbuilder_v3:_0805MP
- removed LM3: 0.47u, microbuilder_v3:_0805MP
- removed LR1, LR3: 220n/470n, microbuilder_v3:_0805MP
- removed PAD1: (no value), wirepad:1,6/0,8
- removed Q3: NTR5103N, kg-generic:SOT23-3
- removed U1: SI446X, kg-sdrlib:QFN20
- removed U6: SI5351A, kg-sdrlib:MSOP10
- removed X1: 32.768kHz, IQD-Frequency-Products:3.2X1.5-2-PAD
- removed XO1: 26.000MHz TCXO, kg-crystal:CRYSTAL-SMD-2.5X2
- added D1: (no value), kg-generic:SOD-323
- added D2: (no value), diode:SOT23
- added JP2, JP3: I2C, pinhead:1X04
- added LED2: (no value), led:CHIPLED_0805
- added Q2: (no value), kg-generic:SOT23-3
- added S4: MOMENTARY-SWITCH-SPST-SMD-6.2MM-TALL, SparkFun-Switches:TACTILE_SWITCH_SMD_6.2MM_TALL
- added TP1: TPSB1,27, testpad:B1,27
- C1: value 10n -> (none)
- C4: value NF/8p2/NF -> (none); device microbuilder_v3:_0603MP -> kg-generic:C603
- L1: device microbuilder_v3:_0805MP -> kg-generic:R0805
- R1, R9: value 10k -> (none); device rcl:R0603 -> kg-generic:R0603
- R12: value 470 -> (none); device rcl:R0603 -> kg-generic:R0603
- R14: value 5.1k -> (none)
- R15: value 10 -> (none)
- R2: value 10k -> (none)
- R3, R4: value 4k7 -> (none); device rcl:R0603 -> kg-generic:R0603
- X4: value (none) -> ANTENNA-PATCH-12X12; device kg-conn-rf:SMA_EDGELAUNCH -> kg-modules:ANT-PATCH-12X12
- moved X3 97.6 mm to (15.0, 64.8), turned to 270 degrees
- moved U$42 92.6 mm to (4.00, 22.0), turned to 270 degrees
- moved LED1 90.9 mm to (4.00, 11.0), turned to 180 degrees
- moved ESD1 90.0 mm to (14.0, 58.5)
- moved R8 88.3 mm to (6.00, 11.0), turned to 270 degrees
- moved R7 86.3 mm to (7.50, 11.0), turned to 90 degrees
- moved C5 85.0 mm to (12.0, 49.5), turned to 270 degrees
- moved JP1 81.3 mm to (11.0, 4.00), flipped to the top
- moved U2 79.5 mm to (10.5, 11.0), turned to 0 degrees
- moved C19 78.3 mm to (13.0, 17.5), turned to 0 degrees
- moved FB5 77.0 mm to (13.0, 19.5), turned to 180 degrees
- moved M1 76.6 mm to (12.0, 37.5), turned to 0 degrees
- moved R6 76.0 mm to (13.0, 21.8), turned to 0 degrees
- moved R5 75.5 mm to (13.0, 23.2), turned to 0 degrees
- moved C18 72.5 mm to (13.0, 12.5), turned to 180 degrees
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Connections:
- removed net !RADIO_ON: Q1.1, R1.1
- removed net !TFT_CS: M3.P$6, U8.26
- removed net !TFT_LED: M3.P$8, U8.28
- removed net !TFT_RST: M3.P$7, U8.25
- removed net !TRX_CS: U1.15, U8.14
- removed net !TRX_EN: U1.1, U8.11
- removed net !TRX_IRQ: U1.11, U8.18
- removed net 3V3_RADIO: C12.2, FB1.2, FB3.1, FB4.2, FB6.1, XO1.4
- removed net 3V3_TRX: C11.1, C21.1, C7.2, C8.1, FB1.1, LR3.2, R11.1, U1.6
- removed net N$22: C15.1, R11.2, U1.8
- removed net N$23: C1.1, U6.2
- removed net N$24: C25.2, ESD3.2, LM3.1, X4.P
- removed net N$25: C26.2, LM1.1, LM3.2
- removed net N$27: U8.4, X1.1
- removed net N$30: C24.2, R15.1
- removed net N$32: CM2.1, LM.1, LM2.2
- removed net N$35: LED4.C, R12.2
- removed net N$36: C16.2, C27.2, LR1.1, Q3.3
- removed net N$37: C6.2, M2.9
- removed net N$38: C22.1, L1.1, L2.2, U1.2
- removed net N$39: C23.2, L1.2, U1.3
- removed net N$40: FB6.2, Q1.3
- removed net N$9: C5.1, ESD1.2, X3.P
- removed net RADIO_XIN: C13.2, U1.17
- removed net RF_TANK: C23.1, CM.1, L0.1, L2.1, LM.2
- removed net RF_TANK1: C16.1, LM1.2
- removed net TCXO_OUT: C1.2, C13.1, XO1.3
- removed net TFT_RS: M3.P$5, U8.27
- removed net TRX_GPIO0: U1.9, U8.20
- removed net TRX_GPIO1: U1.10, U8.19
- removed net TRX_GPIO2: U1.19
- removed net TRX_GPIO3: U1.20
- new net !TFT_CS/DB6: M3.P$6, U8.18
- new net !TFT_LED/DB4: M3.P$8, U8.16
- new net !TFT_RST/DB5: M3.P$7, U8.17
- new net BTN1: D2.1, U8.40
- new net BTN2: S2.A2, U8.41
- new net BTN3: S3.A2, U8.42
- new net BTN4: S4.A2, U8.43
- new net BTN_ON: D2.2, Q1.1, Q2.3, R12.1
- new net DBG_RXD: JP3.3, U8.13
- new net DBG_TXD: JP3.2, U8.12
- new net LCD_E: U8.14
- new net LCD_LED: U8.11
- new net LCD_RS: U8.15
- new net PWR_ON: Q2.1, R14.2, U8.2
- new net TFT_RS/DB7: M3.P$5, U8.19
- net !FLASH_CS: now also R15.1, U8.29
- net !LORA_IRQ: now also U8.20
- net !RST: now also C1.2, R4.1; no longer C14.1, R9.1
- net +3V3: now also FB4.2, JP2.4, JP3.4, R15.2, R2.2, U3.3, U3.7; no longer LED1.A, Q1.2, R1.2, R9.2
- net BAT_CHG: now also D1.A, U8.39; no longer R8.1, U2.1
- net GND: now also C1.1, C4.1, JP2.1, JP3.1, Q2.2, R1.1, R9.1, S1.B2, S2.B2, S3.B2, S4.B2, TP1.TP; no longer C11.2, C12.1, C14.2, C15.2, C20.1, C21.2, C22.2, C25.1, C26.1, C27.1, C4.2, C7.1, C8.2, CM.2, CM2.2, CM3.2, ESD3.1, Q3.2, R12.1, U1.18, U1.5, U1.PAD, U6.8, X4.GND@1, X4.GND@2, X4.GND@3, X4.GND@4, XO1.2
- net GPS_PPS: now also LED2.A, U8.25; no longer TP3.TP, U8.2
- net GPS_RXD: now also TP3.TP
- net LED: now also U8.38
- net MISO: now also U8.27; no longer U1.13, U8.16
- net MOSI: now also U8.28; no longer U1.14, U8.17
- net N$12: now also LED2.C, R1.2; no longer C28.2, LR3.1, U1.4
- net N$13: now also L1.2, R11.1; no longer R15.2, U6.10
- net N$15: now also C5.1, ESD1.2, L1.1, X3.P; no longer C28.1, C4.1, L0.2
- net N$17: now also C4.2, JP1.2, Q1.2, R12.2, U2.3; no longer M1.14
- net N$18: now also Q1.3; no longer JP1.2, U2.3
- net N$19: now also X4.FEED; no longer PAD1.1
- net N$20: now also D2.3, S1.A2; no longer C20.2, FB3.2, LR1.2, R2.2, U6.1, U6.7
- net N$21: now also D1.C, R8.1, U2.1; no longer U8.3, X1.2
- net N$31: now also M2.9; no longer C6.1, CM3.1, LM2.1
- net N$34: now also M1.2
- net N$5: now also LED4.C, R9.2; no longer C24.1, Q3.1, R14.2, R2.1
- net N$8: now also R11.2
- net SCK: now also U8.26; no longer U1.12, U8.15
- net SCL: now also JP2.2, R2.1, U8.45; no longer R3.1, U6.4, U8.42
- net SDA: now also JP2.3, R3.1, U8.46; no longer R4.1, U6.5, U8.43
- net USB_VBUS: now also LED1.A
Routing:
- net +3V3: track 2.60 -> 265.7 mm, vias 0 -> 4
- net SCL: track 0.00 -> 57.0 mm
- net SDA: track 0.00 -> 56.5 mm
- net DBG_RXD: track 0.00 -> 51.1 mm
- net DBG_TXD: track 0.00 -> 49.2 mm
- net TFT_RS/DB7: track 0.00 -> 49.2 mm
- net !TFT_CS/DB6: track 0.00 -> 48.6 mm
- net !TFT_RST/DB5: track 0.00 -> 48.1 mm
- net !TFT_LED/DB4: track 0.00 -> 47.5 mm
- net !LORA_IRQ: track 0.00 -> 46.3 mm, vias 0 -> 1
- net !FLASH_CS: track 0.00 -> 43.1 mm
- net BTN4: track 0.00 -> 41.6 mm
- net !RST: track 0.00 -> 39.9 mm, vias 0 -> 2
- net GPS_PPS: track 0.00 -> 36.2 mm, vias 0 -> 3
- net !TFT_LED: track 34.6 -> 0.00 mm, vias 1 -> 0
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Other:
- board size 100 x 75.5 mm -> 90 x 65 mm
- board text added: "(c) Karlis Goba 2018"
- board text added: "3.3V"
- board text added: "BTN1"
- board text added: "BTN2"
- board text added: "BTN3"
- board text added: "BTN4"
- board text added: "CLK"
- board text added: "DIO"
- board text added: "GND"
- board text added: "GNSS"
- board text added: "LoRa"
- board text added: "LoRa ground station v1.0"
- board text added: "PPS"
- board text added: "Prog"
- board text added: "RST"
- board text added: "RXD"
- board text added: "SCL"
- board text added: "SDA"
- board text added: "Stat"
- board text added: "TXD"
- board text added: "VBAT"
- board text removed: "Ant"
- board text removed: "BKP"
- board text removed: "CFG0"
- board text removed: "TReX"
- board text removed: "v1.1"
