File: eagle/tracker/tracker-ground-v1.brd (EAGLE design)
At the start: 90 x 65 mm, 61 parts, among them M1 UBLOX-NEO-6, M2 HOPE-RFM98W, M3 TFT-2.0-OPENSMART-THT, Q1 Si2365, Q2 CPH3448, U1 RT9013-33, U2 MCP73831, U3 A25L010A, U8 STM32L052C8, X4 ANTENNA-PATCH-12X12

Commit message: Updated ground station production board
Parts:
- added C11: 100n, kg-generic:C603
- added C8: *100n, kg-generic:C603
- C19, C4: device kg-generic:C603 -> kg-generic:C1206
- U8: value STM32L052C8 -> STM32L063C
- moved C17 3.54 mm to (22.5, 17.5)
- moved R10 3.54 mm to (20.5, 17.5)
- moved R13 3.54 mm to (18.5, 17.5)
- moved D1 2.55 mm to (16.5, 11.5)
- moved C2 2.12 mm to (15.5, 21.0)
- moved Q1 2.12 mm to (15.5, 11.5)
- moved R12 2.12 mm to (15.5, 8.50)
- moved U1 2.12 mm to (14.5, 17.5)
- moved C18 1.80 mm to (14.5, 14.0)
- moved R9 1.58 mm to (19.5, 11.5)
- moved LED4 1.12 mm to (21.0, 11.5)
- moved R7 1.12 mm to (8.50, 11.5)
- moved U2 1.12 mm to (11.5, 11.5)
- moved C19 0.50 mm to (13.0, 17.0)
- moved C4 0.50 mm to (11.0, 7.50)
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Connections:
- new net N$22: C11.2, U8.1
- new net N$9: C8.1, U1.4
- net +3V3: no longer U8.1
- net GND: now also C11.1, C8.2
Routing:
- net +3V3: track 255.7 -> 245.8 mm
- net GND: track 15.7 -> 11.3 mm, vias 176 -> 187
- net VBAT_ADC: track 32.1 -> 28.5 mm
- net N$22: track 0.00 -> 2.76 mm
- net BAT_CHG: track 31.7 -> 29.0 mm
- net N$21: track 11.3 -> 13.9 mm
- net N$9: track 0.00 -> 2.26 mm
- net BTN_ON: track 24.5 -> 22.4 mm
- net N$18: track 10.9 -> 12.9 mm
- net N$17: track 9.65 -> 11.4 mm
- net N$26: track 10.0 -> 8.30 mm
- net PWR_ON: track 20.2 -> 21.6 mm
- net LED: track 24.9 -> 23.7 mm
- net GPS_PPS: track 36.2 -> 36.9 mm
- net N$5: track 2.08 -> 1.58 mm
