File: eagle/tracker/tracker-ground-v1.brd (EAGLE design)
At the start: 90 x 65 mm, 63 parts, among them M1 UBLOX-NEO-6, M2 HOPE-RFM98W, M3 TFT-2.0-OPENSMART-THT, Q1 Si2365, Q2 CPH3448, U1 RT9013-33, U2 MCP73831, U3 A25L010A, U8 STM32L063C, X4 ANTENNA-PATCH-12X12

Commit message: Updates in ground tracker (TODO)
Parts:
- moved C7 3.00 mm to (48.5, 52.5)
- moved R15 3.00 mm to (49.5, 55.0)
- moved U3 3.00 mm to (49.5, 51.0)
Connections:
- net !LORA_CS: now also U8.18; no longer U8.21
- net !LORA_RST: now also U8.19; no longer U8.22
- net !TFT_CS: now also U8.21; no longer U8.18
- net TFT_RS: now also U8.22; no longer U8.19
Routing:
- net TFT_RS: track 49.2 -> 52.4 mm
- net !TFT_CS: track 48.6 -> 51.8 mm
- net !FLASH_CS: track 42.2 -> 39.2 mm
- net +3V3: track 245.8 -> 244.5 mm
- net !LORA_RST: track 38.8 -> 37.6 mm, vias 1 -> 3
- net !LORA_CS: track 38.1 -> 36.9 mm, vias 1 -> 3
- net !LORA_IRQ: track 46.3 -> 46.9 mm
- net GND: vias 187 -> 186
