File: eagle/tracker/tracker-ground-v1.sch (EAGLE design)
At the start: 84 parts, among them M1 UBLOX-NEO-6, M2 HOPE-RFM98W, Q3 NTR5103N, Q4 NTR5103N, U1 SI446X, U2 MCP73831, U3 A25L010A, U6 SI5351A, U8 STM32L052C8, X1 32.768kHz

Commit message: Added balloon/ground boards
Parts:
- removed C0: 10p/330p/68p, microbuilder_v3:CAP_CERAMIC_0603MP
- removed CM1: 15p/47p/150p, microbuilder_v3:CAP_CERAMIC_0603MP
- removed CM4: 8p2/27p/NF, microbuilder_v3:CAP_CERAMIC_0603MP
- removed JP4: JUMPER-PAD-2-NOYES_SILK, SparkFun-Passives:JUMPER-PAD-2-NOYES_SILK
- removed JP9: (no value), pinhead:PINHD-1X8
- removed Q2: (no value), kg-generic:MOSFET-P-SOT23-3
- removed Q4: NTR5103N, kg-generic:MOSFET-N-SOT23-3
- removed TP10, TP11: TPSB1,27, testpad:TPSB1,27
- added C22: NF/8p2/NF, microbuilder_v3:CAP_CERAMIC_0603MP
- added C23: (no value), microbuilder_v3:CAP_CERAMIC_0603MP
- added C24: 100n, kg-generic:CAPACITOR_NPOL-0603
- added C25, C26: 180p, kg-generic:CAPACITOR_NPOL-0603
- added C27: 10p, kg-generic:CAPACITOR_NPOL-0603
- added C28: (no value), kg-generic:CAPACITOR_NPOL-0603
- added FB6: (no value), microbuilder_v3:FERRITE_0805
- added L1, L2: (no value), microbuilder_v3:INDUCTOR_0805MP
- added M3: TFT-2.0-OPENSMART-THT, kg-modules:TFT-2.0-OPENSMART-THT
- added PAD1: (no value), wirepad:1,6/0,8
- added R15: 10, kg-generic:RESISTOR-0603
- added S2, S3: MOMENTARY-SWITCH-SPST-SMD-6.2MM-TALL, SparkFun-Switches:MOMENTARY-SWITCH-SPST-SMD-6.2MM-TALL
- C1: device microbuilder_v3:CAP_CERAMIC_0603MP -> kg-generic:CAPACITOR_NPOL-0603
- C16: value (none) -> 10p
- C3: value 0R -> (none); device microbuilder_v3:CAP_CERAMIC_0603MP -> kg-generic:CAPACITOR_NPOL-0603
- C5: value 100n -> NF*; device microbuilder_v3:CAP_CERAMIC_0603MP -> kg-generic:CAPACITOR_NPOL-0603
- LM1: value 18n/68n/1.5u -> 4.7u
- LM3: value 18n/68n/330n -> 0.47u
- R14: value (none) -> 5.1k
- R2: value 100k -> 10k; device rcl:R-EU_R0603 -> kg-generic:RESISTOR-0603
Connections:
- removed net !GPS_ON: Q2.G, R14.1
- removed net CHG_STATUS: LED1.C, U2.STAT
- removed net DBG_RX: U8.PA10
- removed net DBG_TX: U8.PA9
- new net 3V3_TRX: C11.P$1, C21.P$1, C7.2, C8.P$1, FB1.P$1, LR3.2, R11.1, U1.VDDA
- new net BAT_CHG: R8.1, U2.STAT
- new net N$38: C22.P$1, L1.1, L2.2, U1.RXP
- new net N$39: C23.P$2, L1.2, U1.RXN
- new net N$40: FB6.P$2, Q1.D
- net !LORA_CS: now also U8.PB10
- net !LORA_RST: now also U8.PB11
- net !TFT_CS: now also M3.!CS, U8.PB13; no longer JP9.6
- net !TFT_LED: now also M3.LED, U8.PB15; no longer JP9.8
- net !TFT_RST: now also M3.!RST, U8.PB12; no longer JP9.7
- net !TRX_CS: now also U8.PA4
- net !TRX_EN: now also U8.PA1
- net !TRX_IRQ: now also U8.PB0
- net +3V3: now also C3.2, FB2.P$1, LED1.A, M3.VCC; no longer C5.P$1, M1.V_BCKP, Q2.S, R14.2
- net 3V3_RADIO: now also FB6.P$1; no longer C11.P$1, C21.P$1, C7.2, C8.P$1, FB1.P$1, LR3.2, Q1.D, R11.1, U1.VDDA
- net GND: now also C22.P$2, C25.1, C26.1, C27.1, C3.1, M1.V_BCKP, M3.GND, R14.1; no longer C5.P$2, CM1.P$2, CM4.P$2, JP4.2, JP9.1, Q4.S, R2.1
- net GPS_RXD: now also U8.PA10; no longer U8.PB11
- net GPS_TXD: now also U8.PA9; no longer U8.PB10
- net MOSI: now also M3.SDI; no longer JP9.3
- net N$12: now also C28.2; no longer C0.P$2
- net N$13: now also R15.2, U6.CLK0; no longer FB2.P$1, Q2.D
- net N$15: now also C28.1; no longer C0.P$1
- net N$16: now also LED1.C, R8.2; no longer C3.P$2, M1.RF_IN
- net N$17: no longer JP4.1
- net N$19: now also C5.2, M1.RF_IN, PAD1.P; no longer C3.P$1, ESD1.P$2, X3.ANT
- net N$20: now also R2.2
- net N$23: now also C1.1; no longer C1.P$2
- net N$24: now also C25.2; no longer CM4.P$1
- net N$25: now also C26.2; no longer CM1.P$1
- net N$30: now also C24.2, R15.1; no longer JP9.2
- net N$36: now also C27.2; no longer Q4.D
- net N$5: now also C24.1, R14.2, R2.1; no longer Q4.G, R2.2, U6.CLK0
- net N$9: now also C5.1, ESD1.P$2, X3.ANT; no longer LED1.A, R8.1
- net RF_TANK: now also C23.P$1, L2.1
- net SCK: now also M3.SCK; no longer JP9.4
- net TCXO_OUT: now also C1.2; no longer C1.P$1
- net TFT_RS: now also M3.D/C, U8.PB14; no longer JP9.5
- net TRX_GPIO0: now also U8.PB2
- net TRX_GPIO1: now also U8.PB1
- net TRX_GPIO2: no longer TP11.PP
- net TRX_GPIO3: no longer TP10.PP
- net USB_VBUS: no longer R8.2
- net VBAT_ADC: now also U8.PA0
Other:
- note added: "HF LPF and matching"
- note added: "TODO: - prog/debug connectors - GPIO/I2C header? - SD card vs Flash"
- note added: "UHF/VHF LPF"
- note removed: "TODO: - review LDO/Q3 - universal RF match 2m/70cm - prog/debug connectors - Flash package?"
- note removed: "Tuned for 434MHz/144Mhz/21MHz"
- moved on the sheet: C10, C11, C16, C18, C21, C4, C6, C7, C8, CM, CM2, CM3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

Commit message: Updated ground board
Parts:
- removed C11, C14, C15: 100n, microbuilder_v3:CAP_CERAMIC_0603MP
- removed C12, C20, C28, C6, C7: (no value), kg-generic:CAPACITOR_NPOL-0603
- removed C13: 10n, microbuilder_v3:CAP_CERAMIC_0603MP
- removed C16, C27: 10p, kg-generic:CAPACITOR_NPOL-0603
- removed C21: 2u2, microbuilder_v3:CAP_CERAMIC_0603MP
- removed C22: NF/8p2/NF, microbuilder_v3:CAP_CERAMIC_0603MP
- removed C23: (no value), microbuilder_v3:CAP_CERAMIC_0603MP
- removed C24: 100n, kg-generic:CAPACITOR_NPOL-0603
- removed C25, C26: 180p, kg-generic:CAPACITOR_NPOL-0603
- removed C8: 2n2, microbuilder_v3:CAP_CERAMIC_0603MP
- removed CM: 10p/27p/68p, microbuilder_v3:CAP_CERAMIC_0603MP
- removed CM2: 15p/47p/150p, microbuilder_v3:CAP_CERAMIC_0603MP
- removed CM3: 8p2/27p/NF, microbuilder_v3:CAP_CERAMIC_0603MP
- removed ESD3: 0.25p, microbuilder_v3:FERRITE_0603MP
- removed FB1, FB3, FB6: (no value), microbuilder_v3:FERRITE_0805
- removed L0: 56n/100n/3.9u, microbuilder_v3:INDUCTOR_0805MP
- removed L2: (no value), microbuilder_v3:INDUCTOR_0805MP
- removed LM: 18n/68n/1.5u, microbuilder_v3:INDUCTOR_0805MP
- removed LM1: 4.7u, microbuilder_v3:INDUCTOR_0805MP
- removed LM2: 18n/68n/330n, microbuilder_v3:INDUCTOR_0805MP
- removed LM3: 0.47u, microbuilder_v3:INDUCTOR_0805MP
- removed LR1, LR3: 220n/470n, microbuilder_v3:INDUCTOR_0805MP
- removed PAD1: (no value), wirepad:1,6/0,8
- removed Q3: NTR5103N, kg-generic:MOSFET-N-SOT23-3
- removed U1: SI446X, kg-sdrlib:SI446X
- removed U6: SI5351A, kg-sdrlib:SI5351A
- removed X1: 32.768kHz, IQD-Frequency-Products:CRYSTALS-NOGND-CFPX-217
- removed XO1: 26.000MHz TCXO, kg-crystal:XTAL-OSC-2.5X2
- added D1: (no value), kg-generic:DIODE-SCHOTTKY-SOD323
- added D2: (no value), diode:DIODE-2AC|CASOT23
- added JP2, JP3: I2C, pinhead:PINHD-1X4
- added LED2: (no value), led:LEDCHIPLED_0805
- added Q2: (no value), kg-generic:MOSFET-N-SOT23-3
- added S4: MOMENTARY-SWITCH-SPST-SMD-6.2MM-TALL, SparkFun-Switches:MOMENTARY-SWITCH-SPST-SMD-6.2MM-TALL
- added TP1: TPSB1,27, testpad:TPSB1,27
- C1: value 10n -> (none)
- C4: value NF/8p2/NF -> (none); device microbuilder_v3:CAP_CERAMIC_0603MP -> kg-generic:CAPACITOR_NPOL-0603
- L1: device microbuilder_v3:INDUCTOR_0805MP -> kg-generic:L-0805
- R1, R9: value 10k -> (none); device rcl:R-EU_R0603 -> kg-generic:RESISTOR-0603
- R12: value 470 -> (none); device rcl:R-EU_R0603 -> kg-generic:RESISTOR-0603
- R14: value 5.1k -> (none)
- R15: value 10 -> (none)
- R2: value 10k -> (none)
- R3, R4: value 4k7 -> (none); device rcl:R-EU_R0603 -> kg-generic:RESISTOR-0603
- X4: value (none) -> ANTENNA-PATCH-12X12; device kg-conn-rf:SMACONNECTOR_EDGE -> kg-modules:ANTENNA-PATCH-12X12
Connections:
- removed net !RADIO_ON: Q1.G, R1.1
- removed net !TFT_CS: M3.!CS, U8.PB13
- removed net !TFT_LED: M3.LED, U8.PB15
- removed net !TFT_RST: M3.!RST, U8.PB12
- removed net !TRX_CS: U1.!SEL, U8.PA4
- removed net !TRX_EN: U1.SDN, U8.PA1
- removed net !TRX_IRQ: U1.!IRQ, U8.PB0
- removed net 3V3_RADIO: C12.2, FB1.P$2, FB3.P$1, FB4.P$2, FB6.P$1, XO1.VCC
- removed net 3V3_TRX: C11.P$1, C21.P$1, C7.2, C8.P$1, FB1.P$1, LR3.2, R11.1, U1.VDDA
- removed net N$22: C15.P$1, R11.2, U1.VDD
- removed net N$23: C1.1, U6.XA
- removed net N$24: C25.2, ESD3.P$2, LM3.1, X4.ANT
- removed net N$25: C26.2, LM1.1, LM3.2
- removed net N$27: U8.PC15/OSC32O, X1.1
- removed net N$30: C24.2, R15.1
- removed net N$32: CM2.P$1, LM.1, LM2.2
- removed net N$35: LED4.C, R12.2
- removed net N$36: C16.2, C27.2, LR1.1, Q3.D
- removed net N$37: C6.2, M2.ANT
- removed net N$38: C22.P$1, L1.1, L2.2, U1.RXP
- removed net N$39: C23.P$2, L1.2, U1.RXN
- removed net N$40: FB6.P$2, Q1.D
- removed net N$9: C5.1, ESD1.P$2, X3.ANT
- removed net RADIO_XIN: C13.P$2, U1.XIN
- removed net RF_TANK: C23.P$1, CM.P$1, L0.1, L2.1, LM.2
- removed net RF_TANK1: C16.1, LM1.2
- removed net TCXO_OUT: C1.2, C13.P$1, XO1.OUT
- removed net TFT_RS: M3.D/C, U8.PB14
- removed net TRX_GPIO0: U1.GPIO0, U8.PB2
- removed net TRX_GPIO1: U1.GPIO1, U8.PB1
- removed net TRX_GPIO2: U1.GPIO2
- removed net TRX_GPIO3: U1.GPIO3
- new net !TFT_CS/DB6: M3.!CS, U8.PB0
- new net !TFT_LED/DB4: M3.LED, U8.PA6
- new net !TFT_RST/DB5: M3.!RST, U8.PA7
- new net BTN1: D2.A1, U8.PB4
- new net BTN2: S2.1, U8.PB5
- new net BTN3: S3.1, U8.PB6
- new net BTN4: S4.1, U8.PB7
- new net BTN_ON: D2.A2, Q1.G, Q2.D, R12.1
- new net DBG_RXD: JP3.3, U8.PA3
- new net DBG_TXD: JP3.2, U8.PA2
- new net LCD_E: U8.PA4
- new net LCD_LED: U8.PA1
- new net LCD_RS: U8.PA5
- new net PWR_ON: Q2.G, R14.2, U8.PC13
- new net TFT_RS/DB7: M3.D/C, U8.PB1
- net !FLASH_CS: now also R15.1, U8.PA8
- net !LORA_IRQ: now also U8.PB2
- net !RST: now also C1.2, R4.1; no longer C14.P$1, R9.1
- net +3V3: now also FB4.P$2, JP2.4, JP3.4, R15.2, R2.2, U3.HOLD, U3.WP; no longer LED1.A, Q1.S, R1.2, R9.2
- net BAT_CHG: now also D1.A, U8.PB3; no longer R8.1, U2.STAT
- net GND: now also C1.1, C4.1, JP2.1, JP3.1, Q2.S, R1.1, R9.1, S1.2, S2.2, S3.2, S4.2, TP1.PP; no longer C11.P$2, C12.1, C14.P$2, C15.P$2, C20.1, C21.P$2, C22.P$2, C25.1, C26.1, C27.1, C4.P$2, C7.1, C8.P$2, CM.P$2, CM2.P$2, CM3.P$2, ESD3.P$1, Q3.S, R12.1, U1.GND, U1.NC, U6.GND, X4.GND1, X4.GND2, X4.GND3, X4.GND4, XO1.GND
- net GPS_PPS: now also LED2.A, U8.PB12; no longer TP3.PP, U8.PC13
- net GPS_RXD: now also TP3.PP
- net LED: now also U8.PA15
- net MISO: now also U8.PB14; no longer U1.SDO, U8.PA6
- net MOSI: now also U8.PB15; no longer U1.SDI, U8.PA7
- net N$12: now also LED2.C, R1.2; no longer C28.2, LR3.1, U1.TX
- net N$13: now also L1.2, R11.1; no longer R15.2, U6.CLK0
- net N$15: now also C5.1, ESD1.P$2, L1.1, X3.ANT; no longer C28.1, C4.P$1, L0.2
- net N$17: now also C4.2, JP1.2, Q1.S, R12.2, U2.BAT; no longer M1.MOSI/CFG_COM0
- net N$18: now also Q1.D; no longer JP1.2, U2.BAT
- net N$19: now also X4.FEED; no longer PAD1.P
- net N$20: now also D2.C, S1.1; no longer C20.2, FB3.P$2, LR1.2, R2.2, U6.VDD, U6.VDDO
- net N$21: now also D1.C, R8.1, U2.STAT; no longer U8.PC14/OSC32I, X1.2
- net N$31: now also M2.ANT; no longer C6.1, CM3.P$1, LM2.1
- net N$34: now also M1.SS_N
- net N$5: now also LED4.C, R9.2; no longer C24.1, Q3.G, R14.2, R2.1
- net N$8: now also R11.2
- net SCK: now also U8.PB13; no longer U1.SCLK, U8.PA5
- net SCL: now also JP2.2, R2.1, U8.PB8; no longer R3.1, U6.SCL, U8.PB6
- net SDA: now also JP2.3, R3.1, U8.PB9; no longer R4.1, U6.SDA, U8.PB7
- net USB_VBUS: now also LED1.A
Other:
- note removed: "HF LPF and matching"
- note removed: "UHF/VHF LPF"
- moved on the sheet: C1, C17, C18, C19, C2, C9, ESD2, FB2, JP1, LED1, Q1, R10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
