File: eagle/tracker/tracker-ground-v1.sch (EAGLE design)
At the start: 61 parts, among them M1 UBLOX-NEO-6, M2 HOPE-RFM98W, M3 TFT-2.0-OPENSMART-THT, Q1 Si2365, Q2 CPH3448, U1 RT9013-33, U2 MCP73831, U3 A25L010A, U8 STM32L052C8, X4 ANTENNA-PATCH-12X12

Commit message: Updated ground station production board
Parts:
- added C11: 100n, kg-generic:CAPACITOR_NPOL-0603
- added C8: *100n, kg-generic:CAPACITOR_NPOL-0603
- C19, C4: device kg-generic:CAPACITOR_NPOL-0603 -> kg-generic:CAPACITOR_NPOL-1206
- U8: value STM32L052C8 -> STM32L063C; device kg-mcu:STM32L052C8 -> kg-mcu:STM32L063C
Connections:
- new net N$22: C11.2, U8.VLCD/VBAT
- new net N$9: C8.1, U1.BP
- net +3V3: now also U8.VDD1, U8.VDD2, U8.VDDIO2/PF7; no longer U8.VDD, U8.VDDUSB
- net GND: now also C11.1, C8.2, U8.VSS/PF6, U8.VSS1, U8.VSS2; no longer U8.VSS
Other:
- moved on the sheet: C19, C3, C4, D1, LED1, R7, R8, U2
