File: eagle/tracker/tracker-ground-v1.sch (EAGLE design)
At the start: 63 parts, among them M1 UBLOX-NEO-6, M2 HOPE-RFM98W, M3 TFT-2.0-OPENSMART-THT, Q1 Si2365, Q2 CPH3448, U1 RT9013-33, U2 MCP73831, U3 A25L010A, U8 STM32L063C, X4 ANTENNA-PATCH-12X12

Commit message: Updates in ground tracker (TODO)
Connections:
- net !LORA_CS: now also U8.PB0; no longer U8.PB10
- net !LORA_RST: now also U8.PB1; no longer U8.PB11
- net !TFT_CS: now also U8.PB10; no longer U8.PB0
- net TFT_RS: now also U8.PB11; no longer U8.PB1
Other:
- note added: "TODO: - DC barrel + 5V reg - I_bat test bridge/connector - Change to 6 button channels - External button connector (IDC) - External connections at chipLEDs - MicroSD card? - RTC? - GSM? - Supercap for VBAT (GSM)"
- note removed: "TODO: - prog/debug connectors - GPIO/I2C header? - SD card vs Flash"
