File: eagle/tracker/tracker-gsm.sch (EAGLE design)
At the start: 63 parts, among them M1 UBLOX-NEO-6, M2 HOPE-RFM98W, M3 TFT-2.0-OPENSMART-THT, Q1 Si2365, Q2 CPH3448, U1 RT9013-33, U2 MCP73831, U3 A25L010A, U8 STM32L063C, X4 ANTENNA-PATCH-12X12

Commit message: Added standalone GSM tracker
Parts:
- removed D1: (no value), kg-generic:DIODE-SCHOTTKY-SOD323
- removed FB4: (no value), microbuilder_v3:FERRITE_0805
- removed M3: TFT-2.0-OPENSMART-THT, kg-modules:TFT-2.0-OPENSMART-THT
- removed S3, S4: MOMENTARY-SWITCH-SPST-SMD-6.2MM-TALL, SparkFun-Switches:MOMENTARY-SWITCH-SPST-SMD-6.2MM-TALL
- removed X2: (no value), kg-conn-rf:SMACONNECTOR_EDGE
- added R16, R17, R19: 1k, kg-generic:RESISTOR-0603
- added R18, R20: 5.6k, kg-generic:RESISTOR-0603
- added X1: (no value), kg-conn-rf:SMACONNECTOR_EDGE
- C10: value 100n -> NF*
- ESD2: value 0.25p -> NF
- M2: value HOPE-RFM98W -> SIM800L-MODULE; device kg-modules:HOPE-RFM98W -> kg-modules:SIM800L-MODULE
Connections:
- removed net !LORA_CS: M2.!SS, U8.PB10
- removed net !LORA_IRQ: M2.DIO0, U8.PB2
- removed net !LORA_RST: M2.!RESET, U8.PB11
- removed net !TFT_CS: M3.!CS, U8.PB0
- removed net !TFT_LED: M3.LED, U8.PA6
- removed net !TFT_RST: M3.!RST, U8.PA7
- removed net BAT_CHG: D1.A, U8.PB3
- removed net BTN3: S3.1, U8.PB6
- removed net BTN4: S4.1, U8.PB7
- removed net N$28: C10.2, FB4.P$1, M2.3.3V
- removed net N$31: ESD2.P$2, M2.ANT, X2.ANT
- removed net TFT_RS: M3.D/C, U8.PB1
- new net !GSM_RST: M2.!RST, U8.PB1
- new net GSM_DTR: R19.2, U8.PB2
- new net GSM_RXD: R16.2, U8.PB11
- new net GSM_TXD: R17.2, U8.PB10
- new net N$23: C10.1, ESD2.P$2, X1.ANT
- new net N$24: C10.2, M2.ANT
- new net N$25: M2.RXD, R17.1, R18.2
- new net N$27: M2.DTR, R19.1, R20.2
- new net VBAT: C18.2, M2.VCC, Q1.D, R13.2, U1.EN, U1.IN
- net !FLASH_CS: now also U8.PB0; no longer U8.PA8
- net +3V3: no longer FB4.P$2, M3.VCC
- net DBG_RXD: now also U8.PA10; no longer U8.PA3
- net DBG_TXD: now also U8.PA9; no longer U8.PA2
- net GND: now also M2.GND, R18.1, R20.1, X1.GND1, X1.GND2, X1.GND3, X1.GND4; no longer C10.1, M2.GND1, M2.GND2, M2.GND3, M3.GND, S3.2, S4.2, X2.GND1, X2.GND2, X2.GND3, X2.GND4
- net GPS_PPS: now also U8.PA1; no longer U8.PB12
- net GPS_RXD: now also U8.PA3; no longer U8.PA10
- net GPS_TXD: now also U8.PA2; no longer U8.PA9
- net MISO: now also U8.PA6; no longer M2.MISO, U8.PB14
- net MOSI: now also U8.PA7; no longer M2.MOSI, M3.SDI, U8.PB15
- net N$18: now also M2.TXD, R16.1; no longer C18.2, Q1.D, R13.2, U1.EN, U1.IN
- net N$21: no longer D1.C
- net SCK: now also U8.PA5; no longer M2.SCK, M3.SCK, U8.PB13
Other:
- moved on the sheet: C10, ESD2
