File: eagle/tracker/tracker-gsm.brd (EAGLE design)
At the start: 90 x 65 mm, 63 parts, among them M1 UBLOX-NEO-6, M2 HOPE-RFM98W, M3 TFT-2.0-OPENSMART-THT, Q1 Si2365, Q2 CPH3448, U1 RT9013-33, U2 MCP73831, U3 A25L010A, U8 STM32L063C, X4 ANTENNA-PATCH-12X12

Commit message: Added standalone GSM tracker
Parts:
- removed D1: (no value), kg-generic:SOD-323
- removed FB4: (no value), microbuilder_v3:_0805
- removed M3: TFT-2.0-OPENSMART-THT, kg-modules:TFT-2.0-OPENSMART
- removed S3, S4: MOMENTARY-SWITCH-SPST-SMD-6.2MM-TALL, SparkFun-Switches:TACTILE_SWITCH_SMD_6.2MM_TALL
- removed X2: (no value), kg-conn-rf:SMA_EDGELAUNCH
- added R16, R17, R19: 1k, kg-generic:R0603
- added R18, R20: 5.6k, kg-generic:R0603
- added X1: (no value), kg-conn-rf:SMA_EDGELAUNCH
- C10: value 100n -> NF*
- ESD2: value 0.25p -> NF
- M2: value HOPE-RFM98W -> SIM800L-MODULE; device kg-modules:HOPE-RFM -> kg-modules:SIM800L
- moved X3 79.4 mm to (89.8, 38.0), turned to 180 degrees
- moved ESD1 72.2 mm to (83.5, 39.0), turned to 270 degrees
- moved ESD2 68.7 mm to (6.50, 29.5), turned to 90 degrees
- moved L1 66.1 mm to (77.0, 35.5), turned to 270 degrees
- moved C5 63.8 mm to (74.5, 36.5), turned to 0 degrees
- moved X4 62.1 mm to (73.0, 36.5), turned to 90 degrees
- moved R11 61.3 mm to (74.5, 33.0), turned to 0 degrees
- moved C10 55.1 mm to (10.5, 28.0), flipped to the top, turned to 270 degrees
- moved LED2 54.8 mm to (57.5, 44.5), turned to 90 degrees
- moved R1 52.5 mm to (57.5, 42.5), turned to 180 degrees
- moved M1 50.5 mm to (62.5, 36.5), turned to 90 degrees
- moved TP3 43.0 mm to (58.0, 33.5), turned to 0 degrees
- moved TP1 40.6 mm to (55.5, 33.5), turned to 90 degrees
- moved M2 37.4 mm to (27.0, 24.0), flipped to the top, turned to 90 degrees
- moved C9 36.7 mm to (57.0, 28.0), turned to 0 degrees
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Connections:
- removed net !LORA_CS: M2.5, U8.21
- removed net !LORA_IRQ: M2.14, U8.20
- removed net !LORA_RST: M2.6, U8.22
- removed net !TFT_CS: M3.P$6, U8.18
- removed net !TFT_LED: M3.P$8, U8.16
- removed net !TFT_RST: M3.P$7, U8.17
- removed net BAT_CHG: D1.A, U8.39
- removed net BTN3: S3.A2, U8.42
- removed net BTN4: S4.A2, U8.43
- removed net N$28: C10.2, FB4.1, M2.13
- removed net N$31: ESD2.2, M2.9, X2.P
- removed net TFT_RS: M3.P$5, U8.19
- new net !GSM_RST: M2.3, U8.19
- new net GSM_DTR: R19.2, U8.20
- new net GSM_RXD: R16.2, U8.22
- new net GSM_TXD: R17.2, U8.21
- new net N$23: C10.1, ESD2.2, X1.P
- new net N$24: C10.2, M2.1
- new net N$25: M2.4, R17.1, R18.2
- new net N$27: M2.11, R19.1, R20.2
- new net VBAT: C18.2, M2.2, Q1.3, R13.2, U1.1, U1.3
- net !FLASH_CS: now also U8.18; no longer U8.29
- net +3V3: no longer FB4.2, M3.P$2
- net DBG_RXD: now also U8.31; no longer U8.13
- net DBG_TXD: now also U8.30; no longer U8.12
- net GND: now also M2.6, R18.1, R20.1, X1.GND@1, X1.GND@2, X1.GND@3, X1.GND@4; no longer C10.1, M2.1, M2.10, M2.8, M3.P$1, S3.B2, S4.B2, X2.GND@1, X2.GND@2, X2.GND@3, X2.GND@4
- net GPS_PPS: now also U8.11; no longer U8.25
- net GPS_RXD: now also U8.13; no longer U8.31
- net GPS_TXD: now also U8.12; no longer U8.30
- net MISO: now also U8.16; no longer M2.2, U8.27
- net MOSI: now also U8.17; no longer M2.3, M3.P$3, U8.28
- net N$18: now also M2.5, R16.1; no longer C18.2, Q1.3, R13.2, U1.1, U1.3
- net N$21: no longer D1.C
- net SCK: now also U8.15; no longer M2.4, M3.P$4, U8.26
Routing:
- net +3V3: track 245.8 -> 78.7 mm, vias 8 -> 5
- net MOSI: track 70.7 -> 8.46 mm, vias 3 -> 2
- net SCK: track 71.6 -> 11.3 mm, vias 2 -> 0
- net DBG_RXD: track 51.1 -> 0.00 mm
- net SCL: track 57.0 -> 6.55 mm
- net SDA: track 56.5 -> 6.83 mm
- net DBG_TXD: track 49.2 -> 0.00 mm
- net TFT_RS: track 49.2 -> 0.00 mm
- net !TFT_CS: track 48.6 -> 0.00 mm
- net !TFT_RST: track 48.1 -> 0.00 mm
- net !TFT_LED: track 47.5 -> 0.00 mm
- net !LORA_IRQ: track 46.3 -> 0.00 mm, vias 1 -> 0
- net BTN4: track 41.6 -> 0.00 mm
- net !LORA_RST: track 38.8 -> 0.00 mm, vias 1 -> 0
- net MISO: track 49.4 -> 10.8 mm, vias 1 -> 0
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Other:
- board size 90 x 65 mm -> 90 x 50 mm
- board text added: "BTN1/PWR"
- board text removed: "BTN1"
- board text removed: "BTN3"
- board text removed: "BTN4"

Commit message: Updates in ground tracker (TODO)
Parts:
- moved LED4 43.1 mm to (3.00, 34.5), turned to 180 degrees
- moved R15 41.0 mm to (7.50, 31.5), turned to 90 degrees
- moved R9 40.6 mm to (4.50, 34.5), turned to 270 degrees
- moved JP2 37.5 mm to (105.5, 13.5), turned to 90 degrees
- moved C7 37.2 mm to (10.0, 30.5), turned to 90 degrees
- moved U3 35.8 mm to (11.5, 31.5), turned to 0 degrees
- moved R2 35.4 mm to (101.5, 12.0), turned to 0 degrees
- moved R3 33.1 mm to (101.5, 14.0), turned to 0 degrees
- moved JP3 28.0 mm to (105.5, 26.5), turned to 90 degrees
- moved R4 23.8 mm to (30.0, 36.0), turned to 180 degrees
- moved C1 21.8 mm to (30.0, 34.5), turned to 0 degrees
- moved LED1 21.5 mm to (3.00, 12.0), turned to 0 degrees
- moved R8 20.6 mm to (6.00, 12.0), turned to 90 degrees
- moved R7 19.0 mm to (8.00, 12.0)
- moved U2 19.0 mm to (11.0, 12.0)
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Routing:
- net BTN2: track 31.1 -> 0.00 mm
- net USB_DM: track 30.7 -> 0.00 mm
- net USB_DP: track 29.2 -> 0.00 mm
- net LED: track 21.5 -> 0.07 mm, vias 2 -> 0
- net SWDIO: track 26.5 -> 5.71 mm
- net BTN1: track 20.0 -> 0.00 mm
- net SWCLK: track 23.6 -> 3.81 mm
- net !RST: track 37.2 -> 18.0 mm
- net USB_VBUS: track 31.6 -> 14.2 mm, vias 0 -> 2
- net VBAT: track 8.39 -> 17.8 mm
- net N$21: track 7.52 -> 5.28 mm, vias 2 -> 0
- net BTN_ON: track 22.4 -> 23.7 mm
- net N$16: track 2.08 -> 3.08 mm
- net N$26: track 8.30 -> 7.44 mm, vias 2 -> 1
- net N$17: track 11.4 -> 12.2 mm
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Other:
- board size 90 x 50 mm -> 78 x 45 mm
