File: eagle/tracker/flight-28mm.brd (EAGLE design)
At the start: 74 x 28 mm, 72 parts, among them J1 BATT, J2 USB_MINI-B_SMT, J3 BATT_PYRO, U1 LIS3MDL, U10 MPL3115A2, U3 A25L010A, U4 MAG3110FCR1, U5 LSM6DS33, U7 H3LIS100DL, U8 MMA6825, X4 MICROMATCH-8

Commit message: Changes to LoRa tracker
Parts:
- removed J3: BATT_PYRO, kg-amp-ct:JST-2-PTH-VERT
- removed TP4, TP5: TPB1,27, testpad:B1,27
- added C12: 3.0F, rcl:E3,5-8
- JP2: value BYPASS2 -> CFG1
- JP3: value BYPASS2 -> CFG2
- U6: value (none) -> LP3985IM5-2.7
- moved J2 70.1 mm to (69.0, 36.5)
Connections:
- removed net !RFM_RST: U$29.32
- removed net !RFM_SS: U$29.33
- removed net GPS_PPS: U$29.31
- removed net RFM_DIO0: U$29.21
- net GND: now also C12.-; no longer J3.1, TP4.TP, TP5.TP
- net V_PYRO: now also C12.+; no longer J3.2
Routing:
- net RFM_DIO0: track 9.33 -> 0.00 mm, vias 1 -> 0
- net V_PYRO: track 36.8 -> 36.3 mm
Changed lines of the file:
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@@
 <?xml version="1.0" encoding="utf-8"?>
 <!DOCTYPE eagle SYSTEM "eagle.dtd">
-<eagle version="7.7.0">
+<eagle version="7.3.0">
 <drawing>
 <settings>
@@
 </element>
 <element name="U5" library="kg-ic" package="TFLGA16L" value="LSM6DS33" x="44" y="14" rot="R270"/>
-<element name="U6" library="kg-generic" package="SOT23-5" value="" x="23.5" y="24.5" rot="R90"/>
+<element name="U6" library="kg-generic" package="SOT23-5" value="LP3985IM5-2.7" x="23.5" y="24.5" rot="R90"/>
 <element name="C11" library="kg-generic" package="C603" value="1u" x="22" y="25.25" rot="MR180"/>
 <element name="R12" library="kg-generic" package="R0603" value="100" x="22" y="23.5" rot="MR0"/>
@@
 <element name="R25" library="kg-generic" package="R0603" value="100k" x="7.5" y="18.5" rot="MR270"/>
 <element name="JP1" library="SparkFun-Passives" package="PAD-JUMPER-2-NO_YES_SILK" value="BYPASS2" x="27" y="22.5" rot="MR0"/>
-<element name="J3" library="kg-amp-ct" package="JST-2-PTH-VERT" value="BATT_PYRO" x="17" y="24.95" rot="R180"/>
 <element name="J4" library="kg-amp-ct" package="JST-4-PTH-VERT" value="" x="34" y="3"/>
 <element name="C13" library="kg-generic" package="C603" value="100n" x="47.5" y="9.5" rot="MR270"/>
@@
 <attribute name="TP_SIGNAL_NAME" value="" x="57.5" y="4.5" size="1.778" layer="27" display="off"/>
 </element>
-<element name="TP4" library="testpad" package="B1,27" value="TPB1,27" x="31" y="22">
-<attribute name="TP_SIGNAL_NAME" value="" x="31" y="22" size="1.778" layer="27" display="off"/>
-</element>
-<element name="TP5" library="testpad" package="B1,27" value="TPB1,27" x="44.5" y="25.5">
-<attribute name="TP_SIGNAL_NAME" value="" x="44.5" y="25.5" size="1.778" layer="27" display="off"/>
-</element>
 <element name="U10" library="kg-ic" package="LGA8" value="MPL3115A2" x="53.5" y="17.5">
 <attribute name="PROD_ID" value="IC-10869" x="53.5" y="17.5" size="1.778" layer="27" display="off"/>
 </element>
 <element name="C6" library="kg-generic" package="C603" value="" x="56.5" y="14"/>
-<element name="JP2" library="SparkFun-Passives" package="PAD-JUMPER-2-NO_YES_SILK" value="BYPASS2" x="55" y="12"/>
-<element name="JP3" library="SparkFun-Passives" package="PAD-JUMPER-2-NO_YES_SILK" value="BYPASS2" x="52" y="13"/>
+<element name="JP2" library="SparkFun-Passives" package="PAD-JUMPER-2-NO_YES_SILK" value="CFG1" x="55" y="12"/>
+<element name="JP3" library="SparkFun-Passives" package="PAD-JUMPER-2-NO_YES_SILK" value="CFG2" x="52" y="13"/>
 <element name="U1" library="kg-ic" package="VFLGA-12" value="LIS3MDL" x="52" y="7.5" rot="R90"/>
 <element name="C9" library="kg-generic" package="C603" value="" x="52" y="5"/>
-<element name="J2" library="SparkFun-Connectors" package="USB-MINIB" value="USB_MINI-B_SMT" x="5" y="8" rot="MR180">
-<attribute name="SF_ID" value="PRT-00587" x="5" y="8" size="1.778" layer="28" rot="MR180" display="off"/>
-<attribute name="PROD_ID" value="CONN-08193" x="5" y="8" size="1.778" layer="28" rot="MR180" display="off"/>
+<element name="J2" library="SparkFun-Connectors" package="USB-MINIB" value="USB_MINI-B_SMT" x="69" y="36.5" rot="MR180">
+<attribute name="SF_ID" value="PRT-00587" x="69" y="36.5" size="1.778" layer="28" rot="MR180" display="off"/>
+<attribute name="PROD_ID" value="CONN-08193" x="69" y="36.5" size="1.778" layer="28" rot="MR180" display="off"/>
 </element>
 <element name="U8" library="kg-ic" package="QFN16_6X6" value="MMA6825" x="60.5" y="9.5"/>
+<element name="C12" library="rcl" package="E3,5-8" value="3.0F" x="17" y="25.5"/>
 </elements>
 <signals>
@@
 <contactref element="R24" pad="1"/>
 <contactref element="R25" pad="1"/>
-<contactref element="J3" pad="1"/>
 <contactref element="J4" pad="1"/>
 <contactref element="C13" pad="1"/>
@@
 <wire x1="44.2126" y1="7.7874" x2="43.7874" y2="7.7874" width="0.2" layer="16"/>
 <contactref element="TP3" pad="TP"/>
-<contactref element="TP4" pad="TP"/>
-<contactref element="TP5" pad="TP"/>
 <via x="72.5" y="15.5" extent="1-16" drill="0.4" shape="octagon"/>
 <via x="71" y="15.5" extent="1-16" drill="0.4" shape="octagon"/>
@@
 <contactref element="C9" pad="1"/>
 <contactref element="J2" pad="GND"/>
-<wire x1="51.75" y1="6.6" x2="51.1" y2="7.25" width="0" layer="19" extent="1-1"/>
-<wire x1="51.2" y1="5" x2="51.75" y2="6.6" width="0" layer="19" extent="1-1"/>
+<contactref element="C12" pad="-"/>
+<wire x1="70.5" y1="26.5" x2="71.5" y2="38.1" width="0" layer="19" extent="16-16"/>
+<wire x1="51.75" y1="6.6" x2="51.2" y2="5" width="0" layer="19" extent="1-1"/>
+<wire x1="51.1" y1="7.25" x2="51.75" y2="6.6" width="0" layer="19" extent="1-1"/>
 </signal>
 <signal name="KEY">
@@
 <contactref element="U$29" pad="43"/>
 </signal>
-<signal name="GPS_PPS">
-<contactref element="U$29" pad="31"/>
-</signal>
 <signal name="LED">
 <contactref element="R6" pad="2"/>
@@
 <wire x1="23" y1="4.5" x2="25.75" y2="7.25" width="0.254" layer="1"/>
 <wire x1="25.75" y1="7.25" x2="25.75" y2="7.75" width="0.254" layer="1"/>
-</signal>
-<signal name="!RFM_SS">
-<contactref element="U$29" pad="33"/>
-</signal>
-<signal name="RFM_DIO0">
-<wire x1="20.5" y1="16" x2="19.75" y2="15.25" width="0.254" layer="16"/>
-<wire x1="19.75" y1="15.25" x2="19.75" y2="12" width="0.254" layer="16"/>
-<via x="19.75" y="12" extent="1-16" drill="0.4" shape="octagon"/>
-<wire x1="20.5" y1="11.25" x2="19.75" y2="12" width="0.254" layer="1"/>
-<contactref element="U$29" pad="21"/>
-<wire x1="20.5" y1="11.25" x2="22.75" y2="11.25" width="0.254" layer="1"/>
-<wire x1="22.75" y1="11.25" x2="23.25" y2="10.75" width="0.254" layer="1"/>
-<wire x1="23.25" y1="10.75" x2="24.25" y2="10.75" width="0.254" layer="1"/>
-</signal>
-<signal name="!RFM_RST">
-<contactref element="U$29" pad="32"/>
 </signal>
 <signal name="N$9">
@@
 <contactref element="R12" pad="2"/>
 <contactref element="R16" pad="1"/>
-<contactref element="J3" pad="2"/>
 <contactref element="X4" pad="1"/>
 <contactref element="X4" pad="3"/>
@@
 <wire x1="23.5" y1="20.85" x2="23.5" y2="21.5" width="0.254" layer="1"/>
 <wire x1="23.5" y1="21.5" x2="24" y2="22" width="0.254" layer="1"/>
-<wire x1="16" y1="25.5" x2="15.5" y2="25.5" width="0.6096" layer="16"/>
+<contactref element="C12" pad="+"/>
+<wire x1="15.5" y1="25.5" x2="15.222" y2="25.5" width="0" layer="19" extent="16-16"/>
 </signal>
 <signal name="SAFE">
