File: eagle/tracker/flight-28mm.sch (EAGLE design)
At the start: 72 parts, among them J1 BATT, J2 USB_MINI-B_SMT, J3 BATT_PYRO, U1 LIS3MDL, U10 MPL3115A2, U3 A25L010A, U4 MAG3110FCR1, U5 LSM6DS33, U7 H3LIS100DL, U8 MMA6825, X4 MICROMATCH-8

Commit message: Changes to LoRa tracker
Parts:
- removed J3: BATT_PYRO, kg-amp-ct:M2-2MM-JST
- removed TP4, TP5: TPB1,27, testpad:TPB1,27
- added C12: 3.0F, rcl:CPOL-EUE3.5-8
- JP2: value BYPASS2 -> CFG1
- JP3: value BYPASS2 -> CFG2
- U6: value (none) -> LP3985IM5-2.7
Connections:
- removed net !RFM_RST: U$29.PA11
- removed net !RFM_SS: U$29.PA12
- removed net GPS_PPS: U$29.PA10
- removed net RFM_DIO0: U$29.PB10
- net GND: now also C12.-; no longer J3.1, TP4.TP, TP5.TP
- net V_PYRO: now also C12.+; no longer J3.2
Other:
- note added: "MPL3115A2 CFG1=open CFG2=open MPL1115A2 CFG1=open CFG2=short MS5607-02 CFG1=short CFG2=short"
- note removed: "SUPERCAP HERE (PACKAGE BY JST CONNECTOR)"
- moved on the sheet: C6, JP2, JP3, U10
