File: eagle/tracker/tracker-ground-v1_1.brd (EAGLE design)
At the start: 90 x 65 mm, 68 parts, among them M1 UBLOX-NEO-6, M2 HOPE-RFM98W, M3 TFT-2.0-OPENSMART-THT, Q1 Si2365, Q2 CPH3448, U1 RT9013-33, U2 MCP73831, U3 A25L010A, U8 STM32L063C, X1 32.768kHz, X4 ANTENNA-PATCH-18X18

Commit message: Ground station updates
Parts:
- removed C12, C13: 100n, kg-generic:C603
- removed R16: 22, kg-generic:R0603
- removed X1: 32.768kHz, kg-crystal:3.2X1.5-2-PAD
- added J1: (no value), SparkFun-Connectors:SIMHOLDER
- added JP5: (no value), pinhead:1X02
- added M4: SIM800C, kg-modules:SIM800C
- added U4: (no value), kg-generic:DPAK
- JP3: value Debug -> I2C
- JP4: value JUMPER-SMT_2_NO_NO-SILK -> (none); device SparkFun-Jumpers:SMT-JUMPER_2_NO_NO-SILK -> pinhead:1X02
- X4: value ANTENNA-PATCH-18X18 -> ANTENNA-PATCH-12X12; device kg-modules:ANT-PATCH-18X18 -> kg-modules:ANT-PATCH-12X12
- moved JP4 91.5 mm to (106.0, 12.5), flipped to the top
- moved C18 86.5 mm to (101.0, 15.0)
- moved C2 86.5 mm to (102.0, 22.0)
- moved C4 86.5 mm to (97.5, 8.50)
- moved D1 86.5 mm to (103.0, 12.5)
- moved LED1 86.5 mm to (90.5, 12.5)
- moved Q1 86.5 mm to (102.0, 12.5)
- moved R12 86.5 mm to (102.0, 9.50)
- moved R7 86.5 mm to (95.0, 12.5)
- moved R8 86.5 mm to (92.5, 12.5)
- moved U1 86.5 mm to (101.0, 18.5)
- moved U2 86.5 mm to (98.0, 12.5)
- moved JP1 86.5 mm to (97.5, 4.00)
- moved C8 86.0 mm to (97.5, 18.5)
- moved C17 84.5 mm to (107.0, 19.0)
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Connections:
- removed net DBG_DTR: U8.11
- removed net N$23: U8.4, X1.2
- removed net N$24: U8.3, X1.1
- removed net N$25: M1.8, R16.1
- new net N$22: C11.2, U8.1
- new net VCC: J1.C1
- net +3V3: now also JP2.4; no longer C11.2, C12.2, C13.2, JP2.2, U8.1
- net GND: now also J1.C5, M4.13, M4.19, M4.21, M4.27, M4.30, M4.31, M4.33, M4.36, M4.37, M4.8; no longer C12.1, C13.1
- net N$8: now also M1.8; no longer R16.2
- net SCL: now also JP2.2; no longer JP2.4
Routing:
- net +3V3: track 260.5 -> 221.7 mm
- net DBG_RXD: track 51.1 -> 74.7 mm
- net DBG_TXD: track 49.2 -> 72.7 mm
- net VBAT_ADC: track 28.5 -> 6.22 mm, vias 2 -> 1
- net SDA: track 56.9 -> 78.3 mm
- net SCL: track 59.8 -> 78.8 mm, vias 3 -> 0
- net BTN_ON: track 22.4 -> 4.38 mm
- net SWDIO: track 29.4 -> 13.6 mm
- net BAT_CHG: track 29.0 -> 14.1 mm, vias 2 -> 1
- net SWCLK: track 26.5 -> 14.8 mm
- net !RST: track 41.4 -> 31.2 mm
- net N$23: track 9.08 -> 0.00 mm
- net N$24: track 6.22 -> 0.00 mm
- net N$18: track 14.2 -> 9.05 mm
- net N$31: track 8.38 -> 11.4 mm
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Other:
- board size 90 x 65 mm -> 110 x 65 mm
- board text added: "LoRa ground station v1.1"
- board text removed: "LoRa ground station v1.0"

Commit message: Changes to LoRa tracker
Parts:
- removed J1: (no value), SparkFun-Connectors:SIMHOLDER
- removed M4: SIM800C, kg-modules:SIM800C
- added M5: SIM800L-MODULE, kg-modules:SIM800L-BOARD
- added R16, R17, R18, R19, R20: 2.2k, kg-generic:R0603
- added X1: (no value), kg-conn-rf:SMA_EDGELAUNCH
- moved JP4 104.6 mm to (4.00, 35.5), turned to 270 degrees
- moved LED2 102.0 mm to (106.0, 35.0), turned to 270 degrees
- moved JP1 101.7 mm to (4.00, 44.0), turned to 270 degrees
- moved R1 100.1 mm to (106.0, 37.0), turned to 0 degrees
- moved R12 97.2 mm to (9.50, 39.5), turned to 90 degrees
- moved C4 95.8 mm to (8.50, 44.0), turned to 270 degrees
- moved R8 95.5 mm to (4.00, 48.5), turned to 180 degrees
- moved LED1 94.5 mm to (4.00, 50.5), turned to 90 degrees
- moved D1 94.2 mm to (12.5, 38.5), turned to 180 degrees
- moved Q1 93.5 mm to (12.5, 39.5), turned to 90 degrees
- moved U2 90.9 mm to (12.5, 43.5), turned to 270 degrees
- moved C18 89.7 mm to (15.0, 40.5), turned to 270 degrees
- moved R7 89.2 mm to (12.5, 46.5), turned to 0 degrees
- moved U1 85.4 mm to (18.5, 40.5), turned to 90 degrees
- moved C8 83.0 mm to (18.5, 44.0), turned to 0 degrees
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Connections:
- removed net N$17: C4.2, JP1.2, JP4.1, Q1.2, R12.2, U2.3
- removed net VCC: J1.C1
- new net GND1: X1.GND@4
- new net GND2: X1.GND@3
- new net GND3: X1.GND@2
- new net GND4: X1.GND@1
- new net GSM_DTR: R16.2, U8.25
- new net GSM_RXD: R18.2, U8.31
- new net GSM_TXD: R17.2, U8.30
- new net N$23: M5.1, X1.P
- new net N$24: M5.11, R16.1, R19.1
- new net N$25: M5.5, R18.1
- new net N$27: M5.4, R17.1, R20.1
- new net V_BATT: C4.2, JP1.2, JP4.1, M5.2, Q1.2, R12.2, U2.3
- net DBG_RXD: no longer U8.13
- net DBG_TXD: no longer U8.12
- net GND: now also M5.6, R19.2, R20.2; no longer J1.C5, M4.13, M4.19, M4.21, M4.27, M4.30, M4.31, M4.33, M4.36, M4.37, M4.8
- net GPS_PPS: now also U8.14; no longer U8.25
- net GPS_RXD: now also U8.13; no longer U8.31
- net GPS_TXD: now also U8.12; no longer U8.30
Routing:
- net DBG_RXD: track 74.7 -> 0.00 mm
- net DBG_TXD: track 72.7 -> 0.00 mm
- net GPS_PPS: track 36.9 -> 4.95 mm, vias 3 -> 1
- net GPS_RXD: track 22.1 -> 4.82 mm, vias 2 -> 1
- net GPS_TXD: track 17.1 -> 0.00 mm, vias 1 -> 0
- net +3V3: track 221.7 -> 206.6 mm
- net N$17: track 12.4 -> 0.00 mm, vias 1 -> 0
- net USB_VBUS: track 15.5 -> 3.96 mm
- net LED: track 23.7 -> 18.0 mm
- net N$34: track 17.9 -> 13.0 mm
- net N$16: track 2.08 -> 0.00 mm
- net N$12: track 2.08 -> 0.00 mm
- net SDA: track 78.3 -> 76.5 mm
- net SCL: track 78.8 -> 77.0 mm
- net N$21: track 13.9 -> 13.2 mm
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