File: eagle/tracker/tracker-ground-v1_1.sch (EAGLE design)
At the start: 68 parts, among them M1 UBLOX-NEO-6, M2 HOPE-RFM98W, M3 TFT-2.0-OPENSMART-THT, Q1 Si2365, Q2 CPH3448, U1 RT9013-33, U2 MCP73831, U3 A25L010A, U8 STM32L063C, X1 32.768kHz, X4 ANTENNA-PATCH-18X18

Commit message: Ground station updates
Parts:
- removed C12, C13: 100n, kg-generic:CAPACITOR_NPOL-0603
- removed R16: 22, kg-generic:RESISTOR-0603
- removed X1: 32.768kHz, kg-crystal:CRYSTALS-NOGND-CFPX-217
- added J1: (no value), SparkFun-Connectors:SIMHOLDERSIM
- added JP5: (no value), pinhead:PINHD-1X2
- added M4: SIM800C, kg-modules:SIM800C
- added U4: (no value), kg-generic:VREG-3PIN-DPAK
- JP3: value Debug -> I2C
- JP4: value JUMPER-SMT_2_NO_NO-SILK -> (none); device SparkFun-Jumpers:JUMPER-SMT_2_NO_NO-SILK -> pinhead:PINHD-1X2
- X4: value ANTENNA-PATCH-18X18 -> ANTENNA-PATCH-12X12; device kg-modules:ANTENNA-PATCH-18X18 -> kg-modules:ANTENNA-PATCH-12X12
Connections:
- removed net DBG_DTR: U8.PA1
- removed net N$23: U8.PC15/O32O, X1.2
- removed net N$24: U8.PC14/O32I, X1.1
- removed net N$25: M1.RES1, R16.1
- new net N$22: C11.2, U8.VLCD/VBAT
- net +3V3: now also JP2.4; no longer C11.2, C12.2, C13.2, JP2.2, U8.VLCD/VBAT
- net GND: now also M4.GND; no longer C12.1, C13.1
- net N$8: now also M1.RES1; no longer R16.2
- net SCL: now also JP2.2; no longer JP2.4
Other:
- moved on the sheet: R11

Commit message: Changes to LoRa tracker
Parts:
- removed J1: (no value), SparkFun-Connectors:SIMHOLDERSIM
- removed M4: SIM800C, kg-modules:SIM800C
- added M5: SIM800L-MODULE, kg-modules:SIM800L-MODULE
- added R16, R17, R18, R19, R20: 2.2k, kg-generic:RESISTOR-0603
- added X1: (no value), kg-conn-rf:SMACONNECTOR_EDGE
Connections:
- removed net N$17: C4.2, JP1.2, JP4.1, Q1.S, R12.2, U2.BAT
- new net GSM_DTR: R16.2, U8.PB12
- new net GSM_RXD: R18.2, U8.PA10
- new net GSM_TXD: R17.2, U8.PA9
- new net N$23: M5.ANT, X1.ANT
- new net N$24: M5.DTR, R16.1, R19.1
- new net N$25: M5.TXD, R18.1
- new net N$27: M5.RXD, R17.1, R20.1
- new net V_BATT: C4.2, JP1.2, JP4.1, M5.VCC, Q1.S, R12.2, U2.BAT
- net DBG_RXD: no longer U8.PA3
- net DBG_TXD: no longer U8.PA2
- net GND: now also M5.GND, R19.2, R20.2; no longer M4.GND
- net GPS_PPS: now also U8.PA4; no longer U8.PB12
- net GPS_RXD: now also U8.PA3; no longer U8.PA10
- net GPS_TXD: now also U8.PA2; no longer U8.PA9
