File: eagle/tracker/tracker-25mm-full.brd (EAGLE design)
At the start: 74 x 28 mm, 78 parts, among them J1 BATT, J3 BATT_PYRO, M1 UBLOX-NEO-M8, M2 HOPE-RFM98W, M4 UBLOX-MAX-M8, U1 MS5637-02, U3 A25L010A, U4 MAG3110FCR1, U5 LSM6DS33, U7 H3LIS100DL, X2 COAX, X4 MICROMATCH-8, X6 COAX

Commit message: Changes to LoRa tracker
Parts:
- removed TP1, TP2, TP3, TP4, TP5: TPB1,27, testpad:B1,27
- added C12: (no value), kg-generic:C603
- added C18: 100n, kg-generic:C603
- added C19, C20: 1u, kg-generic:C603
- added D2, D3: (no value), kg-generic:R0805
- added J2: WM9734TR-ND, SparkFun-Connectors:USB-B-MICRO-SMD_VERT
- added JP2: CFG1, SparkFun-Passives:PAD-JUMPER-2-NO_YES_SILK
- added JP3: CFG2, SparkFun-Passives:PAD-JUMPER-2-NO_YES_SILK
- added R27, R28, R29, R30, R31: 1k, kg-generic:R0603
- added U10: MPL3115A2LGA8, kg-ic:LGA8
- C8: value 1u -> 100n
- U1: value MS5637-02 -> MCP73831; device kg-ic:MS5637 -> kg-supply:SOT23-5
- U2: value (none) -> MIC5504-3.3/LP3985IM5-3.3
- U6: value (none) -> MIC5504-2.8/LP3985IM5-2.7
- moved U1 16.8 mm to (59.0, 9.00), flipped to the bottom, turned to 180 degrees
- moved D1 9.43 mm to (23.0, 7.00), turned to 90 degrees
- moved R6 8.06 mm to (25.5, 6.00)
- moved J4 8.00 mm to (26.0, 3.00)
- moved J6 8.00 mm to (17.0, 3.00)
- moved C17 3.54 mm to (18.5, 10.0), flipped to the bottom
- moved C3 2.06 mm to (48.0, 17.0), turned to 0 degrees
- moved FB3 1.12 mm to (52.0, 21.0)
- moved PAD1 1.12 mm to (71.8, 11.8)
- moved PAD2 1.12 mm to (71.8, 5.25)
- moved C9 1.00 mm to (55.0, 7.50)
- moved M1 1.00 mm to (59.0, 14.0)
- moved M4 1.00 mm to (60.2, 16.8)
- moved Q1 1.00 mm to (69.0, 6.00)
- moved R15 1.00 mm to (57.0, 20.0)
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Connections:
- new net N$24: C12.2, JP2.1, U10.2
- new net N$26: J2.D+, R29.2
- new net N$27: J2.D-, R28.2
- new net N$28: JP3.1, U10.5
- new net N$30: D3.2, R30.2
- new net N$32: R30.1, U1.1
- new net N$33: R31.2, U1.5
- new net N$8: D2.1, R27.1
- new net RFM_DIO2: M2.16, U$29.2
- new net USB_DM: R28.1, U$29.32
- new net USB_DP: R29.1, U$29.33
- new net VDD_USB: C19.2, D3.1, J2.VBUS, U1.4
- net !RFM_RST: now also U$29.30; no longer U$29.32
- net !RFM_SS: now also U$29.31; no longer U$29.33
- net !RST: no longer TP1.TP
- net 3.3V: now also JP2.2, JP3.2, U10.1, U10.4; no longer U1.1
- net BUZZER: now also U$29.28; no longer U$29.30
- net GND: now also C12.1, C18.1, C19.1, C20.1, D2.2, J2.GND, J2.P1, J2.P2, J2.P3, R31.1, U1.2, U10.3; no longer TP3.TP, TP4.TP, TP5.TP, U1.4
- net GPS_PPS: now also R27.2, U$29.29; no longer TP2.TP, U$29.31
- net GPS_VCC: now also C18.2
- net SCL: now also U10.8; no longer U1.3
- net SDA: now also U10.7; no longer U1.2
- net V_BATT: now also C20.2, U1.3
Routing:
- net N$27: track 0.00 -> 27.2 mm, vias 0 -> 2
- net N$26: track 0.00 -> 27.2 mm, vias 0 -> 2
- net VDD_USB: track 0.00 -> 18.1 mm, vias 0 -> 2
- net RFM_DIO2: track 0.00 -> 12.8 mm, vias 0 -> 3
- net 3.3V: track 139.8 -> 151.2 mm, vias 12 -> 13
- net N$32: track 0.00 -> 8.73 mm
- net N$24: track 0.00 -> 8.40 mm
- net V_BATT: track 60.2 -> 67.3 mm, vias 4 -> 5
- net LED: track 9.07 -> 2.00 mm
- net !RFM_SS: track 12.2 -> 18.0 mm
- net !RFM_RST: track 11.8 -> 17.5 mm
- net DBG_RX: track 14.0 -> 19.4 mm
- net USB_DM: track 0.00 -> 5.12 mm
- net DBG_TX: track 14.5 -> 18.8 mm
- net USB_DP: track 0.00 -> 3.86 mm
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Other:
- board size 74 x 28 mm -> 75 x 28 mm
- board text added: "(c) 2018 Karlis Goba"
- board text added: "J1"
- board text added: "J2"
- board text added: "J3"
- board text added: "J4"
- board text added: "PYRO"
- board text added: "TinySky"
- board text added: "UART"
- board text removed: "(C) Karlis Goba 2017"
- board text removed: "(c) Karlis Goba 2018"
- board text removed: "LoRa-TINY"
- board text removed: "Tracker"

Commit message: Minor update
Parts:
- C1, C8: value 100n -> 10n
- C12: value (none) -> 100n
- D1: value (none) -> RED
- D2: value (none) -> GREEN
- D3: value (none) -> YELLOW
- J4: value (none) -> PROG
- J6: value (none) -> UART
- L1: value (none) -> NF
- M2: device kg-modules:HOPE-RFM -> kg-modules:MOD-RFM95
- Q1, Q2, Q3, Q4: value (none) -> PMV30UN2
- R12: value 100 -> 27
- R2, R5: value 10k -> 100k
- R28, R29: value 1k -> 27
- R3, R4: value 4k7 -> 3.3k
- R31: value 1k -> *2.0k
- R9: value (none) -> 3.3k
- U10: value MPL3115A2LGA8 -> MPL3115A2
- renumbered U$29 to U8
