File: eagle/tracker/tracker-25mm-full.brd (EAGLE design)
At the start: 75 x 28 mm, 88 parts, among them J1 BATT, J2 WM9734TR-ND, J3 BATT_PYRO, J4 PROG, J6 UART, M1 UBLOX-NEO-M8, M2 HOPE-RFM98W, M4 UBLOX-MAX-M8, Q1 PMV30UN2, Q2 PMV30UN2, Q3 PMV30UN2, Q4 PMV30UN2, U1 MCP73831, U10 MPL3115A2, U2 MIC5504-3.3/LP3985IM5-3.3, U3 A25L010A, U4 MAG3110FCR1, U5 LSM6DS33, U6 MIC5504-2.8/LP3985IM5-2.7, U7 H3LIS100DL, U8 STM32L063C, X2 COAX, X4 MICROMATCH-8, X6 COAX

Commit message: Fixed a critical bug in PCB
Connections:
- net 3.3V: now also U7.P15
- net GND: no longer U7.P15
Routing:
- net SCL: track 23.7 -> 25.9 mm
- net GND: track 25.2 -> 26.0 mm, vias 106 -> 105
- net 3.3V: track 151.2 -> 150.4 mm, vias 13 -> 15

Commit message: Updates for v1.01
Parts:
- R27, R6: value 1k -> 470
Other:
- board text added: "v1.01"
- board text removed: "v1.0"
Changed lines of the file:
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@@
 <layer number="19" name="Unrouted" color="14" fill="1" visible="yes" active="yes"/>
 <layer number="20" name="Dimension" color="15" fill="1" visible="yes" active="yes"/>
-<layer number="21" name="tPlace" color="7" fill="1" visible="no" active="yes"/>
-<layer number="22" name="bPlace" color="7" fill="1" visible="no" active="yes"/>
+<layer number="21" name="tPlace" color="7" fill="1" visible="yes" active="yes"/>
+<layer number="22" name="bPlace" color="7" fill="1" visible="yes" active="yes"/>
 <layer number="23" name="tOrigins" color="15" fill="1" visible="yes" active="yes"/>
 <layer number="24" name="bOrigins" color="15" fill="1" visible="yes" active="yes"/>
@@
 <text x="31" y="6.5" size="1.016" layer="21" font="vector" ratio="16" rot="R180">PROG</text>
 <text x="32.5" y="22.5" size="1.016" layer="21" font="vector" ratio="16" rot="R180">BAT</text>
-<text x="68" y="24" size="1.016" layer="21" font="vector" ratio="16">v1.0</text>
+<text x="68" y="24" size="1.016" layer="21" font="vector" ratio="16">v1.01</text>
 <text x="15" y="33.5" size="1.778" layer="48" font="vector">TODO:
 - TABS for battery straps
@@
 <element name="PAD2" library="wirepad" package="SMD2,54-5,08" value="" x="71.75" y="5.25" rot="MR90"/>
 <element name="C10" library="kg-generic" package="C603" value="100n" x="29.5" y="20" rot="R270"/>
-<element name="R6" library="kg-generic" package="R0603" value="1k" x="25.5" y="6"/>
+<element name="R6" library="kg-generic" package="R0603" value="470" x="25.5" y="6"/>
 <element name="R2" library="kg-generic" package="R0603" value="100k" x="69" y="9"/>
 <element name="R7" library="kg-generic" package="R0603" value="1k" x="69" y="11"/>
@@
 <element name="JP2" library="SparkFun-Passives" package="PAD-JUMPER-2-NO_YES_SILK" value="CFG1" x="48.5" y="25" rot="R180"/>
 <element name="JP3" library="SparkFun-Passives" package="PAD-JUMPER-2-NO_YES_SILK" value="CFG2" x="45.5" y="25"/>
-<element name="R27" library="kg-generic" package="R0603" value="1k" x="50.5" y="5" rot="R270"/>
+<element name="R27" library="kg-generic" package="R0603" value="470" x="50.5" y="5" rot="R270"/>
 <element name="D2" library="kg-generic" package="R0805" value="GREEN" x="50.5" y="8.5" rot="R90"/>
 <element name="C18" library="kg-generic" package="C603" value="100n" x="53" y="18.5" rot="MR90"/>

Commit message: Updated documentation
Parts:
- U3: value A25L010A -> A25L010A/SST26VF016B
Changed lines of the file:
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@@
 <elements>
 <element name="FB1" library="microbuilder_v3" package="_0805" value="" x="35" y="17.5" rot="R90"/>
-<element name="U3" library="kg-ic" package="SOP08" value="A25L010A" x="45" y="6.5" rot="R90"/>
+<element name="U3" library="kg-ic" package="SOP08" value="A25L010A/SST26VF016B" x="45" y="6.5" rot="R90"/>
 <element name="R3" library="rcl" package="R0603" value="3.3k" x="45.5" y="18" rot="MR180"/>
 <element name="R4" library="rcl" package="R0603" value="3.3k" x="45.5" y="20" rot="MR180"/>
