File: eagle/tracker/tracker-25mm-full.sch (EAGLE design)
At the start: 67 parts, among them J1 BATT, J2 SHDN, J3 BATT_PYRO, J5 SAFE/ARM, M1 UBLOX-NEO-M8, M2 HOPE-RFM98W, M3 SIM800L-MODULE, U1 MS5637-02, U3 A25L010A, U4 MAG3110FCR1, U5 LSM6DS33, X1 MICROMATCH-4, X5 B3710U410

Commit message: Added pyro sensing and uBlox MAX support
Parts:
- removed D2: (no value), diode:DIODE-2AC|CASOT23
- removed J2: SHDN, kg-amp-ct:M2-CT-V
- removed J5: SAFE/ARM, kg-amp-ct:M2-CT-V
- removed M3: SIM800L-MODULE, kg-modules:SIM800L-MODULE
- added J6: (no value), kg-amp-ct:M3-CT-V
- added L1: (no value), kg-generic:L-0603
- added M4: UBLOX-MAX-M8, kg-modules:UBLOX-MAX-M8
- added Q4: (no value), kg-generic:MOSFET-N-SOT23-3
- added R15: 3.3k, rcl:R-EU_R0603
- added R17, R18: 100k, kg-generic:RESISTOR-0603
- added R20, R26: 1k, kg-generic:RESISTOR-0603
- added X4: MICROMATCH-8, con-amp-micromatch:MICROMATCH-8
- X1: value MICROMATCH-4 -> 87758-0416; device con-amp-micromatch:MICROMATCH-4 -> con-molex:87758-0416
Connections:
- removed net !GSM_EN: M3.DTR
- removed net !GSM_RST: M3.!RST
- removed net GSM_RXD: M3.TXD
- removed net GSM_TXD: M3.RXD
- removed net N$26: C12.+, J3.2, JP1.2, R12.2, R16.1, X1-1.S, X1-3.S
- removed net N$27: Q3.D, R22.1, X1-2.S
- removed net N$28: Q2.D, R21.1, X1-4.S
- removed net N$30: D2.C, J5.2, R5.2
- new net DBG_RX: J6.2, U$29.PA3
- new net DBG_TX: J6.3, U$29.PA2
- new net N$24: M4.!RESET, R15.1
- new net N$29: Q4.G, R20.2, R26.1
- new net PYRO1_OUT: Q2.D, R21.1, X4-2.S
- new net PYRO2_OUT: Q3.D, R22.1, X4-4.S
- new net SAFE: R20.1, R5.2, X4-6.S
- new net SENSE_ARM: R26.2, U$29.PA7
- new net SHDN: R10.1, U2.EN, X4-8.S
- new net VCC_PYRO: C12.+, J3.2, JP1.2, R12.2, R16.1, X4-1.S, X4-3.S
- net !RFM_RST: no longer U$29.PB12
- net !RFM_SS: no longer U$29.PB9
- net 3.3V: now also R5.1
- net CMD1: now also R17.1, U$29.PB0
- net CMD2: now also R18.1, U$29.PB1
- net GND: now also J6.1, L1.1, M4.GND, M4.V_BCKP, Q4.S, R17.2, R18.2, X4-5.S, X4-7.S; no longer J2.1, J5.1, M3.GND, Q2.S, Q3.S, R5.1
- net GPS_PPS: now also M4.TIMEPULSE; no longer U$29.PB8
- net GPS_RXD: now also M4.TXD
- net GPS_TXD: now also M4.RXD
- net GPS_VCC: now also M4.VCC, M4.VCC_IO, R15.2
- net LED: no longer U$29.PA15
- net N$17: now also Q2.S, Q3.S, Q4.D; no longer J2.2, R10.1, U2.EN
- net N$20: no longer D2.A1
- net N$25: no longer D2.A2
- net N$5: now also L1.2
- net N$8: now also M4.RF_IN
- net SENSE1: now also U$29.PA5; no longer U$29.PA3
- net SENSE2: now also U$29.PA4; no longer U$29.PA2
- net V_BATT: no longer M3.VCC
Other:
- moved on the sheet: C10, C11, C12, C2, C4, C5, C8, J1, J3, JP1, JP5, M1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

Commit message: Updates
Parts:
- removed X3: (no value), kg-conn-rf:SMACONNECTOR_EDGE
- added X6: COAX, kg-conn-rf:COAX
- R20: value 1k -> 10k
- R5: value 100k -> 10k
- X2: value (none) -> COAX; device kg-conn-rf:SMACONNECTOR_EDGE -> kg-conn-rf:COAX
Connections:
- net CMD1: now also U$29.PB1; no longer U$29.PB0
- net CMD2: now also U$29.PB0; no longer U$29.PB1
- net GND: now also X2COAX.GND, X6COAX.GND; no longer X2.GND1, X2.GND2, X2.GND3, X2.GND4, X3.GND1, X3.GND2, X3.GND3, X3.GND4
- net N$29: now also R20.1, R5.2; no longer R20.2
- net N$31: now also X6COAX.1; no longer X2.ANT
- net N$5: now also X2COAX.1; no longer X3.ANT
- net RFM_DIO0: now also U$29.PB2
- net SAFE: now also R20.2; no longer R20.1, R5.2
- net SCL: now also U$29.PB8; no longer U$29.PB10
- net SDA: now also U$29.PB9; no longer U$29.PB11
Other:
- moved on the sheet: C13, C14, C15, C6, FB1, M2, R20, R26, R5, U1, U4, U5

Commit message: Updates
Parts:
- removed X5: B3710U410, kg-radio:B3710U410
- C12: device rcl:CPOL-EUE5-8.5 -> rcl:CPOL-EUE3.5-8
Connections:
- removed net N$8: M1.RF_IN, M4.RF_IN, X5.5
- net !FLASH_CS: now also U$29.PA15
- net !RFM_RST: now also U$29.PA11
- net !RFM_SS: now also U$29.PA12
- net !RST: now also J4.4; no longer J4.2
- net BUZZER: now also U$29.PA9
- net GND: no longer X5.1, X5.3, X5.4, X5.6
- net GPS_PPS: now also U$29.PA10
- net N$5: now also M1.RF_IN, M4.RF_IN; no longer X5.2
- net PYRO1_OUT: now also X4-4.S; no longer X4-2.S
- net PYRO2_OUT: now also X4-2.S; no longer X4-4.S
- net SWDIO: now also J4.2; no longer J4.4
Other:
- moved on the sheet: C11, C12, R12, R16, R23

Commit message: Updates to tracker
Parts:
- added J2: (no value), kg-amp-ct:M8-CT-V
- added TP1: TPB1,27, testpad:TPB1,27
- added U7: H3LIS100DL, kg-ic:H3LIS100DL
Connections:
- net !RST: now also TP1.TP; no longer J4.4
- net 3.3V: now also U7.CS, U7.SDO/SA0, U7.VDD, U7.VDD_IO
- net GND: now also U7.GND1, U7.GND2, U7.GND3, U7.GND4, U7.RES1, U7.RES2
- net SCL: now also U7.SCK/SCL
- net SDA: now also U7.SDI/SDA
Changed lines of the file:
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@@
 <part name="X2" library="kg-conn-rf" deviceset="COAX" device=""/>
 <part name="FRAME4" library="SparkFun-Aesthetics" deviceset="FRAME-A4L" device=""/>
+<part name="U7" library="kg-ic" deviceset="H3LIS100" device="DL"/>
+<part name="U$24" library="kg-generic" deviceset="GND" device=""/>
+<part name="U$25" library="kg-generic" deviceset="GND" device=""/>
+<part name="SUPPLY11" library="SparkFun-Aesthetics" deviceset="3.3V" device=""/>
+<part name="TP1" library="testpad" deviceset="TP" device="B1,27"/>
+<part name="J2" library="kg-amp-ct" deviceset="M8" device="-CT-V"/>
 </parts>
 <sheets>
@@
 <instance part="X2" gate="COAX" x="246.38" y="45.72"/>
 <instance part="FRAME4" gate="G$1" x="518.16" y="-185.42"/>
+<instance part="U7" gate="G$1" x="685.8" y="-129.54"/>
+<instance part="U$24" gate="G$1" x="718.82" y="-154.94"/>
+<instance part="U$25" gate="G$1" x="652.78" y="-154.94"/>
+<instance part="SUPPLY11" gate="G$1" x="655.32" y="-96.52"/>
+<instance part="TP1" gate="G$1" x="749.3" y="127"/>
+<instance part="J2" gate="G$1" x="744.22" y="93.98"/>
 </instances>
 <busses>
@@
 <pinref part="U$43" gate="G$1" pin="GND"/>
 </segment>
+<segment>
+<pinref part="U7" gate="G$1" pin="GND4"/>
+<wire x1="678.18" y1="-109.22" x2="678.18" y2="-104.14" width="0.1524" layer="91"/>
+<wire x1="678.18" y1="-104.14" x2="685.8" y2="-104.14" width="0.1524" layer="91"/>
+<wire x1="685.8" y1="-104.14" x2="718.82" y2="-104.14" width="0.1524" layer="91"/>
+<wire x1="718.82" y1="-104.14" x2="718.82" y2="-119.38" width="0.1524" layer="91"/>
+<pinref part="U7" gate="G$1" pin="RES1"/>
+<wire x1="718.82" y1="-119.38" x2="718.82" y2="-124.46" width="0.1524" layer="91"/>
+<wire x1="718.82" y1="-124.46" x2="718.82" y2="-134.62" width="0.1524" layer="91"/>
+<wire x1="718.82" y1="-134.62" x2="718.82" y2="-152.4" width="0.1524" layer="91"/>
+<wire x1="711.2" y1="-134.62" x2="718.82" y2="-134.62" width="0.1524" layer="91"/>
+<junction x="718.82" y="-134.62"/>
+<pinref part="U7" gate="G$1" pin="GND2"/>
+<wire x1="711.2" y1="-124.46" x2="718.82" y2="-124.46" width="0.1524" layer="91"/>
+<junction x="718.82" y="-124.46"/>
+<pinref part="U7" gate="G$1" pin="GND3"/>
+<wire x1="711.2" y1="-119.38" x2="718.82" y2="-119.38" width="0.1524" layer="91"/>
+<junction x="718.82" y="-119.38"/>
+<pinref part="U7" gate="G$1" pin="RES2"/>
+<wire x1="685.8" y1="-109.22" x2="685.8" y2="-104.14" width="0.1524" layer="91"/>
+<junction x="685.8" y="-104.14"/>
+<pinref part="U$24" gate="G$1" pin="GND"/>
+</segment>
+<segment>
+<pinref part="U7" gate="G$1" pin="GND1"/>
+<wire x1="660.4" y1="-139.7" x2="652.78" y2="-139.7" width="0.1524" layer="91"/>
+<wire x1="652.78" y1="-139.7" x2="652.78" y2="-152.4" width="0.1524" layer="91"/>
+<pinref part="U$25" gate="G$1" pin="GND"/>
+</segment>
 </net>
 <net name="SCK" class="0">
@@
 </segment>
 <segment>
-<label x="767.08" y="121.92" size="1.27" layer="95" ratio="12" rot="R180" xref="yes"/>
-<wire x1="767.08" y1="121.92" x2="774.7" y2="121.92" width="0.1524" layer="91"/>
-<pinref part="J4" gate="G$1" pin="4"/>
+<label x="744.22" y="121.92" size="1.27" layer="95" ratio="12" rot="R180" xref="yes"/>
+<wire x1="744.22" y1="121.92" x2="749.3" y2="121.92" width="0.1524" layer="91"/>
+<pinref part="TP1" gate="G$1" pin="TP"/>
+<wire x1="749.3" y1="124.46" x2="749.3" y2="121.92" width="0.1524" layer="91"/>
 </segment>
 </net>
@@
 <label x="538.48" y="-48.26" size="1.27" layer="95" rot="MR0" xref="yes"/>
 </segment>
+<segment>
+<pinref part="U7" gate="G$1" pin="SDI/SDA"/>
+<wire x1="678.18" y1="-149.86" x2="678.18" y2="-160.02" width="0.1524" layer="91"/>
+<wire x1="678.18" y1="-160.02" x2="650.24" y2="-160.02" width="0.1524" layer="91"/>
+<label x="650.24" y="-160.02" size="1.27" layer="95" rot="R180" xref="yes"/>
+</segment>
 </net>
 <net name="SCL" class="0">
@@
 <wire x1="546.1" y1="-50.8" x2="538.48" y2="-50.8" width="0.1524" layer="91"/>
 <label x="538.48" y="-50.8" size="1.27" layer="95" rot="MR0" xref="yes"/>
+</segment>
+<segment>
+<pinref part="U7" gate="G$1" pin="SCK/SCL"/>
+<wire x1="660.4" y1="-134.62" x2="650.24" y2="-134.62" width="0.1524" layer="91"/>
+<label x="650.24" y="-134.62" size="1.27" layer="95" rot="R180" xref="yes"/>
 </segment>
 </net>
@@
 <pinref part="SUPPLY7" gate="G$1" pin="3.3V"/>
 </segment>
-</net>
+<segment>
+<pinref part="U7" gate="G$1" pin="VDD"/>
+<wire x1="693.42" y1="-109.22" x2="693.42" y2="-99.06" width="0.1524" layer="91"/>
+<wire x1="693.42" y1="-99.06" x2="655.32" y2="-99.06" width="0.1524" layer="91"/>
+<wire x1="655.32" y1="-99.06" x2="655.32" y2="-119.38" width="0.1524" layer="91"/>
+<pinref part="U7" gate="G$1" pin="VDD_IO"/>
+<wire x1="655.32" y1="-119.38" x2="660.4" y2="-119.38" width="0.1524" layer="91"/>
+<wire x1="655.32" y1="-99.06" x2="655.32" y2="-96.52" width="0.1524" layer="91"/>
+<junction x="655.32" y="-99.06"/>
+<pinref part="SUPPLY11" gate="G$1" pin="3.3V"/>
+<pinref part="U7" gate="G$1" pin="CS"/>
+<wire x1="693.42" y1="-149.86" x2="693.42" y2="-152.4" width="0.1524" layer="91"/>
+<wire x1="693.42" y1="-152.4" x2="685.8" y2="-152.4" width="0.1524" layer="91"/>
+<wire x1="685.8" y1="-152.4" x2="655.32" y2="-152.4" width="0.1524" layer="91"/>
+<wire x1="655.32" y1="-152.4" x2="655.32" y2="-119.38" width="0.1524" layer="91"/>
+<junction x="655.32" y="-119.38"/>
+<pinref part="U7" gate="G$1" pin="SDO/SA0"/>
+<wire x1="685.8" y1="-149.86" x2="685.8" y2="-152.4" width="0.1524" layer="91"/>
+<junction x="685.8" y="-152.4"/>
+</segment>
+</net>

Commit message: Tracker ready for order
Parts:
- removed C12: (no value), rcl:CPOL-EUE3.5-8
- removed J2: (no value), kg-amp-ct:M8-CT-V
- removed X1: 87758-0416, con-molex:87758-0416
- added C16: 1u, kg-generic:CAPACITOR_NPOL-0603
- added C17: 100n, kg-generic:CAPACITOR_NPOL-0603
- added TP2, TP3, TP4, TP5: TPB1,27, testpad:TPB1,27
Connections:
- net N$24 renamed !GPS_RST
- removed net VCC_PYRO: C12.+, J3.2, JP1.2, R12.2, R16.1, X4-1.S, X4-3.S
- new net V_PYRO: J3.2, JP1.2, R12.2, R16.1, X4-1.S, X4-3.S
- net !RST: now also J4.4
- net 3.3V: now also C16.2, C17.2
- net GND: now also C16.1, C17.1, TP3.TP, TP4.TP, TP5.TP; no longer C12.-
- net GPS_PPS: now also TP2.TP
- net LED: now also U$29.PB12
Other:
- note added: "SUPERCAP HERE (PACKAGE BY JST CONNECTOR)"
- moved on the sheet: C10, R11, R13, TP1

Commit message: Updates
Connections:
- net CMD1 renamed D_PYRO2
- net CMD2 renamed D_PYRO1
- net PYRO_SENSE renamed SENSE_VPYRO
- net SENSE1 renamed SENSE_P2
- net SENSE2 renamed SENSE_P1
- net V_BATT_SENSE renamed SENSE_VBATT
- net RFM_DIO0: now also U$29.PB10; no longer U$29.PB2
Changed lines of the file:
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@@
 </segment>
 <segment>
-<label x="548.64" y="134.62" size="1.27" layer="95" rot="MR0" xref="yes"/>
-<wire x1="548.64" y1="134.62" x2="568.96" y2="134.62" width="0.1524" layer="91"/>
-<pinref part="U$29" gate="G$1" pin="PB2"/>
+<label x="614.68" y="134.62" size="1.27" layer="95" rot="MR180" xref="yes"/>
+<pinref part="U$29" gate="G$1" pin="PB10"/>
+<wire x1="599.44" y1="134.62" x2="614.68" y2="134.62" width="0.1524" layer="91"/>
 </segment>
 </net>
@@
 </segment>
 </net>
-<net name="CMD1" class="0">
+<net name="D_PYRO2" class="0">
 <segment>
 <wire x1="429.26" y1="-83.82" x2="426.72" y2="-83.82" width="0.1524" layer="91"/>
@@
 </segment>
 </net>
-<net name="CMD2" class="0">
+<net name="D_PYRO1" class="0">
 <segment>
 <wire x1="429.26" y1="-111.76" x2="426.72" y2="-111.76" width="0.1524" layer="91"/>
@@
 </segment>
 </net>
-<net name="V_BATT_SENSE" class="0">
+<net name="SENSE_VBATT" class="0">
 <segment>
 <label x="551.18" y="162.56" size="1.27" layer="95" rot="R180" xref="yes"/>
@@
 </segment>
 </net>
-<net name="PYRO_SENSE" class="0">
+<net name="SENSE_VPYRO" class="0">
 <segment>
 <pinref part="R16" gate="G$1" pin="2"/>
@@
 </segment>
 </net>
-<net name="SENSE1" class="0">
+<net name="SENSE_P2" class="0">
 <segment>
 <pinref part="R21" gate="G$1" pin="2"/>
@@
 </segment>
 </net>
-<net name="SENSE2" class="0">
+<net name="SENSE_P1" class="0">
 <segment>
 <pinref part="R22" gate="G$1" pin="2"/>

Commit message: Changes to LoRa tracker
Parts:
- removed TP1, TP2, TP3, TP4, TP5: TPB1,27, testpad:TPB1,27
- added C12: (no value), kg-generic:CAPACITOR_NPOL-0603
- added C18: 100n, kg-generic:CAPACITOR_NPOL-0603
- added C19, C20: 1u, kg-generic:CAPACITOR_NPOL-0603
- added D2, D3: (no value), kg-generic:LED0805
- added J2: WM9734TR-ND, SparkFun-Connectors:USB_MICRO-B_FEMALE-SMT-VERT
- added JP2: CFG1, SparkFun-Passives:JUMPER-PAD-2-NOYES_SILK
- added JP3: CFG2, SparkFun-Passives:JUMPER-PAD-2-NOYES_SILK
- added R27, R28, R29, R30, R31: 1k, kg-generic:RESISTOR-0603
- added U10: MPL3115A2LGA8, kg-ic:MPL3115A2LGA8
- C2: PN (none) -> T491A106K006AT
- C8: value 1u -> 100n
- U1: value MS5637-02 -> MCP73831; device kg-ic:MS5637-02 -> kg-supply:MCP73831
- U2: value (none) -> MIC5504-3.3/LP3985IM5-3.3
- U6: value (none) -> MIC5504-2.8/LP3985IM5-2.7
Connections:
- new net N$24: C12.2, JP2.1, U10.CAP
- new net N$26: J2.D+, R29.2
- new net N$27: J2.D-, R28.2
- new net N$28: JP3.1, U10.INT2
- new net N$30: D3.C, R30.2
- new net N$32: R30.1, U1.STAT
- new net N$33: R31.2, U1.PRG
- new net N$8: D2.A, R27.1
- new net RFM_DIO2: M2.DIO2, U$29.PC13
- new net USB_DM: R28.1, U$29.PA11
- new net USB_DP: R29.1, U$29.PA12
- new net VDD_USB: C19.2, D3.A, J2.VBUS, U1.VDD
- net !RFM_RST: now also U$29.PA9; no longer U$29.PA11
- net !RFM_SS: now also U$29.PA10; no longer U$29.PA12
- net !RST: no longer TP1.TP
- net 3.3V: now also JP2.2, JP3.2, U$29.VLCD/VBAT, U10.VDD, U10.VDDIO; no longer U$29.VBAT, U1.VDD
- net BUZZER: now also U$29.PB15; no longer U$29.PA9
- net GND: now also C12.1, C18.1, C19.1, C20.1, D2.C, J2.GND, J2.SHIELD, R31.1, U1.VSS, U10.GND; no longer TP3.TP, TP4.TP, TP5.TP, U1.GND
- net GPS_PPS: now also R27.2, U$29.PA8; no longer TP2.TP, U$29.PA10
- net GPS_VCC: now also C18.2
- net SCL: now also U10.SCL; no longer U1.SCL
- net SDA: now also U10.SDA; no longer U1.SDA
- net SWCLK: now also U$29.PA14; no longer U$29.SWCLK/PA14
- net SWDIO: now also U$29.PA13; no longer U$29.SWDIO/PA13
- net V_BATT: now also C20.2, U1.BAT
Other:
- note added: "MPL3115A2 CFG1=open CFG2=open MPL1115A2 CFG1=open CFG2=short MS5607-02 CFG1=short CFG2=short"
- note added: "TODO: - SAW filter for GPS - NEO 6/7/8 compatibility - Better MCU power decouple - DIO2/DIO1 to MCU"
- note removed: "TODO: - SAW filter for GPS - NEO 6/7/8 compatibility - Buzzer package - VBat sensing"
- moved on the sheet: C9, FB3

Commit message: Minor update
Parts:
- C1, C8: value 100n -> 10n
- C12: value (none) -> 100n
- D1: value (none) -> RED
- D2: value (none) -> GREEN
- D3: value (none) -> YELLOW
- J1, J3: device kg-amp-ct:M2-CT-V -> kg-amp-ct:M2-2MM-JST
- J4: value (none) -> PROG
- J6: value (none) -> UART
- L1: value (none) -> NF
- Q1, Q2, Q3, Q4: value (none) -> PMV30UN2
- R12: value 100 -> 27
- R2, R5: value 10k -> 100k
- R28, R29: value 1k -> 27
- R3, R4: value 4k7 -> 3.3k
- R31: value 1k -> *2.0k
- R9: value (none) -> 3.3k
- U10: value MPL3115A2LGA8 -> MPL3115A2; device kg-ic:MPL3115A2LGA8 -> kg-ic:MPL3115A2
- renumbered U$29 to U8
Other:
- note added: "MPL3115A2 CFG1=open CFG2=open MPL115A2 CFG1=open CFG2=short MS5607-02 CFG1=short CFG2=short"
- note added: "TODO: - Better MCU supply decouple"
- note removed: "MPL3115A2 CFG1=open CFG2=open MPL1115A2 CFG1=open CFG2=short MS5607-02 CFG1=short CFG2=short"
- note removed: "TODO: - SAW filter for GPS - NEO 6/7/8 compatibility - Better MCU power decouple - DIO2/DIO1 to MCU"
- moved on the sheet: C2, C5, JP5
