File: eagle/tracker/tracker-25mm-full.sch (EAGLE design)
At the start: 88 parts, among them J1 BATT, J2 WM9734TR-ND, J3 BATT_PYRO, J4 PROG, J6 UART, M1 UBLOX-NEO-M8, M2 HOPE-RFM98W, M4 UBLOX-MAX-M8, Q1 PMV30UN2, Q2 PMV30UN2, Q3 PMV30UN2, Q4 PMV30UN2, U1 MCP73831, U10 MPL3115A2, U2 MIC5504-3.3/LP3985IM5-3.3, U3 A25L010A, U4 MAG3110FCR1, U5 LSM6DS33, U6 MIC5504-2.8/LP3985IM5-2.7, U7 H3LIS100DL, U8 STM32L063C, X2 COAX, X4 MICROMATCH-8, X6 COAX

Commit message: Fixed a critical bug in PCB
Connections:
- net 3.3V: now also U7.RES2
- net GND: no longer U7.RES2
Changed lines of the file:
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@@
 <pinref part="U7" gate="G$1" pin="GND4"/>
 <wire x1="678.18" y1="-109.22" x2="678.18" y2="-104.14" width="0.1524" layer="91"/>
-<wire x1="678.18" y1="-104.14" x2="685.8" y2="-104.14" width="0.1524" layer="91"/>
-<wire x1="685.8" y1="-104.14" x2="718.82" y2="-104.14" width="0.1524" layer="91"/>
+<wire x1="678.18" y1="-104.14" x2="718.82" y2="-104.14" width="0.1524" layer="91"/>
 <wire x1="718.82" y1="-104.14" x2="718.82" y2="-119.38" width="0.1524" layer="91"/>
 <pinref part="U7" gate="G$1" pin="RES1"/>
@@
 <wire x1="711.2" y1="-119.38" x2="718.82" y2="-119.38" width="0.1524" layer="91"/>
 <junction x="718.82" y="-119.38"/>
-<pinref part="U7" gate="G$1" pin="RES2"/>
-<wire x1="685.8" y1="-109.22" x2="685.8" y2="-104.14" width="0.1524" layer="91"/>
-<junction x="685.8" y="-104.14"/>
 <pinref part="U$24" gate="G$1" pin="GND"/>
 </segment>
@@
 <pinref part="U7" gate="G$1" pin="VDD"/>
 <wire x1="693.42" y1="-109.22" x2="693.42" y2="-99.06" width="0.1524" layer="91"/>
-<wire x1="693.42" y1="-99.06" x2="655.32" y2="-99.06" width="0.1524" layer="91"/>
+<wire x1="693.42" y1="-99.06" x2="685.8" y2="-99.06" width="0.1524" layer="91"/>
+<wire x1="685.8" y1="-99.06" x2="655.32" y2="-99.06" width="0.1524" layer="91"/>
 <wire x1="655.32" y1="-99.06" x2="655.32" y2="-119.38" width="0.1524" layer="91"/>
 <pinref part="U7" gate="G$1" pin="VDD_IO"/>
@@
 <wire x1="685.8" y1="-149.86" x2="685.8" y2="-152.4" width="0.1524" layer="91"/>
 <junction x="685.8" y="-152.4"/>
-</segment>
-<segment>
+<pinref part="U7" gate="G$1" pin="RES2"/>
+<wire x1="685.8" y1="-109.22" x2="685.8" y2="-99.06" width="0.1524" layer="91"/>
+<junction x="685.8" y="-99.06"/>
+</segment>
+<segment>

Commit message: Updates for v1.01
Parts:
- R27, R6: value 1k -> 470
Other:
- note added: "Replacements: - Q2/Q3/Q4: IRLML0030"
- note added: "TODO: - Better MCU supply decouple - High-side SAFE switch? - Remove UART - Add I2C extension connector - 5 pin prog. connector? - 5V supercap? - LIS3MDL mag? - MMA6825 accel?"
- note removed: "TODO: - Better MCU supply decouple"
- moved on the sheet: C19, C4
Changed lines of the file:
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@@
 <part name="C10" library="kg-generic" deviceset="CAPACITOR_NPOL" device="-0603" value="100n"/>
 <part name="U$28" library="kg-generic" deviceset="GND" device=""/>
-<part name="R6" library="kg-generic" deviceset="RESISTOR" device="-0603" value="1k"/>
+<part name="R6" library="kg-generic" deviceset="RESISTOR" device="-0603" value="470"/>
 <part name="R2" library="kg-generic" deviceset="RESISTOR" device="-0603" value="100k"/>
 <part name="R7" library="kg-generic" deviceset="RESISTOR" device="-0603" value="1k"/>
@@
 <part name="JP3" library="SparkFun-Passives" deviceset="JUMPER-PAD-2-NO" device="YES_SILK" value="CFG2"/>
 <part name="SUPPLY18" library="SparkFun-Aesthetics" deviceset="3.3V" device=""/>
-<part name="R27" library="kg-generic" deviceset="RESISTOR" device="-0603" value="1k"/>
+<part name="R27" library="kg-generic" deviceset="RESISTOR" device="-0603" value="470"/>
 <part name="D2" library="kg-generic" deviceset="LED" device="0805" value="GREEN"/>
 <part name="U$52" library="kg-generic" deviceset="GND" device=""/>
@@
 <text x="533.4" y="-116.84" size="3.81" layer="90" font="vector" ratio="12" align="top-left">TODO:
 - Better MCU supply decouple
-</text>
+- High-side SAFE switch?
+- Remove UART
+- Add I2C extension connector
+- 5 pin prog. connector?
+- 5V supercap?
+- LIS3MDL mag?
+- MMA6825 accel?</text>
 <text x="335.28" y="58.42" size="1.27" layer="97">75uA in Inactive State
 15uA Backup battery current</text>
@@
 MPL115A2 CFG1=open CFG2=short
 MS5607-02 CFG1=short CFG2=short</text>
+<text x="533.4" y="-96.52" size="3.81" layer="90" align="top-left">Replacements:
+- Q2/Q3/Q4: IRLML0030</text>
 </plain>
 <instances>
@@
 <instance part="FRAME3" gate="G$1" x="518.16" y="2.54"/>
 <instance part="FRAME2" gate="G$1" x="236.22" y="-185.42"/>
-<instance part="SUPPLY1" gate="G$1" x="299.72" y="-111.76"/>
+<instance part="SUPPLY1" gate="G$1" x="289.56" y="-111.76"/>
 <instance part="U3" gate="G$1" x="632.46" y="43.18"/>
 <instance part="R3" gate="G$1" x="756.92" y="165.1" rot="R90"/>
@@
 <instance part="U$8" gate="G$1" x="358.14" y="-139.7"/>
 <instance part="U$12" gate="G$1" x="266.7" y="-139.7"/>
-<instance part="C4" gate="C" x="299.72" y="-132.08" rot="R90"/>
-<instance part="U$5" gate="G$1" x="299.72" y="-139.7"/>
+<instance part="C4" gate="C" x="289.56" y="-132.08" rot="R90"/>
+<instance part="U$5" gate="G$1" x="289.56" y="-139.7"/>
 <instance part="C5" gate="C" x="365.76" y="-132.08" rot="R90"/>
 <instance part="U$16" gate="G$1" x="365.76" y="-139.7"/>
@@
 <instance part="D3" gate="G$1" x="353.06" y="-162.56" rot="R270"/>
 <instance part="U$56" gate="G$1" x="312.42" y="-177.8"/>
-<instance part="C19" gate="C" x="368.3" y="-165.1" rot="R90"/>
-<instance part="U$57" gate="G$1" x="368.3" y="-177.8"/>
+<instance part="C19" gate="C" x="365.76" y="-165.1" rot="R90"/>
+<instance part="U$57" gate="G$1" x="365.76" y="-177.8"/>
 <instance part="C20" gate="C" x="289.56" y="-165.1" rot="R90"/>
 <instance part="U$58" gate="G$1" x="289.56" y="-177.8"/>
@@
 <pinref part="C4" gate="C" pin="1"/>
 <pinref part="U$5" gate="G$1" pin="GND"/>
-<wire x1="299.72" y1="-137.16" x2="299.72" y2="-134.62" width="0.1524" layer="91"/>
+<wire x1="289.56" y1="-137.16" x2="289.56" y2="-134.62" width="0.1524" layer="91"/>
 </segment>
 <segment>
@@
 <pinref part="U$57" gate="G$1" pin="GND"/>
 <pinref part="C19" gate="C" pin="1"/>
-<wire x1="368.3" y1="-175.26" x2="368.3" y2="-167.64" width="0.1524" layer="91"/>
+<wire x1="365.76" y1="-175.26" x2="365.76" y2="-167.64" width="0.1524" layer="91"/>
 </segment>
 <segment>
@@
 <segment>
 <wire x1="314.96" y1="-124.46" x2="307.34" y2="-124.46" width="0.1524" layer="91"/>
-<wire x1="307.34" y1="-124.46" x2="299.72" y2="-124.46" width="0.1524" layer="91"/>
-<wire x1="299.72" y1="-124.46" x2="271.78" y2="-124.46" width="0.1524" layer="91"/>
-<junction x="299.72" y="-124.46"/>
+<wire x1="307.34" y1="-124.46" x2="289.56" y2="-124.46" width="0.1524" layer="91"/>
+<wire x1="289.56" y1="-124.46" x2="271.78" y2="-124.46" width="0.1524" layer="91"/>
+<junction x="289.56" y="-124.46"/>
 <wire x1="271.78" y1="-124.46" x2="261.62" y2="-124.46" width="0.1524" layer="91"/>
-<wire x1="299.72" y1="-124.46" x2="299.72" y2="-114.3" width="0.1524" layer="91"/>
+<wire x1="289.56" y1="-124.46" x2="289.56" y2="-114.3" width="0.1524" layer="91"/>
 <pinref part="SUPPLY1" gate="G$1" pin="V_BATT"/>
 <pinref part="JP5" gate="G$1" pin="1"/>
-<wire x1="299.72" y1="-114.3" x2="299.72" y2="-111.76" width="0.1524" layer="91"/>
-<wire x1="353.06" y1="-114.3" x2="299.72" y2="-114.3" width="0.1524" layer="91"/>
-<junction x="299.72" y="-114.3"/>
+<wire x1="289.56" y1="-114.3" x2="289.56" y2="-111.76" width="0.1524" layer="91"/>
+<wire x1="353.06" y1="-114.3" x2="289.56" y2="-114.3" width="0.1524" layer="91"/>
+<junction x="289.56" y="-114.3"/>
 <pinref part="C4" gate="C" pin="2"/>
 <pinref part="J1" gate="G$1" pin="2"/>
 <pinref part="U2" gate="G$1" pin="IN"/>
-<wire x1="299.72" y1="-127" x2="299.72" y2="-124.46" width="0.1524" layer="91"/>
+<wire x1="289.56" y1="-127" x2="289.56" y2="-124.46" width="0.1524" layer="91"/>
 <wire x1="307.34" y1="-127" x2="307.34" y2="-124.46" width="0.1524" layer="91"/>
 <junction x="307.34" y="-124.46"/>
@@
 <pinref part="U1" gate="G$1" pin="VDD"/>
 <wire x1="335.28" y1="-157.48" x2="353.06" y2="-157.48" width="0.1524" layer="91"/>
-<label x="381" y="-157.48" size="1.27" layer="95" xref="yes"/>
+<label x="373.38" y="-157.48" size="1.27" layer="95" xref="yes"/>
 <pinref part="D3" gate="G$1" pin="A"/>
-<wire x1="353.06" y1="-157.48" x2="368.3" y2="-157.48" width="0.1524" layer="91"/>
-<wire x1="368.3" y1="-157.48" x2="381" y2="-157.48" width="0.1524" layer="91"/>
+<wire x1="353.06" y1="-157.48" x2="365.76" y2="-157.48" width="0.1524" layer="91"/>
+<wire x1="365.76" y1="-157.48" x2="373.38" y2="-157.48" width="0.1524" layer="91"/>
 <wire x1="353.06" y1="-160.02" x2="353.06" y2="-157.48" width="0.1524" layer="91"/>
 <junction x="353.06" y="-157.48"/>
 <pinref part="C19" gate="C" pin="2"/>
-<wire x1="368.3" y1="-160.02" x2="368.3" y2="-157.48" width="0.1524" layer="91"/>
-<junction x="368.3" y="-157.48"/>
-</segment>
-<segment>
+<wire x1="365.76" y1="-160.02" x2="365.76" y2="-157.48" width="0.1524" layer="91"/>
+<junction x="365.76" y="-157.48"/>
+</segment>
+<segment>

Commit message: Updated documentation
Parts:
- U3: value A25L010A -> A25L010A/SST26VF016B
Other:
- note added: "TODO: - Better MCU supply decouple - High-side SAFE switch? - Remove UART - Add I2C extension connector - 200mil SOIJ flash - Better supercap position/mount - Battery connector position - 5 pin prog. connector? - 5V supercap? - LIS3MDL mag? - MMA6825 accel?"
- note removed: "TODO: - Better MCU supply decouple - High-side SAFE switch? - Remove UART - Add I2C extension connector - 5 pin prog. connector? - 5V supercap? - LIS3MDL mag? - MMA6825 accel?"
Changed lines of the file:
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@@
 <schematic xreflabel="%F%N/%S.%C%R" xrefpart="/%S.%C%R">
 <attributes>
+<attribute name="DESIGNER" value="K. GOBA"/>
 </attributes>
 <variantdefs>
@@
 <part name="FRAME2" library="SparkFun-Aesthetics" deviceset="FRAME-A4L" device=""/>
 <part name="SUPPLY1" library="SparkFun-Aesthetics" deviceset="V_BATT" device=""/>
-<part name="U3" library="kg-ic" deviceset="A25L010A" device=""/>
+<part name="U3" library="kg-ic" deviceset="A25L010A" device="" value="A25L010A/SST26VF016B"/>
 <part name="R3" library="rcl" deviceset="R-EU_" device="R0603" value="3.3k"/>
 <part name="R4" library="rcl" deviceset="R-EU_" device="R0603" value="3.3k"/>
@@
 <sheet>
 <plain>
-<text x="533.4" y="-116.84" size="3.81" layer="90" font="vector" ratio="12" align="top-left">TODO:
+<text x="533.4" y="-109.22" size="3.81" layer="90" font="vector" ratio="12" align="top-left">TODO:
 - Better MCU supply decouple
 - High-side SAFE switch?
 - Remove UART
 - Add I2C extension connector
+- 200mil SOIJ flash
+- Better supercap position/mount
+- Battery connector position
 - 5 pin prog. connector?
 - 5V supercap?
@@
 MPL115A2 CFG1=open CFG2=short
 MS5607-02 CFG1=short CFG2=short</text>
-<text x="533.4" y="-96.52" size="3.81" layer="90" align="top-left">Replacements:
+<text x="533.4" y="-88.9" size="3.81" layer="90" align="top-left">Replacements:
 - Q2/Q3/Q4: IRLML0030</text>
 </plain>

Commit message: Updates
Other:
- note added: "TODO: - Better MCU supply decouple - High-side SAFE switch? - Remove UART - Add I2C extension connector - 200mil SOIJ flash - Better supercap position/mount - Battery connector position - Buzzer PB14/13 (PWM) - Supercap discharge - 5 pin prog. connector? - 5V supercap? - LIS3MDL mag? - MMA6825 accel?"
- note removed: "TODO: - Better MCU supply decouple - High-side SAFE switch? - Remove UART - Add I2C extension connector - 200mil SOIJ flash - Better supercap position/mount - Battery connector position - 5 pin prog. connector? - 5V supercap? - LIS3MDL mag? - MMA6825 accel?"
Changed lines of the file:
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@@
 <sheet>
 <plain>
-<text x="533.4" y="-109.22" size="3.81" layer="90" font="vector" ratio="12" align="top-left">TODO:
+<text x="533.4" y="-88.9" size="3.81" layer="90" font="vector" ratio="12" align="top-left">TODO:
 - Better MCU supply decouple
 - High-side SAFE switch?
@@
 - Better supercap position/mount
 - Battery connector position
+- Buzzer PB14/13 (PWM)
+- Supercap discharge
 - 5 pin prog. connector?
 - 5V supercap?
@@
 MPL115A2 CFG1=open CFG2=short
 MS5607-02 CFG1=short CFG2=short</text>
-<text x="533.4" y="-88.9" size="3.81" layer="90" align="top-left">Replacements:
+<text x="533.4" y="-17.78" size="3.81" layer="90" align="top-left">Replacements:
 - Q2/Q3/Q4: IRLML0030</text>
 </plain>
