File: eagle/relay_shield/mosfet_shield.brd (EAGLE design)
At the start: 80 x 60 mm, 47 parts, among them IC1 ULN2003AD, J1 ARDUINO_R3_SHIELDNOLABELS, J2 Y1B, J3 Y1A, J4 Y2A, J5 X2, J6 Y2B, J7 X1, Q1 PMV33, Q2 PMV33, Q3 PMV33, Q4 PMV33, Q5 PMV33, U1 NCP5501DT50G

Commit message: Updates to tracker
Parts:
- moved C5 6.35 mm to (21.6, 50.8)
- moved R7 6.35 mm to (25.4, 50.8)
- moved R8 6.35 mm to (25.4, 48.3)
Connections:
- net N$15: now also J1.D10; no longer J1.D8
Routing:
- net N$17: track 25.4 -> 19.0 mm
- net N$15: track 3.34 -> 0.00 mm
Changed lines of the file:
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@@
 <layer number="45" name="Holes" color="7" fill="1" visible="yes" active="yes"/>
 <layer number="46" name="Milling" color="3" fill="1" visible="no" active="yes"/>
-<layer number="47" name="Measures" color="7" fill="1" visible="no" active="yes"/>
+<layer number="47" name="Measures" color="7" fill="1" visible="yes" active="yes"/>
 <layer number="48" name="Document" color="7" fill="1" visible="yes" active="yes"/>
 <layer number="49" name="Reference" color="7" fill="1" visible="yes" active="yes"/>
@@
 <hole x="6.35" y="53.975" drill="3.1"/>
 <text x="30.48" y="41.91" size="1.778" layer="16" font="vector" ratio="15" rot="MR0">KG 2018</text>
+<dimension x1="0" y1="57" x2="80" y2="57" x3="40" y3="62.23" textsize="1.27" textratio="14" layer="47"/>
 </plain>
 <attributes>
@@
 <element name="C3" library="kg-generic" package="C1206" value="2.2u" x="16.51" y="19.05" rot="MR270"/>
 <element name="C4" library="kg-generic" package="C1206" value="2.2u" x="31.75" y="19.05" rot="MR270"/>
-<element name="R7" library="kg-generic" package="R0603" value="1k" x="31.75" y="50.8" rot="MR180"/>
-<element name="R8" library="kg-generic" package="R0603" value="1k" x="31.75" y="48.26" rot="MR0"/>
-<element name="C5" library="kg-generic" package="C603" value="" x="27.94" y="50.8" rot="MR0"/>
+<element name="R7" library="kg-generic" package="R0603" value="1k" x="25.4" y="50.8" rot="MR180"/>
+<element name="R8" library="kg-generic" package="R0603" value="1k" x="25.4" y="48.26" rot="MR0"/>
+<element name="C5" library="kg-generic" package="C603" value="" x="21.59" y="50.8" rot="MR0"/>
 <element name="JP5" library="pinhead" package="1X02" value="" x="3.81" y="46.99" rot="R270"/>
 <element name="R9" library="kg-generic" package="R0603" value="1k" x="48.26" y="15.24" rot="MR0"/>
@@
 </signal>
 <signal name="N$15">
-<contactref element="J1" pad="D8"/>
 <contactref element="R7" pad="2"/>
-<wire x1="33.02" y1="53.965" x2="33.02" y2="51.22" width="0.6096" layer="16"/>
-<wire x1="33.02" y1="51.22" x2="32.6" y2="50.8" width="0.6096" layer="16"/>
+<contactref element="J1" pad="D10"/>
+<wire x1="26.25" y1="50.8" x2="27.94" y2="53.965" width="0" layer="19" extent="16-16"/>
 </signal>
 <signal name="N$23">
@@
 <contactref element="R8" pad="2"/>
 <contactref element="C5" pad="1"/>
-<wire x1="28.79" y1="50.8" x2="30.9" y2="50.8" width="0.6096" layer="16"/>
-<wire x1="30.9" y1="50.8" x2="30.9" y2="48.26" width="0.6096" layer="16"/>
+<wire x1="22.44" y1="50.8" x2="24.55" y2="50.8" width="0.6096" layer="16"/>
+<wire x1="24.55" y1="50.8" x2="24.55" y2="48.26" width="0.6096" layer="16"/>
 </signal>
 <signal name="N$17">
 <contactref element="C5" pad="2"/>
 <contactref element="JP5" pad="2"/>
-<wire x1="3.81" y1="45.72" x2="22.01" y2="45.72" width="0.6096" layer="16"/>
-<wire x1="22.01" y1="45.72" x2="27.09" y2="50.8" width="0.6096" layer="16"/>
+<wire x1="3.81" y1="45.72" x2="15.66" y2="45.72" width="0.6096" layer="16"/>
+<wire x1="15.66" y1="45.72" x2="20.74" y2="50.8" width="0.6096" layer="16"/>
 </signal>
 <signal name="NTC_ADC">
