File: eagle/relay_shield/mosfet_shield.sch (EAGLE design)
At the start: 47 parts, among them IC1 ULN2003AD, J1 ARDUINO_R3_SHIELDNOLABELS, J2 Y1B, J3 Y1A, J4 Y2A, J5 X2, J6 Y2B, J7 X1, Q1 PMV33, Q2 PMV33, Q3 PMV33, Q4 PMV33, Q5 PMV33, U1 NCP5501DT50G

Commit message: Updates to tracker
Connections:
- net N$15: now also J1.*D10; no longer J1.D8
Changed lines of the file:
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@@
 <label x="30.48" y="154.94" size="1.4224" layer="95" rot="R180" xref="yes"/>
+</segment>
+<segment>
+<wire x1="86.36" y1="147.32" x2="81.28" y2="147.32" width="0.1524" layer="91"/>
+<label x="86.36" y="147.32" size="1.4224" layer="95" xref="yes"/>
 </segment>
 </net>
@@
 <net name="N$15" class="0">
 <segment>
-<pinref part="J1" gate="G$1" pin="D8"/>
-<wire x1="60.96" y1="139.7" x2="71.12" y2="139.7" width="0.1524" layer="91"/>
 <pinref part="R7" gate="G$1" pin="2"/>
-<wire x1="71.12" y1="99.06" x2="71.12" y2="139.7" width="0.1524" layer="91"/>
+<wire x1="71.12" y1="99.06" x2="71.12" y2="134.62" width="0.1524" layer="91"/>
+<pinref part="J1" gate="G$1" pin="*D10"/>
+<wire x1="60.96" y1="134.62" x2="71.12" y2="134.62" width="0.1524" layer="91"/>
 </segment>
 </net>
