File: eagle/misc/thermostat-2layer-v1.brd (EAGLE design)
At the start: 40 x 18 mm, 36 parts, among them J1 V_EXT, J7 V_EXT, J8 V_BATT, J9 NTC 10k, U1 TL431DBZ

Commit message: Thermostat updates
Parts:
- removed JP1: VREF_LOCAL, SparkFun-Jumpers:SMT-JUMPER_2_NO_NO-SILK
- added PAD1, PAD2: WIREPADSMD1,27-254, wirepad:SMD1,27-2,54
- added R22: NF, kg-generic:R0603
- D4: value (none) -> NF
- R10, R12, R14, R15, R16, R17, R18, R19, R2, R20, R21, R4, R6, R7, R9: value 82 -> 10
- moved R10 23.8 mm to (6.50, 15.0)
- moved R2 23.0 mm to (6.50, 3.00)
- moved R16 18.5 mm to (23.0, 3.00)
- moved R4 17.9 mm to (6.50, 9.00)
- moved R17 17.5 mm to (23.0, 15.0)
- moved R19 15.9 mm to (28.5, 3.00)
- moved R18 12.7 mm to (23.0, 9.00)
- moved R7 11.5 mm to (12.0, 15.0)
- moved R9 8.51 mm to (12.0, 9.00)
- moved R12 8.49 mm to (17.5, 3.00)
- moved R14 6.00 mm to (17.5, 15.0)
- moved R15 6.00 mm to (17.5, 9.00)
- moved R21 5.59 mm to (28.5, 9.00)
- moved R6 5.52 mm to (12.0, 3.00)
- moved R20 5.02 mm to (28.5, 15.0)
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Connections:
- new net N$25: R16.1, R18.2
- net EN/VREF: now also R22.1; no longer JP1.2, R11.2
- net GND: now also PAD2.1, R10.1, R14.1, R7.1; no longer R18.1, R19.1, R21.1
- net LOAD: now also R12.2, R16.2, R19.2; no longer R4.2, R7.2, R9.2
- net N$12: now also R10.2, R4.1; no longer R10.1, R21.2
- net N$19: now also R6.1, R9.2; no longer R12.1, R20.2
- net N$20: now also R7.2, R9.1; no longer R14.1, R19.2
- net N$22: now also R12.1, R15.2; no longer R15.1, R18.2
- net N$24: now also R14.2, R15.1; no longer R16.1, R17.2
- net N$26: now also R17.2, R18.1; no longer R16.2, R9.1
- net N$27: now also R19.1, R21.2; no longer R15.2, R7.1
- net N$28: now also R20.2, R21.1; no longer R14.2, R6.1
- net N$29: now also R11.2, R22.2; no longer R12.2, R4.1
- net N$8: no longer JP1.1
- net N$9: now also R4.2; no longer R10.2
- net SENSE_T: now also PAD1.1
Routing:
- net N$13: track 33.4 -> 27.0 mm
- net N$25: track 0.00 -> 3.16 mm
- net N$23: track 5.83 -> 2.78 mm
- net EN/VREF: track 28.0 -> 26.3 mm
- net LOAD: track 10.2 -> 8.90 mm
- net N$29: track 2.66 -> 1.50 mm
- net N$17: track 20.2 -> 19.2 mm
- net N$15: track 3.95 -> 2.95 mm
- net N$22: track 2.66 -> 3.16 mm
- net N$19: track 2.66 -> 3.16 mm
- net N$9: track 2.66 -> 3.16 mm
- net N$27: track 2.66 -> 3.16 mm
- net N$24: track 2.66 -> 3.16 mm
- net N$20: track 2.66 -> 3.16 mm
- net N$12: track 2.66 -> 3.16 mm
Other:
- board text removed: "TODO: - TABS for battery straps - Check buzzer size - Wire widths"
