File: eagle/misc/thermostat-2layer-v1.sch (EAGLE design)
At the start: 36 parts, among them J1 V_EXT, J7 V_EXT, J8 V_BATT, J9 NTC 10k, U1 TL431DBZ

Commit message: Thermostat updates
Parts:
- removed JP1: VREF_LOCAL, SparkFun-Jumpers:JUMPER-SMT_2_NO_NO-SILK
- added PAD1, PAD2: WIREPADSMD1,27-254, wirepad:WIREPADSMD1,27-254
- added R22: NF, kg-generic:RESISTOR-0603
- D4: value (none) -> NF
- R10, R12, R14, R15, R16, R17, R18, R19, R2, R20, R21, R4, R6, R7, R9: value 82 -> 10
Connections:
- new net N$25: R16.1, R18.2
- net EN/VREF: now also R22.1; no longer JP1.2, R11.2
- net GND: now also PAD2.P, R10.1, R14.1, R7.1; no longer R18.1, R19.1, R21.1
- net LOAD: now also R12.2, R16.2, R19.2; no longer R4.2, R7.2, R9.2
- net N$12: now also R10.2, R4.1; no longer R10.1, R21.2
- net N$19: now also R6.1, R9.2; no longer R12.1, R20.2
- net N$20: now also R7.2, R9.1; no longer R14.1, R19.2
- net N$22: now also R12.1, R15.2; no longer R15.1, R18.2
- net N$24: now also R14.2, R15.1; no longer R16.1, R17.2
- net N$26: now also R17.2, R18.1; no longer R16.2, R9.1
- net N$27: now also R19.1, R21.2; no longer R15.2, R7.1
- net N$28: now also R20.2, R21.1; no longer R14.2, R6.1
- net N$29: now also R11.2, R22.2; no longer R12.2, R4.1
- net N$8: no longer JP1.1
- net N$9: now also R4.2; no longer R10.2
- net SENSE_T: now also PAD1.P
Other:
- moved on the sheet: J9, R10, R12, R14, R15, R16, R17, R18, R19, R20, R21, R4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
